File: GPS-Compass/DEBUG.kicad_sch (KiCad schematic)
At the start: 16 parts

Commit message: gps upd
Parts:
- added D6: BLUE, LED_SMD:LED_0805_2012Metric, symbol Device:LED_Small
- added Q4: BC337, Package_TO_SOT_THT:TO-92_Inline, symbol Transistor_BJT:BC337
- added R29, R33: 1k, Resistor_SMD:R_0805_2012Metric, symbol Device:R_Small
- added R40: 0R, Resistor_SMD:R_0805_2012Metric, symbol Device:R
- BZ1: footprint (none) -> gps-compass_brd:CEM-1203_Buzzer
- D3, D4, D5: footprint (none) -> LED_SMD:LED_0805_2012Metric
- D7: renamed from D6; footprint (none) -> LED_SMD:LED_0805_2012Metric
- D8: renamed from D7; footprint (none) -> LED_SMD:LED_0805_2012Metric
- D9: renamed from D8; footprint (none) -> LED_SMD:LED_0805_2012Metric
- R30: renamed from R28; footprint Resistor_SMD:R_0805_2012Metric_Pad1.20x1.40mm_HandSolder -> Resistor_SMD:R_0805_2012Metric
- R31: renamed from R29; footprint Resistor_SMD:R_0805_2012Metric_Pad1.20x1.40mm_HandSolder -> Resistor_SMD:R_0805_2012Metric
- R32: renamed from R30; footprint Resistor_SMD:R_0805_2012Metric_Pad1.20x1.40mm_HandSolder -> Resistor_SMD:R_0805_2012Metric
- R34: renamed from R31; footprint Resistor_SMD:R_0805_2012Metric_Pad1.20x1.40mm_HandSolder -> Resistor_SMD:R_0805_2012Metric
- R35: renamed from R32; footprint Resistor_SMD:R_0805_2012Metric_Pad1.20x1.40mm_HandSolder -> Resistor_SMD:R_0805_2012Metric
- R36: renamed from R33; footprint Resistor_SMD:R_0805_2012Metric_Pad1.20x1.40mm_HandSolder -> Resistor_SMD:R_0805_2012Metric
- R37: renamed from R34; footprint Resistor_SMD:R_0805_2012Metric_Pad1.20x1.40mm_HandSolder -> Resistor_SMD:R_0805_2012Metric
- R38: renamed from R35; footprint Resistor_SMD:R_0805_2012Metric_Pad1.20x1.40mm_HandSolder -> Resistor_SMD:R_0805_2012Metric
- R39: renamed from R36; footprint Resistor_SMD:R_0805_2012Metric_Pad1.20x1.40mm_HandSolder -> Resistor_SMD:R_0805_2012Metric
Connections:
- net +3V3: now also D6.2 (A)
- net GND: now also BZ1.2 (-), Q4.3 (E)
- net LED_IOXX: now reaches R37.1
- net LED_IOXX: now also R38.1, R39.1
- net at BZ1.1 (+): now also R40.2
- new net: Q4.1 (C), R33.2
- new net: Q4.2 (B), R29.1
- new net: D6.1 (K), R33.1
- new net BZ_PWM: R40.1
- new net GNSS_PPS: R29.2
Other:
- note added: "AUDIO"
- note added: "CHARGER DEBUG"
- note added: "GNSS DEBUG"
- note added: "MISC. DEBUG"
- note added: "good input source"
- note removed: "FIND BUZZR"
- note removed: "good input source signalisation"
- moved on the sheet: BZ1, D3, D4, D5, D7, D8, D9, R30, R31, R32, R34, R35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

Commit message: GNSS layout
Parts:
- removed D6: BLUE, LED_SMD:LED_0805_2012Metric, symbol Device:LED_Small
- removed Q4: BC337, Package_TO_SOT_THT:TO-92_Inline, symbol Transistor_BJT:BC337
- removed R29, R33: 1k, Resistor_SMD:R_0805_2012Metric, symbol Device:R_Small
Other:
- note removed: "GNSS DEBUG"
