File: GPS-Compass/GNSS.kicad_sch (KiCad schematic)
At the start: 25 parts, among them U10 TESEO-LIV3R, U11 TESEO-LIV3R, U12 BGA725L6E6327FTSA1

Commit message: gps upd
Parts:
- removed C32, C33: 56p, Capacitor_SMD:C_0402_1005Metric, symbol Device:C_Small
- removed C34: 10n, Capacitor_SMD:C_0402_1005Metric, symbol Device:C_Small
- removed FL1: B39162B8813P810, Filter:Filter_1109-5_1.1x0.9mm, symbol Filter:B39162B8813P810
- removed L5: 27n, Inductor_SMD:L_0402_1005Metric, symbol Device:L_Small
- removed R37, R38, R41: 10k, Resistor_SMD:R_0603_1608Metric, symbol Device:R_Small
- removed R39, R40: 22, Resistor_SMD:R_0402_1005Metric, symbol Device:R_Small
- removed U11: TESEO-LIV3R, TESEO-LIV3R:TESEOLIV3R, symbol TESEO-LIV3R:TESEO-LIV3R
- added AE1: Antenna, gps-compass_brd:ANT2525B00DT1516S, symbol Device:Antenna
- added C31: 56nF, Capacitor_SMD:C_0402_1005Metric, symbol Device:C_Small
- added FL1: B39162B4327P810, gps-compass_brd:FIL_B39162B4327P810, symbol gps-compass_sch:B39162B4327P810
- C28: renamed from C35; footprint (none) -> Capacitor_SMD:C_0402_1005Metric
- C29: footprint (none) -> Capacitor_SMD:C_0402_1005Metric
- C30: renamed from C31; footprint (none) -> Capacitor_SMD:C_0402_1005Metric
- C32: renamed from C30; footprint (none) -> Capacitor_SMD:C_0402_1005Metric
- C33: renamed from C28; footprint (none) -> Capacitor_SMD:C_0402_1005Metric
- JP5: renamed from JP6; footprint (none) -> Jumper:SolderJumper-2_P1.3mm_Open_RoundedPad1.0x1.5mm
- JP6: renamed from JP5; footprint (none) -> Jumper:SolderJumper-2_P1.3mm_Open_RoundedPad1.0x1.5mm
- JP7: renamed from JP3; footprint (none) -> Jumper:SolderJumper-2_P1.3mm_Open_RoundedPad1.0x1.5mm
- JP8: renamed from JP4; footprint (none) -> Jumper:SolderJumper-2_P1.3mm_Open_RoundedPad1.0x1.5mm
- L4: renamed from L6; footprint (none) -> Inductor_SMD:L_0402_1005Metric
- L5: renamed from L4; footprint (none) -> Inductor_SMD:L_0402_1005Metric
- R41: renamed from R42; footprint (none) -> Resistor_SMD:R_0805_2012Metric
- U10: renamed from U12; footprint BGA725L6E6327FTSA1:AMP_BGA725L6E6327FTSA1 -> gps-compass_brd:AMP_BGA725L6E6327FTSA1
- U11: renamed from U10; footprint ARRAY_LIV3R_STM -> gps-compass_brd:ARRAY_LIV3R_STM
Connections:
- net +3V3: no longer C29.1, U10.2 (VCC)
- net GND: now also U11.1 (GND), U11.10 (GND_RF), U11.12 (GND_RF), C31.2, FL1.2 (GND), FL1.3 (GND), FL1.5 (GND)
- net GNSS_ANT: now also AE1.1 (A)
- net VCC_RF: now also C29.1, U10.2 (VCC), U11.14 (VCC_RF), C31.1
- net at U10.3 (AO): now also FL1.1 (INPUT)
- net at C30.1: now also FL1.4 (OUTPUT)
- net RF_IN: now reaches U11.11 (RF_IN)
- net RF_IN: now also C30.2
- net GNSS_RST: now reaches U11.9 (SYS_RSTn)
- net RX_GNSS renamed GNSS_RX
- net TX_GNSS renamed GNSS_TX
- no-connect marks 7 -> 2
Other:
- note added: "ANTENNA"
- note added: "GNSS MODULE"
- note added: "RF AMPLIFIER + SAW FL"
- note added: "checked pinout and size"
- moved on the sheet: C28, C29, C30, C32, C33, JP5, JP6, JP7, JP8, L4, L5, R41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

Commit message: GNSS layout
Parts:
- removed AE1: Antenna, gps-compass_brd:ANT2525B00DT1516S, symbol Device:Antenna
- removed C28, C30: 120pF, Capacitor_SMD:C_0402_1005Metric, symbol Device:C_Small
- removed C29: 1nF, Capacitor_SMD:C_0402_1005Metric, symbol Device:C_Small
- removed C31, C32: 56nF, Capacitor_SMD:C_0402_1005Metric, symbol Device:C_Small
- removed C33: 10nF, Capacitor_SMD:C_0402_1005Metric, symbol Device:C_Small
- removed FL1: B39162B4327P810, gps-compass_brd:FIL_B39162B4327P810, symbol gps-compass_sch:B39162B4327P810
- removed JP5, JP6, JP7, JP8: Jumper_2_Small_Open, Jumper:SolderJumper-2_P1.3mm_Open_RoundedPad1.0x1.5mm, symbol Jumper:Jumper_2_Small_Open
- removed L4: 5.6nH, Inductor_SMD:L_0402_1005Metric, symbol Device:L_Small
- removed L5: 27nH, Inductor_SMD:L_0402_1005Metric, symbol Device:L_Small
- removed R41: 10k, Resistor_SMD:R_0805_2012Metric, symbol Device:R_Small
- removed U10: BGA725L6E6327FTSA1, gps-compass_brd:AMP_BGA725L6E6327FTSA1, symbol gps-compass_sch:BGA725L6E6327FTSA1
- removed U11: TESEO-LIV3R, gps-compass_brd:ARRAY_LIV3R_STM, symbol gps-compass_sch:TESEO-LIV3R
Connections:
- no-connect marks 2 -> 0
Other:
- note removed: "ANTENNA"
- note removed: "GNSS MODULE"
- note removed: "RF AMPLIFIER + SAW FL"
- note removed: "checked pinout and size"
Changed lines of the file:
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@@
 	(generator_version "9.0")
 	(paper "A4")
+)
