File: GPS-Compass/MCU.kicad_sch (KiCad schematic)
At the start: 13 parts, among them J2 USB_TypeC, U1 USBLC6-2SC6, U3 ESP32-S3-WROOM-1

Commit message: Schematic update
Parts:
- removed C1, C19: 100nF, Capacitor_SMD:C_0805_2012Metric_Pad1.18x1.45mm_HandSolder, symbol Device:C
- removed F1: Polyfuse/50R, Fuse:Fuse_0805_2012Metric, symbol Device:Polyfuse
- removed J2: USB_TypeC, sumec_brd:HRO_TYPE-C-31-M-12, symbol sumec_sch_lib:USB_TypeC
- removed R14, R3: 15R, Resistor_SMD:R_0805_2012Metric_Pad1.20x1.40mm_HandSolder, symbol Device:R
- removed R2: 100k, Resistor_SMD:R_0805_2012Metric_Pad1.20x1.40mm_HandSolder, symbol Device:R
- removed U1: USBLC6-2SC6, Package_TO_SOT_SMD:TSOT-23-6_HandSoldering, symbol sumec_library:USBLC6-2SC6
- renumbered C22 to C1, C23 to C2, R12 to R1, R13 to R2, U3 to U1
Connections:
- net SCL: now also U1.35 (IO42); no longer U1.34 (IO41)
- net SDA: now also U1.34 (IO41); no longer U1.35 (IO42)
- net ACC_INT: no longer names the net of U1.32 (IO39)
- net BTN_IO04: no longer names the net of U1.4 (IO4)
- net BTN_IO05: no longer names the net of U1.5 (IO5)
- net BZ_IO02: no longer names the net of U1.38 (IO2)
- net EN_L: no longer names the net of U1.7 (IO7)
- net EN_R: no longer names the net of U1.12 (IO8)
- net GYR_INT: no longer names the net of U1.33 (IO40)
- net IR_MODULE: no longer names the net of U1.30 (IO37)
- net LED_IO01: no longer names the net of U1.39 (IO1)
- net LED_IO36: no longer names the net of U1.29 (IO36)
- net LED_IO43: no longer names the net of U1.37 (IO43)
- net LED_IO44: no longer names the net of U1.36 (IO44)
- net PH_L: no longer names the net of U1.6 (IO6)
- net PH_R: no longer names the net of U1.11 (IO18)
- net POL_L: no longer names the net of U1.28 (IO35)
- net POL_M: no longer names the net of U1.19 (IO11)
- net POL_R: no longer names the net of U1.20 (IO12)
- net QRE_BACK: no longer names the net of U1.9 (IO16)
- net QRE_L: no longer names the net of U1.22 (IO14)
- net QRE_R: no longer names the net of U1.21 (IO13)
- net SHARP_L: no longer names the net of U1.31 (IO38)
- net SHARP_R: no longer names the net of U1.18 (IO10)
- net VOLTAGE_ALERT: no longer names the net of U1.17 (IO9)
- no-connect marks 10 -> 6
Other:
- note added: "ESP32-S3-WROOM1"
- note removed: "ESD PROTECTION"
- note removed: "ESP32-S3-WROOM1-N4"
- note removed: "GPIO USB 20 D+ (green) 19 D- (white) GND GND (black) VBUS +5V (red)"
- note removed: "USB"
- note removed: "USB CONNECTOR"
- note removed: "USB Type-C Connector Data transfer USB connector connected to ESP32 using CDC method"
- moved on the sheet: C1, C2, R1, R2, U1

Commit message: gps upd
Parts:
- R1, R2: footprint Resistor_SMD:R_0805_2012Metric_Pad1.20x1.40mm_HandSolder -> Resistor_SMD:R_0805_2012Metric
Changed lines of the file:
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@@
 		)
 	)
-	(global_label "SDA"
-		(shape bidirectional)
-		(at 215.9 110.49 0)
+	(global_label "GNSS_WKP"
+		(shape input)
+		(at 144.78 118.11 180)
 		(fields_autoplaced yes)
 		(effects
@@
 				(color 0 0 0 1)
 			)
-			(justify left)
+			(justify right)
 		)
 		(property "Intersheetrefs" "${INTERSHEET_REFS}"
-			(at 221.5812 110.49 0)
-			(effects
-				(font
-					(size 1.27 1.27)
-				)
-				(justify left)
-				(hide yes)
-			)
-		)
-	)
-	(global_label "M1"
-		(shape input)
-		(at 152.4 129.54 180)
+			(at 135.4533 118.11 0)
+			(effects
+				(font
+					(size 1.27 1.27)
+				)
+				(justify right)
+				(hide yes)
+			)
+		)
+	)
+	(global_label "SDA"
+		(shape bidirectional)
+		(at 215.9 110.49 0)
 		(fields_autoplaced yes)
 		(effects
@@
 				(color 0 0 0 1)
 			)
-			(justify right)
+			(justify left)
 		)
 		(property "Intersheetrefs" "${INTERSHEET_REFS}"
-			(at 148.3626 129.54 0)
-			(effects
-				(font
-					(size 1.27 1.27)
-				)
-				(justify right)
-				(hide yes)
-			)
-		)
-	)
-	(global_label "MOSI"
+			(at 221.5812 110.49 0)
+			(effects
+				(font
+					(size 1.27 1.27)
+				)
+				(justify left)
+				(hide yes)
+			)
+		)
+	)
+	(global_label "M1"
 		(shape input)
-		(at 144.78 133.35 180)
+		(at 152.4 129.54 180)
 		(fields_autoplaced yes)
 		(effects
@@
 		)
 		(property "Intersheetrefs" "${INTERSHEET_REFS}"
-			(at 139.4052 133.35 0)
+			(at 148.3626 129.54 0)
 			(effects
 				(font
@@
 		)
 	)
-	(global_label "STEP"
+	(global_label "MOSI"
 		(shape input)
-		(at 152.4 121.92 180)
+		(at 144.78 133.35 180)
 		(fields_autoplaced yes)
 		(effects
@@
 		)
 		(property "Intersheetrefs" "${INTERSHEET_REFS}"
-			(at 146.9548 121.92 0)
+			(at 139.4052 133.35 0)
 			(effects
 				(font
@@
 		)
 	)
-	(global_label "~{CS}"
+	(global_label "STEP"
 		(shape input)
-		(at 144.78 128.27 180)
+		(at 152.4 121.92 180)
 		(fields_autoplaced yes)
 		(effects
@@
 		)
 		(property "Intersheetrefs" "${INTERSHEET_REFS}"
-			(at 140.9048 128.27 0)
+			(at 146.9548 121.92 0)
 			(effects
 				(font
@@
 		)
 	)
-	(global_label "SCL"
-		(shape bidirectional)
-		(at 223.52 113.03 0)
+	(global_label "~{CS}"
+		(shape input)
+		(at 144.78 128.27 180)
 		(fields_autoplaced yes)
 		(effects
@@
 				(color 0 0 0 1)
 			)
+			(justify right)
+		)
+		(property "Intersheetrefs" "${INTERSHEET_REFS}"
+			(at 140.9048 128.27 0)
+			(effects
+				(font
+					(size 1.27 1.27)
+				)
+				(justify right)
+				(hide yes)
+			)
+		)
+	)
+	(global_label "SCL"
+		(shape bidirectional)
+		(at 223.52 113.03 0)
+		(fields_autoplaced yes)
+		(effects
+			(font
+				(face "Bahnschrift")
+				(size 1 1)
+				(color 0 0 0 1)
+			)
 			(justify left)
 		)
 		(property "Intersheetrefs" "${INTERSHEET_REFS}"
 			(at 229.0586 113.03 0)
+			(effects
+				(font
+					(size 1.27 1.27)
+				)
+				(justify left)
+				(hide yes)
+			)
+		)
+	)
+	(global_label "SNS_MCU"
+		(shape input)
+		(at 153.67 113.03 0)
+		(fields_autoplaced yes)
+		(effects
+			(font
+				(face "Bahnschrift")
+				(size 1 1)
+				(color 0 0 0 1)
+			)
+			(justify left)
+		)
+		(property "Intersheetrefs" "${INTERSHEET_REFS}"
+			(at 161.9904 113.03 0)
 			(effects
 				(font
@@
 			)
 		)
-		(property "Footprint" "Resistor_SMD:R_0805_2012Metric_Pad1.20x1.40mm_HandSolder"
+		(property "Footprint" "Resistor_SMD:R_0805_2012Metric"
 			(at 216.408 105.41 90)
 			(effects
@@
 			)
 		)
-		(property "Footprint" "Resistor_SMD:R_0805_2012Metric_Pad1.20x1.40mm_HandSolder"
+		(property "Footprint" "Resistor_SMD:R_0805_2012Metric"
 			(at 224.028 105.41 90)
 			(effects

Commit message: GNSS layout
Parts:
- removed C1: 10uF, Capacitor_Tantalum_SMD:CP_EIA-3216-18_Kemet-A_Pad1.58x1.35mm_HandSolder, symbol Device:C_Polarized
- removed C2: 100nF, Capacitor_SMD:C_0805_2012Metric_Pad1.18x1.45mm_HandSolder, symbol Device:C
- added C19: 10uF, Capacitor_SMD:C_0805_2012Metric, symbol Device:C_Small
- added C28: 100nF, Capacitor_SMD:C_0805_2012Metric, symbol Device:C_Small
- added J5: Conn_01x08_Pin, symbol Connector:Conn_01x08_Pin
Connections:
- net +3V3: now also C19.1, C28.1
- net GND: now also C19.2, C28.2
