File: GPS-Compass/POWER.kicad_sch (KiCad schematic)
At the start: 14 parts, among them IC1 TPS565242DRLR, Q1 Q_PMOS

Commit message: Schematic update
Parts:
- removed R1: 10k, Resistor_SMD:R_0805_2012Metric_Pad1.20x1.40mm_HandSolder, symbol Device:R
- added BT1: 2xLi-Ion_cells, gps-compass_brd:18650_2S_Holder, symbol gps-compass_sch:2xLi-Ion_cells
- added C10, C13: 10uF, symbol Device:C_Polarized_Small
- added C12: 44uF, symbol Device:C_Polarized_Small
- added C15, C17: 22uF, Capacitor_Tantalum_SMD:CP_EIA-2012-12_Kemet-R_Pad1.30x1.05mm_HandSolder, symbol Device:C_Polarized
- added C3: 10uF, Capacitor_Tantalum_SMD:CP_EIA-3216-18_Kemet-A_Pad1.58x1.35mm_HandSolder, symbol Device:C_Polarized
- added C4: 1uF, symbol Device:C_Polarized_Small
- added C7: 100nF, Capacitor_SMD:C_0805_2012Metric_Pad1.18x1.45mm_HandSolder, symbol Device:C_Small
- added C8: 47nF, symbol Device:C_Small
- added C9: 4.7uF, symbol Device:C_Polarized_Small
- added JP1: Jumper, symbol Jumper:Jumper_2_Small_Open
- added JP2: Jumper, Jumper:SolderJumper-3_P1.3mm_Open_RoundedPad1.0x1.5mm_NumberLabels, symbol Jumper:SolderJumper_3_Open
- added L2: 3.3uH, Inductor_SMD:L_Vishay_IHLP-1616, symbol Device:L
- added L3: 1uH, symbol Device:L_Small
- added Q2: Q_PMOS, Package_TO_SOT_SMD:SOT-23-3, symbol Device:Q_PMOS_GSD
- added R10: 9.5R, symbol Device:R_Small
- added R11, R5: 52.3k, Resistor_SMD:R_0805_2012Metric_Pad1.20x1.40mm_HandSolder, symbol Device:R_Small
- added R12: 10k, Resistor_SMD:R_0805_2012Metric_Pad1.20x1.40mm_HandSolder, symbol Device:R_Small
- added R13, R14, R15, R16: 10k, Resistor_SMD:R_0805_2012Metric_Pad1.20x1.40mm_HandSolder, symbol Device:R
- added R4: 100k, Resistor_SMD:R_0805_2012Metric_Pad1.20x1.40mm_HandSolder, symbol Device:R_Small
- added R6: 10k, symbol Device:R_Small
- added R7: 383R, symbol Device:R_Small
- added R9: 300R, symbol Device:R_Small
- added SW1: SW_DPDT_x2, sumec_brd:Custom_SPDT_2.5_Switch, symbol Switch:SW_DPDT_x2
- added TH1: 10k NTC, symbol Device:Thermistor_NTC
- added U2: AP62300Z6, Package_TO_SOT_SMD:SOT-563, symbol Regulator_Switching:AP62300Z6
- added U3: BQ25887, Package_DFN_QFN:VQFN-24-1EP_4x4mm_P0.5mm_EP2.5x2.5mm, symbol Battery_Management:BQ25887
- renumbered C7 to C11, C8 to C14, C10 to C16, C12 to C18, C4 to C5, C5 to C6, R5 to R3
Connections:
- net +3V3: now also R6.1
- net GND: now also BT1.4 (NEG), C10.2, C12.2, C13.2, C15.2, C17.2, C3.2, C4.2, C9.2, R12.2, R14.1, R15.2, R5.2, R7.2, SW1.2 (B), TH1.2, U2.3 (GND), U3.19 (GND), U3.20 (GND), U3.3 (CD)
- net VBUS 5V: now also JP1.1 (A); no longer Q1.1 (G)
- new net: R7.1, U3.8 (ILIM)
- new net: JP1.2 (B), Q1.1 (G), R15.1
- new net: R10.2, U3.10 (CBSET)
- new net: C8.2, U3.12 (BTST)
- new net: C12.1, U3.15 (SNS), U3.16 (SNS)
- new net: C13.1, L3.1, U3.21 (PMID), U3.22 (PMID)
- new net: R9.2, U3.9 (MID)
- new net: C7.2, U2.4 (BST)
- new net: R4.2, R5.1, U2.5 (EN)
- new net +8V: C3.1, Q2.3 (D), R4.1, U2.1 (VIN)
- new net BMID: R10.1, R9.1
- new net FB_5V: R11.2, R12.1, U2.6 (FB)
- new net FET_SW: Q2.1 (G), R16.2, SW1.1 (A)
- new net LDO: C9.1, R13.2, U3.11 (REGN)
- new net PSEL: R6.2, U3.24 (PSEL)
- new net SCL: U3.5 (SCL)
- new net SDA: U3.4 (SDA)
- new net STAT: U3.2 (STAT)
- new net SW: C7.1, C8.1, L2.1, L3.2, U2.2 (SW), U3.17 (SW), U3.18 (SW)
- new net TS: R13.1, R14.2, TH1.1, U3.7 (TS)
- new net USB_VBUS: C4.1, U3.23 (VBUS)
- new net VBATT: BT1.1 (POS), C10.1, Q2.2 (S), R16.1, U3.13 (BAT), U3.14 (BAT)
- new net VBATT_MID: JP2.2 (C)
- new net VBATT_NEG: BT1.2 (NEG), JP2.1 (A)
- new net VBATT_POS: BT1.3 (POS), JP2.3 (B)
- new net VOUT_5V: C15.1, C17.1, L2.2, R11.1
- new net ~{INT}: U3.6 (~{INT})
- new net ~{PG}: U3.1 (~{PG})
- no-connect marks 0 -> 1
Other:
- note added: "AP62301Z6-7 Step down converter Input: 4.2-18V Output: 5V Current output: 3A Switching freq.: 750kHz Inductor Inductance: 3.3uH Max. current: 2.7A"
- note added: "BATTERY"
- note added: "MAIN SWITCH"
- note added: "STEPDOWN CONVERTER 5V"
- note added: "charging status"
- note added: "good input source signalisation"
- note added: "link - library for the BMS"
- note added: "status and report"
- moved on the sheet: C11, C14, C16, C18, C5, C6, IC1, L1, Q1, R3, R8

Commit message: gps upd
Parts:
- removed C9: 4.7uF, symbol Device:C_Polarized_Small
- added C15: 4.7uF, Capacitor_SMD:C_0805_2012Metric, symbol Device:C_Small
- added JP3: Jumper, Jumper:SolderJumper-2_P1.3mm_Open_RoundedPad1.0x1.5mm, symbol Jumper:Jumper_2_Small_Open
- C10: renamed from C17; footprint Capacitor_Tantalum_SMD:CP_EIA-2012-12_Kemet-R_Pad1.30x1.05mm_HandSolder -> Capacitor_SMD:C_0805_2012Metric
- C11: renamed from C16; footprint Capacitor_Tantalum_SMD:CP_EIA-2012-12_Kemet-R_Pad1.30x1.05mm_HandSolder -> Capacitor_SMD:C_0805_2012Metric
- C12: renamed from C18; footprint Capacitor_SMD:C_0805_2012Metric_Pad1.18x1.45mm_HandSolder -> Capacitor_SMD:C_0805_2012Metric
- C13: renamed from C4; footprint (none) -> Capacitor_Tantalum_SMD:CP_EIA-3216-18_Kemet-A_Pad1.58x1.35mm_HandSolder
- C14: renamed from C8; footprint (none) -> Capacitor_SMD:C_0805_2012Metric
- C16: renamed from C10; footprint (none) -> Capacitor_Tantalum_SMD:CP_EIA-3216-18_Kemet-A_Pad1.58x1.35mm_HandSolder
- C17: renamed from C12; footprint (none) -> Capacitor_SMD:C_0805_2012Metric
- C18: renamed from C13; footprint (none) -> Capacitor_Tantalum_SMD:CP_EIA-3216-18_Kemet-A_Pad1.58x1.35mm_HandSolder
- C4: renamed from C5; footprint Capacitor_Tantalum_SMD:CP_EIA-2012-12_Kemet-R_Pad1.30x1.05mm_HandSolder -> Capacitor_SMD:C_0805_2012Metric
- C5: renamed from C7; footprint Capacitor_SMD:C_0805_2012Metric_Pad1.18x1.45mm_HandSolder -> Capacitor_SMD:C_0805_2012Metric
- C6: footprint Capacitor_SMD:C_0805_2012Metric_Pad1.18x1.45mm_HandSolder -> Capacitor_SMD:C_0805_2012Metric
- C7: renamed from C11; footprint Capacitor_Tantalum_SMD:CP_EIA-2012-12_Kemet-R_Pad1.30x1.05mm_HandSolder -> Capacitor_SMD:C_0805_2012Metric
- C8: renamed from C15; footprint Capacitor_Tantalum_SMD:CP_EIA-2012-12_Kemet-R_Pad1.30x1.05mm_HandSolder -> Capacitor_SMD:C_0805_2012Metric
- C9: renamed from C14; footprint Capacitor_Tantalum_SMD:CP_EIA-2012-12_Kemet-R_Pad1.30x1.05mm_HandSolder -> Capacitor_SMD:C_0805_2012Metric
- D1, D2: footprint Diode_SMD:D_1206_3216Metric_Pad1.42x1.75mm_HandSolder -> Diode_SMD:D_1206_3216Metric
- JP2: renamed from JP1; footprint (none) -> Jumper:SolderJumper-2_P1.3mm_Open_RoundedPad1.0x1.5mm
- L3: footprint (none) -> Inductor_SMD:L_Walsin_WLFM201609x
- R10: renamed from R6; footprint (none) -> Resistor_SMD:R_0805_2012Metric
- R11: renamed from R7; footprint (none) -> Resistor_SMD:R_0805_2012Metric
- R12: renamed from R9; footprint (none) -> Resistor_SMD:R_0805_2012Metric
- R13: renamed from R10; footprint (none) -> Resistor_SMD:R_0805_2012Metric
- R14: renamed from R15; footprint Resistor_SMD:R_0805_2012Metric_Pad1.20x1.40mm_HandSolder -> Resistor_SMD:R_0805_2012Metric
- R15: renamed from R13; value 10k -> 5.23k; footprint Resistor_SMD:R_0805_2012Metric_Pad1.20x1.40mm_HandSolder -> Resistor_SMD:R_0805_2012Metric
- R16: renamed from R14; value 10k -> 30.1k; footprint Resistor_SMD:R_0805_2012Metric_Pad1.20x1.40mm_HandSolder -> Resistor_SMD:R_0805_2012Metric
- R3, R4, R5: footprint Resistor_SMD:R_0805_2012Metric_Pad1.20x1.40mm_HandSolder -> Resistor_SMD:R_0805_2012Metric
- R6: renamed from R8; footprint Resistor_SMD:R_0805_2012Metric_Pad1.20x1.40mm_HandSolder -> Resistor_SMD:R_0805_2012Metric
- R7: renamed from R16; footprint Resistor_SMD:R_0805_2012Metric_Pad1.20x1.40mm_HandSolder -> Resistor_SMD:R_0805_2012Metric
- R8: renamed from R11; footprint Resistor_SMD:R_0805_2012Metric_Pad1.20x1.40mm_HandSolder -> Resistor_SMD:R_0805_2012Metric
- R9: renamed from R12; footprint Resistor_SMD:R_0805_2012Metric_Pad1.20x1.40mm_HandSolder -> Resistor_SMD:R_0805_2012Metric
- TH1: footprint (none) -> Resistor_SMD:R_0402_1005Metric
- renumbered JP2 to JP1, Q2 to Q1, Q1 to Q2
Connections:
- net VBATT_MID is gone; now on net BMID: JP1.2 (C)
- net GND: now also C15.2
- net LDO: now also C15.1
- net SNS: now reaches C17.1, U3.15 (SNS), U3.16 (SNS)
- net SNS: now also JP3.1 (A)
- new net SNS_MCU: JP3.2 (B)
Other:
- note added: "CHARGER + BMS"
- note removed: "charging status"
- note removed: "good input source signalisation"
- note removed: "status and report"
- moved on the sheet: BT1, C10, C11, C12, C13, C14, C16, C17, C18, C3, C4, C5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

Commit message: GNSS layout
Parts:
- removed C10, C11, C4, C7, C8, C9: 22uF, Capacitor_SMD:C_0805_2012Metric, symbol Device:C_Polarized
- removed C12, C6: 100nF, Capacitor_SMD:C_0805_2012Metric, symbol Device:C
- removed C13: 1uF, Capacitor_Tantalum_SMD:CP_EIA-3216-18_Kemet-A_Pad1.58x1.35mm_HandSolder, symbol Device:C_Polarized_Small
- removed C16, C18: 10uF, Capacitor_Tantalum_SMD:CP_EIA-3216-18_Kemet-A_Pad1.58x1.35mm_HandSolder, symbol Device:C_Polarized_Small
- removed C17: 44uF, Capacitor_SMD:C_0805_2012Metric, symbol Device:C_Polarized_Small
- removed C3: 10uF, Capacitor_Tantalum_SMD:CP_EIA-3216-18_Kemet-A_Pad1.58x1.35mm_HandSolder, symbol Device:C_Polarized
- added C11, C12, C18, C8: 22uF, Capacitor_SMD:C_0805_2012Metric, symbol Device:C_Small
- added C13: 1uF, Capacitor_SMD:C_0805_2012Metric, symbol Device:C_Small
- added C16, C17, C3, C4: 10uF, Capacitor_SMD:C_0805_2012Metric, symbol Device:C_Small
- added C22, C6, C7, C9: 100nF, Capacitor_SMD:C_0805_2012Metric, symbol Device:C_Small
- added C23: 44uF, Capacitor_SMD:C_0805_2012Metric, symbol Device:C_Small
Connections:
- net VBUS 5V is gone; now on net USB_VBUS: D2.2 (A), JP2.1 (A)
- net VOUT 5V is gone; now on net VOUT_5V: Q2.2 (S)
- net +3V3: now also C11.1, C12.1, C7.1
- net +5V: now also C4.1, C9.1
- net +8V: now also C3.1, C6.1
- net GND: now also C11.2, C12.2, C13.2, C16.2, C17.2, C18.2, C22.2, C23.2, C3.2, C4.2, C6.2, C7.2, C8.2, C9.2
- net SNS: now also C23.1
- net SW: no longer C14.1, L3.2, U3.17 (SW), U3.18 (SW)
- net USB_VBUS: now also C13.1
- net VBATT: now also C17.1
- net VOUT_5V: now also C18.1, C8.1
- net at L3.1, U3.21 (PMID), U3.22 (PMID): now also C16.1, C22.1
- new net SWC: C14.1, L3.2, U3.17 (SW), U3.18 (SW)
Other:
- moved on the sheet: IC1, JP3, L1, L2, L3, R15, R16, R3, R4, R5, R6, R8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
