File: GPS-Compass/GPS-Compass.kicad_pcb (KiCad board)
At the start: 2 copper layers, 95 parts, among them IC1 TPS565242DRLR, J1 USB_TypeC, Q1 Q_PMOS, Q2 Q_PMOS, SW1 SW_DPDT_x2, SW2 SW_Push, SW3 SW_Push, SW4 SW_Push, SW5 SW_Push, U1 ESP32-S3-WROOM-1, U10 TESEO-LIV3R, U2 AP62300Z6, U3 BQ25887, U5 OPS-S3911LE-GW, U6 OPS-S3911LE-GW, U7 OPS-S3911LE-GW, U8 MAX7219, U9 USBLC6-2SC6

Commit message: gps upd
Parts:
- removed C34: 10n, Capacitor_SMD:C_0402_1005Metric
- removed TP1: TestPoint, sumec_graphic:SPS_LOGO_IMG
- removed TP2: TestPoint, sumec_graphic:SCHRACK_LOGO_IMG
- removed TP3: TestPoint, sumec_graphic:BRAND_BERSERK
- removed TP4: TestPoint, sumec_graphic:BOCCHI_IMG
- added AE1: Antenna, gps-compass_brd:ANT2525B00DT1516S, F.Cu at (636.8, 172.8)
- added BZ1: Buzzer, gps-compass_brd:CEM-1203_Buzzer, F.Cu at (531.3, 49.4)
- added C10: 22uF, Capacitor_SMD:C_0805_2012Metric, F.Cu at (463.0, -3.53)
- added C12: 100nF, Capacitor_SMD:C_0805_2012Metric, F.Cu at (467.5, -9.55)
- added C13: 1uF, Capacitor_Tantalum_SMD:CP_EIA-3216-18_Kemet-A_Pad1.58x1.35mm_HandSolder, F.Cu at (478.0, -6.33)
- added C19: 10uF, Capacitor_Tantalum_SMD:CP_EIA-3216-18_Kemet-A_Pad1.58x1.35mm_HandSolder, F.Cu at (455.7, 58.5)
- added C20: 10nF, Capacitor_SMD:C_0402_1005Metric, F.Cu at (455.3, 51.4)
- added C21: 100nF, Capacitor_SMD:C_0805_2012Metric, F.Cu at (456.1, 48.9)
- added C28: 120pF, Capacitor_SMD:C_0402_1005Metric, F.Cu at (474.7, 20.9)
- added C30: 120pF, Capacitor_SMD:C_0402_1005Metric, F.Cu at (474.7, 24.8)
- added C4: 22uF, Capacitor_SMD:C_0805_2012Metric, F.Cu at (458.6, -9.55)
- added C8: 22uF, Capacitor_SMD:C_0805_2012Metric, F.Cu at (463.0, -9.55)
- added C9: 22uF, Capacitor_SMD:C_0805_2012Metric, F.Cu at (463.0, -6.54)
- added D3: LED, LED_SMD:LED_0805_2012Metric, F.Cu at (522.1, 44.3)
- added D4: LED, LED_SMD:LED_0805_2012Metric, F.Cu at (522.1, 47.3)
- added D5: LED, LED_SMD:LED_0805_2012Metric, F.Cu at (522.1, 50.4)
- added D6: BLUE, LED_SMD:LED_0805_2012Metric, F.Cu at (522.1, 53.4)
- added D7: LED, LED_SMD:LED_0805_2012Metric, F.Cu at (522.1, 56.4)
- added D8: LED, LED_SMD:LED_0805_2012Metric, F.Cu at (522.1, 59.5)
- added D9: LED, LED_SMD:LED_0805_2012Metric, F.Cu at (522.1, 62.5)
- added J2: USB_TypeC, sumec_brd:HRO_TYPE-C-31-M-12, F.Cu at (329.5, 125.5)
- added J3: Conn_01x02_Pin, Connector_JST:JST_XH_B2B-XH-A_1x02_P2.50mm_Vertical, F.Cu at (504.4, 9.07)
- added J4: Conn_01x02_Pin, Connector_JST:JST_XH_B2B-XH-A_1x02_P2.50mm_Vertical, F.Cu at (504.4, 16.9)
- added JP1: Jumper, Jumper:SolderJumper-3_P1.3mm_Open_RoundedPad1.0x1.5mm_NumberLabels, F.Cu at (508.1, -4.63)
- added JP3: Jumper, Jumper:SolderJumper-2_P1.3mm_Open_RoundedPad1.0x1.5mm, F.Cu at (488.3, -0.08)
- added JP4: Jumper, Jumper:SolderJumper-3_P1.3mm_Open_RoundedPad1.0x1.5mm_NumberLabels, F.Cu at (455.5, 55.1)
- added JP5: Jumper_2_Small_Open, Jumper:SolderJumper-2_P1.3mm_Open_RoundedPad1.0x1.5mm, F.Cu at (475.5, 7.47)
- added JP6: Jumper_2_Small_Open, Jumper:SolderJumper-2_P1.3mm_Open_RoundedPad1.0x1.5mm, F.Cu at (475.5, 11.0)
- added JP7: Jumper_2_Small_Open, Jumper:SolderJumper-2_P1.3mm_Open_RoundedPad1.0x1.5mm, F.Cu at (475.5, 14.6)
- added JP8: Jumper_2_Small_Open, Jumper:SolderJumper-2_P1.3mm_Open_RoundedPad1.0x1.5mm, F.Cu at (475.5, 18.1)
- added L3: 1uH, Inductor_SMD:L_Walsin_WLFM201609x, F.Cu at (507.8, -1.24)
- added L4: 5.6nH, Inductor_SMD:L_0402_1005Metric, F.Cu at (456.9, 37.6)
- added Q3: Q_NMOS_GSD, Package_TO_SOT_SMD:SOT-23-3, F.Cu at (450.1, 55.8)
- added Q4: BC337, Package_TO_SOT_THT:TO-92_Inline, F.Cu at (539.6, 59.3)
- added R10: 10k, Resistor_SMD:R_0805_2012Metric, F.Cu at (449.7, -3.68)
- added R17: R(SET), Resistor_SMD:R_0805_2012Metric, F.Cu at (445.3, 48.9)
- added R18: R(SET), Resistor_SMD:R_0805_2012Metric, F.Cu at (445.3, 51.8)
- added R23: 100k, Resistor_SMD:R_0805_2012Metric, F.Cu at (498.7, 13.1)
- added R24: 10k, Resistor_SMD:R_0805_2012Metric, F.Cu at (498.7, 16.0)
- added R6: 10k, Resistor_SMD:R_0805_2012Metric, F.Cu at (445.3, -0.73)
- added R7: 10k, Resistor_SMD:R_0805_2012Metric, F.Cu at (445.3, 2.22)
- added R9: 10k, Resistor_SMD:R_0805_2012Metric, F.Cu at (449.7, -6.63)
- added SW6: SW_Push, sumec_brd:SW_SPST_EVQPE1, F.Cu at (492.1, 28.4)
- added TH1: 10k NTC, Resistor_SMD:R_0402_1005Metric, F.Cu at (506.8, 1.38)
- added U11: TESEO-LIV3R, gps-compass_brd:ARRAY_LIV3R_STM, F.Cu at (449.3, 39.5)
- added U4: DRV8834RGER, gps-compass_brd:DRIVER_DRV8834RGER, F.Cu at (450.9, 50.4)
- BT1: moved to B.Cu
- C11: footprint Capacitor_Tantalum_SMD:CP_EIA-2012-12_Kemet-R_Pad1.30x1.05mm_HandSolder -> Capacitor_SMD:C_0805_2012Metric
- C14: value 22uF -> 47nF; footprint Capacitor_Tantalum_SMD:CP_EIA-2012-12_Kemet-R_Pad1.30x1.05mm_HandSolder -> Capacitor_SMD:C_0805_2012Metric
- C15: value 22uF -> 4.7uF; footprint Capacitor_Tantalum_SMD:CP_EIA-2012-12_Kemet-R_Pad1.30x1.05mm_HandSolder -> Capacitor_SMD:C_0805_2012Metric
- C16: value 22uF -> 10uF; footprint Capacitor_Tantalum_SMD:CP_EIA-2012-12_Kemet-R_Pad1.30x1.05mm_HandSolder -> Capacitor_Tantalum_SMD:CP_EIA-3216-18_Kemet-A_Pad1.58x1.35mm_HandSolder
- C17: value 22uF -> 44uF; footprint Capacitor_Tantalum_SMD:CP_EIA-2012-12_Kemet-R_Pad1.30x1.05mm_HandSolder -> Capacitor_SMD:C_0805_2012Metric
- C18: value 100nF -> 10uF; footprint Capacitor_SMD:C_0805_2012Metric_Pad1.18x1.45mm_HandSolder -> Capacitor_Tantalum_SMD:CP_EIA-3216-18_Kemet-A_Pad1.58x1.35mm_HandSolder
- C23, C24, C25, C26, C27, C6: footprint Capacitor_SMD:C_0805_2012Metric_Pad1.18x1.45mm_HandSolder -> Capacitor_SMD:C_0805_2012Metric
- C29: value 56p -> 1nF
- C31, C32: value 56p -> 56nF
- C33: value 56p -> 10nF
- C5: value 22uF -> 100nF; footprint Capacitor_Tantalum_SMD:CP_EIA-2012-12_Kemet-R_Pad1.30x1.05mm_HandSolder -> Capacitor_SMD:C_0805_2012Metric
- C7: value 100nF -> 22uF; footprint Capacitor_SMD:C_0805_2012Metric_Pad1.18x1.45mm_HandSolder -> Capacitor_SMD:C_0805_2012Metric
- D1, D2: footprint Diode_SMD:D_1206_3216Metric_Pad1.42x1.75mm_HandSolder -> Diode_SMD:D_1206_3216Metric
- FL1: value B39162B8813P810 -> B39162B4327P810; footprint Filter:Filter_1109-5_1.1x0.9mm -> gps-compass_brd:FIL_B39162B4327P810
- J1: value USB_TypeC -> RFShield_OnePiece; footprint sumec_brd:HRO_TYPE-C-31-M-12 -> RF_Shielding:Laird_Technologies_97-2003_12.70x13.37mm
- JP2: footprint Jumper:SolderJumper-3_P1.3mm_Open_RoundedPad1.0x1.5mm_NumberLabels -> Jumper:SolderJumper-2_P1.3mm_Open_RoundedPad1.0x1.5mm
- L5: value 27n -> 27nH
- R1, R14, R2, R20, R21, R22, R27, R3, R30, R4, R5: footprint Resistor_SMD:R_0805_2012Metric_Pad1.20x1.40mm_HandSolder -> Resistor_SMD:R_0805_2012Metric
- R11: value 52.3k -> 383R; footprint Resistor_SMD:R_0805_2012Metric_Pad1.20x1.40mm_HandSolder -> Resistor_SMD:R_0805_2012Metric
- R12: value 10k -> 300R; footprint Resistor_SMD:R_0805_2012Metric_Pad1.20x1.40mm_HandSolder -> Resistor_SMD:R_0805_2012Metric
- R13: value 10k -> 9.5R; footprint Resistor_SMD:R_0805_2012Metric_Pad1.20x1.40mm_HandSolder -> Resistor_SMD:R_0805_2012Metric
- R15: value 10k -> 5.23k; footprint Resistor_SMD:R_0805_2012Metric_Pad1.20x1.40mm_HandSolder -> Resistor_SMD:R_0805_2012Metric
- R16: value 10k -> 30.1k; footprint Resistor_SMD:R_0805_2012Metric_Pad1.20x1.40mm_HandSolder -> Resistor_SMD:R_0805_2012Metric
- R19: footprint Resistor_THT:R_Axial_DIN0207_L6.3mm_D2.5mm_P10.16mm_Horizontal -> Resistor_SMD:R_0805_2012Metric
- R25: value 100k -> 10k; footprint Resistor_SMD:R_0805_2012Metric_Pad1.20x1.40mm_HandSolder -> Resistor_SMD:R_0805_2012Metric
- R26: value 15R -> 10k; footprint Resistor_SMD:R_0805_2012Metric_Pad1.20x1.40mm_HandSolder -> Resistor_SMD:R_0805_2012Metric
- R28: value 2.2k -> 15R; footprint Resistor_SMD:R_0805_2012Metric_Pad1.20x1.40mm_HandSolder -> Resistor_SMD:R_0805_2012Metric
- R29: value 2.2k -> 1k; footprint Resistor_SMD:R_0805_2012Metric_Pad1.20x1.40mm_HandSolder -> Resistor_SMD:R_0805_2012Metric
- R31, R32: value 10k -> 2.2k; footprint Resistor_SMD:R_0805_2012Metric_Pad1.20x1.40mm_HandSolder -> Resistor_SMD:R_0805_2012Metric
- R33: value 10k -> 1k; footprint Resistor_SMD:R_0805_2012Metric_Pad1.20x1.40mm_HandSolder -> Resistor_SMD:R_0805_2012Metric
- R34, R35, R36: value 220R -> 10k; footprint Resistor_SMD:R_0805_2012Metric_Pad1.20x1.40mm_HandSolder -> Resistor_SMD:R_0805_2012Metric
- R37, R38: value 10k -> 220R; footprint Resistor_SMD:R_0603_1608Metric -> Resistor_SMD:R_0805_2012Metric
- R39: value 22 -> 220R; footprint Resistor_SMD:R_0402_1005Metric -> Resistor_SMD:R_0805_2012Metric
- R40: value 22 -> 0R; footprint Resistor_SMD:R_0402_1005Metric -> Resistor_SMD:R_0805_2012Metric
- R41: footprint Resistor_SMD:R_0603_1608Metric -> Resistor_SMD:R_0805_2012Metric
- R8: value 10k -> 52.3k; footprint Resistor_SMD:R_0805_2012Metric_Pad1.20x1.40mm_HandSolder -> Resistor_SMD:R_0805_2012Metric
- U10: value TESEO-LIV3R -> BGA725L6E6327FTSA1; footprint gps-compass_brd:ARRAY_LIV3R_STM -> gps-compass_brd:AMP_BGA725L6E6327FTSA1
- moved BT1 516.4 mm to (611.3, 217.3), turned to 180 degrees
- moved C22 456.3 mm to (535.8, 25.3)
- moved C23 456.1 mm to (541.0, 25.2)
- moved R20 455.7 mm to (545.4, 25.2)
- moved C16 403.8 mm to (478.0, -3.18)
- moved D1 401.7 mm to (496.2, -9.36)
- moved D2 401.7 mm to (496.2, -5.97)
- moved IC1 399.8 mm to (501.2, -3.25)
- moved U2 399.8 mm to (501.2, -0.26)
- moved L1 399.2 mm to (508.2, -8.73)
- moved U3 399.2 mm to (502.2, -7.90)
- moved Q1 398.3 mm to (483.5, -8.65)
- moved Q2 398.3 mm to (483.5, -4.03)
- moved C24 397.7 mm to (515.7, 7.20)
- moved C25 397.7 mm to (515.7, 10.2)
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Connections:
- net Net-(U11-TX) renamed BZ_PWM
- C14 pad 1: +3V3 -> SW
- C14 pad 2: GND -> Net-(U3-BTST)
- C15 pad 1: VOUT_5V -> LDO
- C16 pad 1: +3V3 -> VBATT
- C17 pad 1: VOUT_5V -> SNS
- C18 pad 1: +3V3 -> Net-(C18-Pad1)
- C29 pad 1: TX_GNSS -> VCC_RF
- C31 pad 1: RX_GNSS -> VCC_RF
- C32 pad 1: VCC_RF -> Net-(U11-VBATT)
- C33 pad 1: VCC -> +3V3
- C5 pad 1: +5V -> SW
- C5 pad 2: GND -> Net-(U2-BST)
- C7 pad 1: SW -> +3V3
- C7 pad 2: Net-(U2-BST) -> GND
- FL1 pad 1: unconnected-(FL1-Pad1) -> Net-(FL1-INPUT)
- FL1 pad 2: Net-(FL1-Pad2) -> GND
- FL1 pad 3: unconnected-(FL1-Pad3) -> GND
- FL1 pad 4: unconnected-(FL1-Pad4) -> Net-(FL1-OUTPUT)
- FL1 pad 5: Net-(FL1-Pad2) -> GND
- JP2 pad 1: VBATT_NEG -> VBUS 5V
- JP2 pad 2: VBATT_MID -> Net-(JP2-B)
- L5 pad 1: VCC -> +3V3
- L5 pad 2: +3V3 -> Net-(U11-VBATT)
- Q1 pad 1: Net-(JP1-B) -> /POWER/FET_SW
- Q1 pad 2: VOUT 5V -> VBATT
- Q1 pad 3: Net-(D1-A) -> +8V
- Q2 pad 1: /POWER/FET_SW -> Net-(JP2-B)
- Q2 pad 2: VBATT -> VOUT 5V
- Q2 pad 3: +8V -> Net-(D1-A)
- R11 pad 1: VOUT_5V -> Net-(U3-ILIM)
- R11 pad 2: /POWER/FB_5V -> GND
- R12 pad 1: /POWER/FB_5V -> BMID
- R12 pad 2: GND -> Net-(U3-MID)
- R13 pad 1: TS -> BMID
- R13 pad 2: LDO -> Net-(U3-CBSET)
- R14 pad 1: GND -> Net-(JP2-B)
- R14 pad 2: TS -> GND
- R15 pad 1: Net-(JP1-B) -> TS
- R15 pad 2: GND -> LDO
- R16 pad 1: VBATT -> GND
- R16 pad 2: /POWER/FET_SW -> TS
- R25 pad 1: /MECHANICAL/SHLD -> +3V3
- R25 pad 2: GND -> BT_IOXY
- R26 pad 1: D+ IN -> +3V3
- R26 pad 2: Net-(R26-Pad2) -> GNSS_RST
- R27 pad 1: D- IN -> D+ IN
- R28 pad 1: +3V3 -> D- IN
- R28 pad 2: Net-(D3-A) (its old number) -> Net-(R28-Pad2)
- R29 pad 1: +3V3 -> Net-(Q4-B)
- R29 pad 2: Net-(D4-A) -> GNSS_PPS
- R31 pad 1: STAT -> +3V3
- R31 pad 2: +3V3 -> Net-(D4-A)
- R32 pad 1: ~{INT} -> +3V3
- R32 pad 2: +3V3 -> Net-(D5-A)
- R33 pad 1: ~{PG} -> Net-(D6-K)
- R33 pad 2: +3V3 -> Net-(Q4-C)
- R34 pad 1: unconnected-(R34-Pad1) -> STAT
- R34 pad 2: Net-(D6-A) -> +3V3
- R35 pad 1: unconnected-(R35-Pad1) -> ~{INT}
- R35 pad 2: Net-(D7-A) -> +3V3
- R36 pad 1: unconnected-(R36-Pad1) -> ~{PG}
- R36 pad 2: Net-(D8-A) -> +3V3
- R37 pad 1: Net-(U11-ANT_OFF) -> LED_IOXX
- R37 pad 2: GND -> Net-(D7-A)
- R38 pad 1: +3V3 -> LED_IOXX
- R38 pad 2: GPS_!RST -> Net-(D8-A)
- R39 pad 1: Net-(U11-RX) -> LED_IOXX
- R39 pad 2: UART_RX -> Net-(D9-A)
- R40 pad 2: UART_TX -> Net-(BZ1-+)
- R41 pad 1: +3V3 -> GND
- R41 pad 2: GPS_WAKEUP -> ANT_OFF
- R8 pad 1: FB -> VOUT_5V
- R8 pad 2: GND -> /POWER/FB_5V
- U10 pad 1: unconnected-(U10-GND-Pad1) -> GND
- U10 pad 2: Net-(JP3-B) -> VCC_RF
- U10 pad 3: Net-(JP4-B) -> Net-(FL1-INPUT)
- U10 pad 4: GNSS_PPS -> GND
- U10 pad 5: GNSS_WKP -> Net-(U10-AI)
- U10 pad 6: Net-(U10-VBATT) -> ANT_OFF
- U3 pad 15: Net-(C12-Pad1) -> SNS
- U3 pad 16: Net-(C12-Pad1) -> SNS
- U3 pad 21: Net-(C13-Pad1) -> Net-(C18-Pad1)
- U3 pad 22: Net-(C13-Pad1) -> Net-(C18-Pad1)
- U9 pad 1: Net-(R26-Pad2) -> Net-(R27-Pad2)
- U9 pad 3: Net-(R27-Pad2) -> Net-(R28-Pad2)
Other:
- board outline added: 452.9 x 130 mm

Commit message: pcb update
Parts:
- JP1: moved to B.Cu
- moved AE1 581.6 mm to (56.8, 129.8)
- moved C23 550.0 mm to (-5.88, 83.3)
- moved D3 550.0 mm to (-24.8, 102.4)
- moved D4 550.0 mm to (-24.8, 105.4)
- moved D5 550.0 mm to (-24.8, 108.4)
- moved D6 550.0 mm to (-24.8, 111.5)
- moved D7 550.0 mm to (-24.8, 114.5)
- moved D8 550.0 mm to (-24.8, 117.6)
- moved D9 550.0 mm to (-24.8, 120.6)
- moved R13 550.0 mm to (-92.7, 48.5)
- moved R14 550.0 mm to (-92.7, 51.5)
- moved R15 550.0 mm to (-92.7, 54.4)
- moved R16 550.0 mm to (-92.7, 57.4)
- moved BZ1 550.0 mm to (-15.6, 107.5)
- moved C1 550.0 mm to (-43.5, 99.2)
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Other:
- board size 452.9 x 130 mm -> 100 x 100 mm

Commit message: Finished PCB layout on edgecuts
Parts:
- removed C22: 10uF, Capacitor_Tantalum_SMD:CP_EIA-3216-18_Kemet-A_Pad1.58x1.35mm_HandSolder
- removed C23: 100nF, Capacitor_SMD:C_0805_2012Metric
- removed R20: 10k, Resistor_SMD:R_0805_2012Metric
- removed U5, U6, U7: OPS-S3911LE-GW, gps-compass_brd:OPS-S3911LE-GW
- removed U8: MAX7219, Package_SO:SOP-24_7.5x15.4mm_P1.27mm
- BT1, JP1: moved to F.Cu
- moved J2 311.9 mm to (17.7, 117.9), turned to 0 degrees
- moved J1 276.8 mm to (15.1, 137.1)
- moved H2 151.1 mm to (-5.75, 107.5), turned to 0 degrees
- moved H4 140.8 mm to (-5.75, 123.4)
- moved C1 97.8 mm to (54.3, 97.2)
- moved C2 97.8 mm to (53.7, 106.1)
- moved R1 97.8 mm to (53.5, 100.2)
- moved R2 97.8 mm to (53.5, 103.2)
- moved C19 97.0 mm to (2.88, 140.5)
- moved C20 97.0 mm to (2.42, 133.4)
- moved C21 97.0 mm to (3.21, 130.9)
- moved JP4 97.0 mm to (2.67, 137.1)
- moved R17 97.0 mm to (-7.51, 130.9)
- moved R18 97.0 mm to (-7.51, 133.8)
- moved R19 97.0 mm to (-7.51, 136.8)
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Other:
- board size 100 x 100 mm -> 102.5 x 100 mm

Commit message: GNSS layout
Parts:
- removed AE1: Antenna, gps-compass_brd:ANT2525B00DT1516S
- removed C1: 10uF, Capacitor_Tantalum_SMD:CP_EIA-3216-18_Kemet-A_Pad1.58x1.35mm_HandSolder
- removed C2: 100nF, Capacitor_SMD:C_0805_2012Metric_Pad1.18x1.45mm_HandSolder
- removed C29: 1nF, Capacitor_SMD:C_0402_1005Metric
- removed C30: 120pF, Capacitor_SMD:C_0402_1005Metric
- removed C31, C32: 56nF, Capacitor_SMD:C_0402_1005Metric
- removed C33: 10nF, Capacitor_SMD:C_0402_1005Metric
- removed D6: BLUE, LED_SMD:LED_0805_2012Metric
- removed FL1: B39162B4327P810, gps-compass_brd:FIL_B39162B4327P810
- removed JP5, JP6, JP7, JP8: Jumper_2_Small_Open, Jumper:SolderJumper-2_P1.3mm_Open_RoundedPad1.0x1.5mm
- removed L4: 5.6nH, Inductor_SMD:L_0402_1005Metric
- removed L5: 27nH, Inductor_SMD:L_0402_1005Metric
- removed Q4: BC337, Package_TO_SOT_THT:TO-92_Inline
- removed R29, R33: 1k, Resistor_SMD:R_0805_2012Metric
- removed R41: 10k, Resistor_SMD:R_0805_2012Metric
- removed U10: BGA725L6E6327FTSA1, gps-compass_brd:AMP_BGA725L6E6327FTSA1
- removed U11: TESEO-LIV3R, gps-compass_brd:ARRAY_LIV3R_STM
- added C22: 100nF, Capacitor_SMD:C_0805_2012Metric, F.Cu at (93.1, 82.1)
- added C23: 44uF, Capacitor_SMD:C_0805_2012Metric, F.Cu at (90.2, 78.1)
- BT1: moved to B.Cu
- C10, C4: value 22uF -> 10uF
- C12: value 100nF -> 22uF
- C13, C16, C19, C3: footprint Capacitor_Tantalum_SMD:CP_EIA-3216-18_Kemet-A_Pad1.58x1.35mm_HandSolder -> Capacitor_SMD:C_0805_2012Metric
- C17: value 44uF -> 10uF
- C18: value 10uF -> 22uF; footprint Capacitor_Tantalum_SMD:CP_EIA-3216-18_Kemet-A_Pad1.58x1.35mm_HandSolder -> Capacitor_SMD:C_0805_2012Metric
- C28: value 120pF -> 100nF; footprint Capacitor_SMD:C_0402_1005Metric -> Capacitor_SMD:C_0805_2012Metric
- C7, C9: value 22uF -> 100nF
- H1, H2: footprint MountingHole:MountingHole_3.2mm_M3_Pad_Via -> MountingHole:MountingHole_3.2mm_M3_Pad
- TP5, TP6, TP7, TP8, TP9: footprint TestPoint:TestPoint_Pad_1.0x1.0mm -> TestPoint:TestPoint_Pad_D1.0mm
- moved H3 187.3 mm to (168.3, 46.2), turned to 90 degrees
- moved R4 149.7 mm to (104.8, 99.5), turned to 180 degrees
- moved R5 149.6 mm to (104.8, 101.5)
- moved R8 142.5 mm to (101.1, 102.5)
- moved R9 141.8 mm to (101.1, 100.5), turned to 180 degrees
- moved R10 140.9 mm to (101.2, 82.4), turned to 180 degrees
- moved R11 138.6 mm to (98.1, 72.9), turned to 90 degrees
- moved R12 137.1 mm to (96.2, 72.9), turned to -90 degrees
- moved R16 135.9 mm to (100.3, 78.4), turned to 180 degrees
- moved R15 135.8 mm to (100.3, 76.5)
- moved C8 135.0 mm to (108.1, 92.8), turned to 90 degrees
- moved C6 135.0 mm to (103.8, 96.8), turned to -90 degrees
- moved C5 132.7 mm to (101.0, 98.5)
- moved JP1 129.9 mm to (147.2, 65.8)
- moved R13 129.7 mm to (94.3, 72.9), turned to -90 degrees
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Connections:
- C10 pad 1: VOUT_5V -> VM
- C14 pad 1: SW -> SWC
- C16 pad 1: VBATT -> Net-(C16-Pad1)
- C17 pad 1: SNS -> VBATT
- C18 pad 1: Net-(C18-Pad1) -> VOUT_5V
- C19 pad 1: VM -> +3V3
- C20 pad 1: VM -> Net-(U4-VCP)
- C20 pad 2: GND -> VM
- C28 pad 1: GNSS_ANT -> +3V3
- C28 pad 2: Net-(C28-Pad2) -> GND
- C5 pad 1: SW -> /POWER/SW
- C6 pad 1: +5V -> +8V
- C9 pad 1: +3V3 -> +5V
- D2 pad 2: VBUS 5V -> USB_VBUS
- JP2 pad 1: VBUS 5V -> USB_VBUS
- L2 pad 1: SW -> /POWER/SW
- L3 pad 1: Net-(C18-Pad1) -> Net-(C16-Pad1)
- L3 pad 2: SW -> SWC
- Q2 pad 2: VOUT 5V -> VOUT_5V
- R27 pad 1: D+ IN -> D- IN
- R28 pad 1: D- IN -> D+ IN
- U2 pad 2: SW -> /POWER/SW
- U3 pad 17: SW -> SWC
- U3 pad 18: SW -> SWC
- U3 pad 21: Net-(C18-Pad1) -> Net-(C16-Pad1)
- U3 pad 22: Net-(C18-Pad1) -> Net-(C16-Pad1)
- U4 pad 14: VM -> Net-(U4-VCP)
- U9 pad 4: D- -> D+
- U9 pad 6: D+ -> D-
Routing:
- net SWC: track 0.00 -> 8.49 mm
- net SNS: track 0.00 -> 7.26 mm
- net D- IN: track 0.00 -> 6.28 mm
- net VBATT: track 0.00 -> 5.77 mm
- net D+ IN: track 0.00 -> 4.76 mm
- net LDO: track 0.00 -> 4.51 mm
- net Net-(U3-ILIM): track 0.00 -> 4.47 mm
- net /POWER/SW: track 0.00 -> 4.14 mm
- net TS: track 0.00 -> 3.61 mm
- net Net-(U3-MID): track 0.00 -> 3.43 mm
- net Net-(U3-CBSET): track 0.00 -> 2.75 mm
- net Net-(R28-Pad2): track 0.00 -> 2.15 mm
- net Net-(R27-Pad2): track 0.00 -> 2.15 mm
- net VM: track 0.00 -> 2.09 mm
- net Net-(U2-BST): track 0.00 -> 1.78 mm
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Other:
- board size 102.5 x 100 mm -> 100 x 78.5 mm
- board text added: "MOTOR"

Commit message: GNSS and Mian ocb
Parts:
- added REF**: PinHeader_1x10_P2.54mm_Horizontal, Connector_PinHeader_2.54mm:PinHeader_1x10_P2.54mm_Horizontal, F.Cu at (105.5, 117.3)

Commit message: schematric remake
Parts:
- removed BZ1: Buzzer, gps-compass_brd:CEM-1203_Buzzer
- removed C19: 10uF, Capacitor_SMD:C_0805_2012Metric
- removed C24, C25, C28: 100nF, Capacitor_SMD:C_0805_2012Metric
- removed D1, D2: D_Schottky, Diode_SMD:D_1206_3216Metric
- removed D7, D8, D9: LED, LED_SMD:LED_0805_2012Metric
- removed J1: RFShield_OnePiece, RF_Shielding:Laird_Technologies_97-2003_12.70x13.37mm
- removed J3, J4: Conn_01x02_Pin, Connector_JST:JST_XH_B2B-XH-A_1x02_P2.50mm_Vertical
- removed JP2: Jumper, Jumper:SolderJumper-2_P1.3mm_Open_RoundedPad1.0x1.5mm
- removed Q1, Q2: Q_PMOS, Package_TO_SOT_SMD:SOT-23-3
- removed R1, R14, R2, R21, R22, R24, R25, R26, R7: 10k, Resistor_SMD:R_0805_2012Metric
- removed R37, R38, R39: 220R, Resistor_SMD:R_0805_2012Metric
- removed R40: 0R, Resistor_SMD:R_0805_2012Metric
- removed SW1: SW_DPDT_x2, sumec_brd:Custom_SPDT_2.5_Switch
- removed SW2, SW3, SW4, SW5, SW6: SW_Push, sumec_brd:SW_SPST_EVQPE1
- removed TP5, TP6, TP7, TP8, TP9: TestPoint, TestPoint:TestPoint_Pad_D1.0mm
