File: GPS-Compass/GPS-Compass.kicad_pcb (KiCad board)
At the start: 4 copper layers, 125.5 x 108.7 mm, 87 parts, among them IC1 TPS565242DRLR, J1 FFC2B28-12-G, J3 Motor_conn, J4 FFC2B28-12-G, J5 01x10, J6 USB_TypeC, Q1 SI2393DS, SW1 RESET, SW1 SPDT, SW2 BOOT, SW2 SW_SPDT, SW3 EXT, SW4 RESET, SW5 RESET, SW6 EXT, SW7 EXT, SW8 EXT, U1 DRV8834RGER, U3 USBLC6-2SC6, U4 ESP32-S3-WROOM-1

Commit message: asdasd
Parts:
- removed the C2 at (182.8, 85.8)
- removed the C3 at (182.8, 78.4)
- removed the D2 at (186.0, 135.5)
- removed the D3 at (186.0, 98.7)
- removed the D3 at (79.8, 51.2)
- removed the H1 at (187.0, 147.7)
- removed the H2 at (187.0, 60.7)
- removed the J1 at (179.0, 63.2)
- removed J4: FFC2B28-12-G, gps-compass_brd:GCT_FFC2B28-12-G
- removed the R1 at (183.8, 130.2)
- removed the R10 at (182.8, 109.9)
- removed the R2 at (183.6, 71.0)
- removed the R5 at (78.3, 54.3)
- removed the R5 at (182.8, 87.8)
- removed the R6 at (182.8, 89.8)
- removed the R7 at (182.8, 95.1)
- removed the R8 at (182.8, 80.4)
- removed the R9 at (182.8, 82.4)
- removed the SW1 at (186.0, 142.9)
- removed the SW2 at (186.0, 69.2)
- removed SW3, SW6, SW7, SW8: EXT, Connector_Wire:SolderWire-0.1sqmm_1x02_P3.6mm_D0.4mm_OD1mm_Relief
- removed SW5: RESET, Connector_Wire:SolderWire-0.1sqmm_1x02_P3.6mm_D0.4mm_OD1mm_Relief
- added BT1: LiPo cell, TestPoint:TestPoint_Pad_D2.0mm, F.Cu at (21.2, 48.4)
- added C18: 1u, Capacitor_SMD:C_0805_2012Metric, F.Cu at (34.4, 36.2)
- added C19: 47n, Capacitor_SMD:C_0805_2012Metric, F.Cu at (34.4, 39.3)
- added C20: 10u, Capacitor_SMD:C_0805_2012Metric, F.Cu at (34.4, 42.3)
- added C21: 4.7u, Capacitor_SMD:C_0805_2012Metric, F.Cu at (34.4, 45.3)
- added C22: 10u, Capacitor_SMD:C_0805_2012Metric, F.Cu at (34.4, 48.3)
- added C23: 47u, Capacitor_SMD:C_1210_3225Metric, F.Cu at (22.0, 40.8)
- added C24: 10u, Capacitor_SMD:C_0805_2012Metric, F.Cu at (34.4, 51.3)
- added D10: LED, LED_SMD:LED_0805_2012Metric, F.Cu at (38.9, 48.5)
- added D12: Schottky, Diode_SMD:D_1206_3216Metric, F.Cu at (22.0, 44.6)
- added D3: LED, LED_SMD:LED_0805_2012Metric, F.Cu at (38.9, 33.3)
- added D4: LED, LED_SMD:LED_0805_2012Metric, F.Cu at (38.9, 36.3)
- added D5: LED, LED_SMD:LED_0805_2012Metric, F.Cu at (38.9, 39.4)
- added D6: LED, LED_SMD:LED_0805_2012Metric, F.Cu at (38.9, 42.4)
- added D9: LED, LED_SMD:LED_0805_2012Metric, F.Cu at (38.9, 45.4)
- added J2: Conn_01x02_Pin, Connector_JST:JST_PH_S2B-PH-K_1x02_P2.00mm_Horizontal, F.Cu at (44.0, 31.1)
- added J8: Conn_01x02_Pin, Connector_Wire:SolderWire-0.1sqmm_1x02_P3.6mm_D0.4mm_OD1mm_Relief, F.Cu at (42.9, 40.2)
- added J9: FFC2B28-12-G, gps-compass_brd:GCT_FFC2B28-12-G, F.Cu at (41.0, 24.0)
- added L1: 2,2u, Inductor_SMD:L_Murata_DFE201610P, F.Cu at (26.0, 48.8)
- added L3: 2.2uH, Inductor_SMD:L_Walsin_WLFM201609x, F.Cu at (21.7, 52.0)
- added M2: Motor_DC, Connector_Wire:SolderWire-0.5sqmm_1x02_P4.6mm_D0.9mm_OD2.1mm_Relief, F.Cu at (29.4, 13.8)
- added Q10: SI2393DS, Package_TO_SOT_SMD:SOT-23-3, F.Cu at (29.6, 40.4)
- added Q11: SI2393DS, Package_TO_SOT_SMD:SOT-23-3, F.Cu at (29.6, 45.0)
- added Q12: DMG3406L, Package_TO_SOT_SMD:SOT-23, F.Cu at (16.7, 44.0)
- added Q13: DMG3406L, Package_TO_SOT_SMD:SOT-23, F.Cu at (16.7, 48.6)
- added Q14: SI2365EDS, Package_TO_SOT_SMD:SOT-23, F.Cu at (16.7, 53.3)
- added Q2: DMG3406L, Package_TO_SOT_SMD:SOT-23, F.Cu at (11.8, 34.8)
- added Q3: NMOS, Package_TO_SOT_SMD:SOT-23, F.Cu at (11.8, 39.4)
- added Q4: NMOS, Package_TO_SOT_SMD:SOT-23, F.Cu at (11.8, 44.0)
- added Q5: NMOS, Package_TO_SOT_SMD:SOT-23, F.Cu at (11.8, 48.6)
- added Q6: DMG3406L, Package_TO_SOT_SMD:SOT-23, F.Cu at (11.8, 53.3)
- added Q7: SI2365EDS, Package_TO_SOT_SMD:SOT-23, F.Cu at (16.7, 34.8)
- added Q8: DMG3406L, Package_TO_SOT_SMD:SOT-23, F.Cu at (16.7, 39.4)
- added Q9: SI2393DS, Package_TO_SOT_SMD:SOT-23-3, F.Cu at (29.6, 35.8)
- added R14: 10k, Resistor_SMD:R_0805_2012Metric, F.Cu at (11.6, 25.0)
- added R20: 2.2k, Resistor_SMD:R_0805_2012Metric, F.Cu at (11.6, 30.9)
- added R22: 2.2k, Resistor_SMD:R_0805_2012Metric, F.Cu at (16.0, 13.2)
- added R23: 10k, Resistor_SMD:R_0805_2012Metric, F.Cu at (16.0, 16.1)
- added R25: 10k, Resistor_SMD:R_0805_2012Metric, F.Cu at (16.0, 19.1)
- added R26: RLIM, Resistor_SMD:R_0805_2012Metric, F.Cu at (16.0, 22.1)
- added R27: 2.2k, Resistor_SMD:R_0805_2012Metric, F.Cu at (16.0, 25.0)
- added R30: 10k, Resistor_SMD:R_0805_2012Metric, F.Cu at (16.0, 27.9)
- added R31: 220R, Resistor_SMD:R_0805_2012Metric, F.Cu at (16.0, 30.9)
- added R32: 220R, Resistor_SMD:R_0805_2012Metric, F.Cu at (20.4, 13.2)
- added R33: 5.23k, Resistor_SMD:R_0805_2012Metric, F.Cu at (20.4, 16.1)
- added R34: 30.1k, Resistor_SMD:R_0805_2012Metric, F.Cu at (20.4, 19.1)
- added R40: 10k, Resistor_SMD:R_0805_2012Metric, F.Cu at (20.4, 22.1)
- added R41: 5.1k, Resistor_SMD:R_0805_2012Metric, F.Cu at (20.4, 25.0)
- added R42: 36k, Resistor_SMD:R_0805_2012Metric, F.Cu at (20.4, 27.9)
- added R43: 36k, Resistor_SMD:R_0805_2012Metric, F.Cu at (20.4, 30.9)
- added R45: 5.1K, Resistor_SMD:R_0805_2012Metric, F.Cu at (24.8, 13.2)
- added R47: 5.1K, Resistor_SMD:R_0805_2012Metric, F.Cu at (24.8, 16.1)
- added R5: 10k, Resistor_SMD:R_0805_2012Metric, F.Cu at (11.6, 19.1)
- added R50: 36k, Resistor_SMD:R_0805_2012Metric, F.Cu at (24.8, 19.1)
- added R51: 36k, Resistor_SMD:R_0805_2012Metric, F.Cu at (24.8, 22.1)
- added TH1: 10k NTC, Resistor_SMD:R_0402_1005Metric, F.Cu at (42.5, 54.0)
- added TP1: TestPoint, TestPoint:TestPoint_Pad_D1.0mm, F.Cu at (37.8, 13.2)
- added TP2: TestPoint, TestPoint:TestPoint_Pad_D1.0mm, F.Cu at (37.8, 16.3)
- added TP3: TestPoint, TestPoint:TestPoint_Pad_D1.0mm, F.Cu at (37.8, 19.4)
- added TP4: TestPoint, TestPoint:TestPoint_Pad_D1.0mm, F.Cu at (40.9, 13.2)
- added TP5: TestPoint, TestPoint:TestPoint_Pad_D1.0mm, F.Cu at (40.9, 16.3)
- added TP6: TestPoint, TestPoint:TestPoint_Pad_D1.0mm, F.Cu at (40.9, 19.4)
- added TP7: TestPoint, TestPoint:TestPoint_Pad_D1.0mm, F.Cu at (43.9, 13.2)
- added TP8: TestPoint, TestPoint:TestPoint_Pad_D1.0mm, F.Cu at (43.9, 16.3)
- added TP9: TestPoint, TestPoint:TestPoint_Pad_D1.0mm, F.Cu at (43.9, 19.4)
- added U2: TPS613222ADBV, Package_TO_SOT_SMD:SOT-23-5, F.Cu at (29.6, 49.6)
- added U5: BQ25895RTW, Package_DFN_QFN:Texas_RTW_WQFN-24-1EP_4x4mm_P0.5mm_EP2.7x2.7mm_ThermalVias, F.Cu at (22.3, 35.5)
- C4: value 100nF -> 22u
- D1: footprint Connector_Wire:SolderWire-0.1sqmm_1x02_P3.6mm_D0.4mm_OD1mm_Relief -> LED_SMD:LED_0805_2012Metric
- R3: value 1k -> 10k
- R4: value 10k -> 2.2K
- SW4: value RESET -> SHIP-MODE; footprint Connector_Wire:SolderWire-0.1sqmm_1x02_P3.6mm_D0.4mm_OD1mm_Relief -> gps-compass_brd:SW_SPST_EVQPE1
- moved R11 193.3 mm to (11.6, 22.1)
- moved R3 193.1 mm to (11.6, 13.2), turned to 0 degrees
- moved R4 192.7 mm to (11.6, 16.1)
- moved C4 166.1 mm to (34.4, 33.2), turned to 0 degrees
- moved C1 164.2 mm to (34.4, 30.2), turned to 0 degrees
- moved SW4 157.1 mm to (45.5, 50.5), turned to 0 degrees
- moved D1 154.2 mm to (38.9, 30.2), turned to 0 degrees
- moved R18 68.8 mm to (11.6, 27.9)
- moved Q1 56.7 mm to (29.6, 31.1)
Connections:
- C1 pad 1: GND -> +5V
- C1 pad 2: /DBNCD_1 -> GND
- C4 pad 1: GND -> +5V
- C4 pad 2: /DBNCD_0 -> GND
- D1 pad 1: GND -> Net-(D1-K)
- D1 pad 2: Net-(D1-A) -> +3V3
- J6 pad A4_B9: USB_VBUS -> /VBUS_PIN
- J6 pad A5: Net-(J6-CC1) -> /CC1
- J6 pad B4_A9: USB_VBUS -> /VBUS_PIN
- J6 pad B5: Net-(J6-CC2) -> /CC2
- R10 pad 2: Net-(J6-CC1) -> Net-(Q3-S)
- R11 pad 1: /DBNCD_0 -> /SDA
- R3 pad 1: /DB_1 -> Net-(U1-NFAULT)
- R3 pad 2: /DBNCD_1 -> +3V3
- R4 pad 1: /DBNCD_1 -> Net-(D1-K)
- R4 pad 2: +3V3 -> Net-(U1-NFAULT)
- SW4 pad 2: /EN -> Net-(U5-~{QON})
Routing:
- net /MSW_ON: track 86.0 -> 0.00 mm
- net +3V3: track 93.2 -> 18.0 mm, vias 9 -> 3
- net /GNSS_RST: track 64.8 -> 0.00 mm, vias 1 -> 0
- net /EN: track 63.4 -> 4.94 mm
- net /DBNCD_0: track 52.1 -> 0.00 mm, vias 2 -> 0
- net /DBNCD_1: track 44.5 -> 0.00 mm
- net /LED_EXT: track 37.0 -> 0.00 mm, vias 2 -> 0
- net /DBNCD_2: track 31.1 -> 0.00 mm
- net /DBNCD_3: track 25.2 -> 0.00 mm, vias 2 -> 0
- net /OTG_ON: track 15.4 -> 0.00 mm
- net GND: track 27.9 -> 20.4 mm, vias 53 -> 13
- net VBATT: track 6.60 -> 0.00 mm, vias 2 -> 0
- net Net-(J6-CC1): track 3.64 -> 0.00 mm
- net (no net): track 0.00 -> 3.64 mm
- net Net-(D1-A): track 2.88 -> 0.00 mm
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- removed copper zone on B.Cu, net VBATT
- removed copper zone on F.Cu, net VBATT
Other:
- board size 125.5 x 108.7 mm -> 100 x 78.5 mm
- board text removed: "DBNCD-0 GPIO"
- board text removed: "DBNCD-1 GPIO"
- board text removed: "DBNCD-2 GPIO"
- board text removed: "DBNCD-3 GPIO"
- board text removed: "EXTERNAL LED"
- board text removed: "GNSS RESET"
- board text removed: "MAIN SWITCH"
- board text removed: "MCU RESET"
- board text removed: "OTG ON"
- board text removed: "OTG SWITCH"
- board text removed: "POWER ON"

Commit message: asdasd
Parts:
- removed the BT1 at (21.2, 48.4)
- removed the BT1 at (122.8, 63.2)
- removed J9: FFC2B28-12-G, gps-compass_brd:GCT_FFC2B28-12-G
- added BT1: LiPo cell, TestPoint:TestPoint_Pad_D2.0mm, B.Cu at (122.8, 63.2)
- added J4: FFC2B28-12-G, gps-compass_brd:GCT_FFC2B28-12-G, F.Cu at (169.5, 55.8)
- BZ1: footprint inset:AST0827MW-03BTRQ_MAL -> Buzzer_Beeper:MagneticBuzzer_StarMicronics_QMB-108
- J8: footprint Connector_Wire:SolderWire-0.1sqmm_1x02_P3.6mm_D0.4mm_OD1mm_Relief -> Connector_Wire:SolderWire-0.5sqmm_1x02_P4.6mm_D0.9mm_OD2.1mm_Relief
- R35: value 220R -> 0R
- moved M2 144.3 mm to (163.1, 67.8), turned to 90 degrees
- moved R25 113.2 mm to (38.5, 130.1), turned to 90 degrees
- moved R26 111.0 mm to (41.5, 130.1), turned to 90 degrees
- moved R33 110.6 mm to (35.5, 125.7), turned to 90 degrees
- moved R34 108.1 mm to (38.5, 125.7), turned to 90 degrees
- moved C24 101.3 mm to (42.7, 152.3)
- moved C18 101.3 mm to (42.7, 137.2)
- moved C19 101.3 mm to (42.7, 140.2)
- moved C20 101.3 mm to (42.7, 143.2)
- moved C21 101.3 mm to (42.7, 146.2)
- moved C22 101.3 mm to (42.7, 149.3)
- moved C23 101.3 mm to (30.3, 141.8)
- moved L3 101.3 mm to (30.0, 153.0)
- moved SW4 101.3 mm to (53.9, 151.5)
- moved TH1 101.3 mm to (50.9, 155.0)
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Routing:
- added copper zone on B.Cu, net (none)
- removed copper zone on B.Cu, net /VBATT_POS
