File: GPS-Compass/GPS-Compass.kicad_pcb (KiCad board)
At the start: 4 copper layers, 100 x 78.5 mm, 128 parts, among them IC1 TPS565242DRLR, J1 FFC2B28-12-G, J2 Conn_01x02_Pin, J3 Motor_conn, J4 FFC2B28-12-G, J5 01x10, J6 USB_TypeC, J8 Conn_01x02_Pin, M2 Motor_DC, Q1 SI2393DS, Q10 SI2393DS, Q11 SI2393DS, Q12 DMG3406L, Q13 DMG3406L, Q14 SI2365EDS, Q2 DMG3406L, Q3 NMOS, Q4 NMOS, Q5 NMOS, Q6 DMG3406L, Q7 SI2365EDS, Q8 DMG3406L, Q9 SI2393DS, SW1 RESET, SW2 BOOT, SW4 SHIP-MODE, U1 DRV8834RGER, U2 TPS613222ADBV, U3 USBLC6-2SC6, U4 ESP32-S3-WROOM-1, U5 BQ25895RTW

Commit message: ?sd,.fvsd';
Parts:
- removed C6: 100n, Capacitor_SMD:C_0805_2012Metric
- removed Q10, Q11, Q9: SI2393DS, Package_TO_SOT_SMD:SOT-23-3
- removed Q3, Q4, Q5: NMOS, Package_TO_SOT_SMD:SOT-23
- removed R10, R41, R7: 5.1k, Resistor_SMD:R_0805_2012Metric
- removed R42, R43: 36k, Resistor_SMD:R_0805_2012Metric
- removed R6: 100k, Resistor_SMD:R_0805_2012Metric
- moved L3 118.0 mm to (96.8, 55.8), turned to 90 degrees
- moved SW4 113.4 mm to (96.2, 46.2)
- moved C23 110.2 mm to (103.3, 59.2)
- moved R22 110.1 mm to (55.8, 132.2)
- moved R23 110.1 mm to (55.8, 135.2)
- moved C24 109.8 mm to (94.6, 55.5), turned to -90 degrees
- moved U5 107.4 mm to (100.6, 55.0), turned to 180 degrees
- moved C22 106.2 mm to (92.6, 55.5), turned to -90 degrees
- moved C20 106.1 mm to (96.8, 52.0), turned to 90 degrees
- moved R27 105.4 mm to (55.8, 138.2)
- moved R30 105.4 mm to (55.8, 141.1)
- moved TH1 104.2 mm to (90.3, 58.6), turned to -90 degrees
- moved C21 103.7 mm to (100.0, 59.9), turned to -90 degrees
- moved C18 102.7 mm to (105.3, 55.8), turned to 90 degrees
- moved R25 102.2 mm to (103.6, 51.2), turned to 180 degrees
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Routing:
- net /TS: track 0.00 -> 20.2 mm, vias 0 -> 2
- net /D+: track 26.3 -> 46.3 mm, vias 0 -> 2
- net /D-: track 26.3 -> 45.7 mm, vias 0 -> 2
- net GND: track 20.4 -> 39.5 mm, vias 13 -> 24
- net VBATT: track 0.00 -> 15.0 mm
- net VSYS: track 0.00 -> 10.3 mm
- net REGN: track 0.00 -> 8.65 mm
- net Net-(C6-Pad1): track 25.4 -> 17.0 mm
- net Net-(U5-~{QON}): track 0.00 -> 7.04 mm
- net Net-(C19-Pad1): track 0.00 -> 5.08 mm
- net Net-(U5-ILIM): track 0.00 -> 4.03 mm
- net /SCL: track 5.03 -> 8.88 mm, vias 0 -> 1
- net /CC1: track 0.00 -> 3.64 mm
- net (no net): track 3.64 -> 0.00 mm
- net Net-(J6-CC2): track 3.62 -> 0.00 mm
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- added copper zone on F.Cu, net VBATT

Commit message: im to tired to write this shi
Parts:
- removed D12: Schottky, Diode_SMD:D_1206_3216Metric
- removed J8: Conn_01x02_Pin, Connector_Wire:SolderWire-0.5sqmm_1x02_P4.6mm_D0.9mm_OD2.1mm_Relief
- removed Q12, Q13, Q6, Q8: DMG3406L, Package_TO_SOT_SMD:SOT-23
- removed Q14, Q7: SI2365EDS, Package_TO_SOT_SMD:SOT-23
- removed the R11 at (24.6, 56.9)
- removed the R14 at (24.6, 59.9)
- removed the R20 at (24.6, 65.8)
- removed the R31 at (29.0, 59.9)
- removed R40: 10k, Resistor_SMD:R_0805_2012Metric
- removed R45, R47: 5.1K, Resistor_SMD:R_0805_2012Metric
- removed R50, R51: 36k, Resistor_SMD:R_0805_2012Metric
- added C17: 100n, Capacitor_SMD:C_0805_2012Metric, F.Cu at (83.5, 59.2)
- added C18: 330p, Capacitor_SMD:C_0805_2012Metric, F.Cu at (83.5, 61.2)
- added C19: 330p, Capacitor_SMD:C_0805_2012Metric, F.Cu at (83.5, 57.2)
- added C6: 100n, Capacitor_SMD:C_0805_2012Metric, F.Cu at (77.2, 57.2)
- added D11: LED, LED_SMD:LED_0805_2012Metric, F.Cu at (107.2, 67.4)
- added J7: Conn_01x02_Pin, Connector_Wire:SolderWire-0.1sqmm_1x02_P3.6mm_D0.4mm_OD1mm, F.Cu at (80.5, 56.6)
- added R12: 10k, Resistor_SMD:R_0805_2012Metric, F.Cu at (62.2, 45.5)
- added R16: 2.2k, Resistor_SMD:R_0805_2012Metric, F.Cu at (59.4, 94.2)
- added R17: 2.2k, Resistor_SMD:R_0805_2012Metric, F.Cu at (59.4, 97.2)
- added R27: 220R, Resistor_SMD:R_0805_2012Metric, F.Cu at (105.5, 87.8)
- added R28: 2.2k, Resistor_SMD:R_0805_2012Metric, F.Cu at (107.2, 63.9)
- added R6: 100k, Resistor_SMD:R_0805_2012Metric, F.Cu at (73.8, 57.2)
- added R9: 10k, Resistor_SMD:R_0805_2012Metric, F.Cu at (62.2, 47.8)
- added U5: FUSB302B11MPX, Package_DFN_QFN:WQFN-14-1EP_2.5x2.5mm_P0.5mm_EP1.45x1.45mm, F.Cu at (87.3, 59.2)
- D9: value LED -> Schottky; footprint LED_SMD:LED_0805_2012Metric -> Diode_SMD:D_1206_3216Metric
- R18: value 2.2k -> 10k
- R32: value 220R -> 10k
- moved D1 164.6 mm to (183.1, 71.2)
- moved R3 155.0 mm to (178.6, 65.3)
- moved R4 155.0 mm to (178.6, 68.3)
- moved D9 140.1 mm to (160.2, 64.7), turned to 90 degrees
- moved R32 128.4 mm to (157.3, 67.4)
- moved Q2 120.3 mm to (157.3, 64.5), turned to 90 degrees
- moved D10 89.1 mm to (105.5, 91.8), turned to 90 degrees
- moved L1 84.0 mm to (113.8, 75.2), turned to -90 degrees
- moved C4 75.2 mm to (121.2, 75.2), turned to -90 degrees
- moved C1 73.9 mm to (119.2, 75.2), turned to -90 degrees
- moved U2 71.9 mm to (116.5, 75.2), turned to 90 degrees
- moved R5 66.0 mm to (90.5, 55.5), turned to -90 degrees
- moved D3 55.9 mm to (55.8, 94.2)
- moved D4 55.9 mm to (55.8, 97.3)
- moved R18 39.9 mm to (62.2, 49.8), turned to 180 degrees
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- renumbered C18 to C20, C19 to C21, C20 to C22, C21 to C23, C22 to C24, C23 to C25, C24 to C26, R12 to R10, R13 to R11, R15 to R13, R16 to R14, R17 to R15, R22 to R19, R23 to R20, R25 to R21, R27 to R22, R26 to R23, R30 to R24, R28 to R25, R29 to R26, R33 to R29, R34 to R30, R35 to R31, R8 to R7, R9 to R8, SW4 to SW3, U5 to U6
Connections:
- net /BZ_PWM renamed /PWM_BZ
- D9 pad 1: GND -> +3V3
- J6 pad A4_B9: /VBUS_PIN -> USB_VBUS
- J6 pad B4_A9: /VBUS_PIN -> USB_VBUS
- M2 pad 2: Net-(D12-A) -> Net-(D9-A)
- Q2 pad 1: /PWM_HAPTICS -> /PWM_HPTCS
- Q2 pad 3: Net-(D12-A) -> Net-(D9-A)
- R18 pad 1: +8V -> /INT_UCON
- R18 pad 2: Net-(D3-A) -> +3V3
- R21 pad 2: /INT -> /INT_CHRG
- R32 pad 1: /LED_IOXX -> /PWM_HPTCS
- R32 pad 2: Net-(D10-A) -> GND
- U4 pad 17: /MOSI -> unconnected-(U4-IO9-Pad17)
- U4 pad 36: unconnected-(U4-IO44-Pad36) -> /GNSS_TX
- U4 pad 37: unconnected-(U4-IO43-Pad37) -> /GNSS_RX
- U4 pad 38: /STEP -> unconnected-(U4-IO2-Pad38)
- U4 pad 39: /INT -> unconnected-(U4-IO1-Pad39)
- U4 pad 4: /DIR -> unconnected-(U4-IO4-Pad4)
- U4 pad 5: /~{CS} -> unconnected-(U4-IO5-Pad5)
- U4 pad 6: /CLK -> unconnected-(U4-IO6-Pad6)
- U6 pad 7: /INT -> /INT_CHRG
Routing:
- net /D+: track 46.3 -> 0.82 mm, vias 2 -> 0
- net /D-: track 45.7 -> 1.40 mm, vias 2 -> 1
- net USB_VBUS: track 2.99 -> 24.3 mm, vias 0 -> 19
- net /CC2: track 0.00 -> 15.8 mm, vias 0 -> 2
- net /CC1: track 3.64 -> 17.5 mm, vias 0 -> 2
- net /DN_IN: track 6.59 -> 15.2 mm
- net /DP_IN: track 5.32 -> 13.5 mm
- net /PWM_BZ: track 0.00 -> 6.62 mm
- net VBATT: track 15.0 -> 20.1 mm
- net +3V3: track 18.0 -> 22.6 mm, vias 3 -> 5
- net Net-(BZ1-+): track 0.00 -> 4.34 mm
- net Net-(J3-Pin_1): track 10.4 -> 6.08 mm
- net GND: track 39.5 -> 35.3 mm, vias 24 -> 25
- net Net-(J3-Pin_3): track 9.97 -> 6.20 mm, vias 2 -> 0
- net VSYS: track 10.3 -> 6.62 mm
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- added copper zone on F.Cu, net USB_VBUS
- added copper zone on In2.Cu, net USB_VBUS

Commit message: cannot bother
Parts:
- removed the D10 at (105.5, 91.8)
- removed the D6 at (49.5, 110.2)
- removed the R20 at (54.0, 106.9)
- removed the R25 at (163.2, 74.8)
- removed the R9 at (62.2, 47.8)
- removed TP1, TP2, TP3, TP4, TP5, TP6, TP7, TP8, TP9: TestPoint, TestPoint:TestPoint_Pad_D1.0mm
- added D11: LED, LED_SMD:LED_0805_2012Metric, F.Cu at (161.4, 71.7)
- added D9: LED, LED_SMD:LED_0805_2012Metric, F.Cu at (161.4, 74.8)
- added IC2: KTS1605EUB-1-TR, gps-compass_brd:KTS1605EUB1TR, F.Cu at (102.2, 63.2)
- added R11: 10k, Resistor_SMD:R_0805_2012Metric, F.Cu at (106.0, 51.0)
- added R21: 2.2k, Resistor_SMD:R_0805_2012Metric, F.Cu at (95.2, 68.8)
- added R28: 220R, Resistor_SMD:R_0805_2012Metric, F.Cu at (157.2, 71.8)
- R17: value 2.2k -> 2.2K
- R18, R24: value 10k -> 2.2k
- R19, R22: value 2.2k -> 10k
- R26: value 220R -> 10k
- moved D5 86.4 mm to (129.5, 74.5), turned to -90 degrees
- moved D8 76.3 mm to (90.5, 72.2), turned to -90 degrees
- moved R26 74.8 mm to (88.5, 70.5), turned to -90 degrees
- moved R18 73.5 mm to (131.5, 74.5), turned to -90 degrees
- moved D3 73.0 mm to (126.0, 74.5), turned to -90 degrees
- moved D7 71.5 mm to (95.2, 72.2), turned to -90 degrees
- moved R16 67.5 mm to (124.0, 74.5), turned to -90 degrees
- moved R24 57.2 mm to (90.5, 68.8), turned to -90 degrees
- moved R22 55.6 mm to (93.2, 70.5), turned to -90 degrees
- moved R27 53.3 mm to (157.2, 74.8), turned to 180 degrees
- moved R12 46.0 mm to (107.9, 51.0), turned to 90 degrees
- moved R19 44.8 mm to (83.8, 70.5), turned to -90 degrees
- moved D4 39.1 mm to (85.8, 72.2), turned to -90 degrees
- moved R17 38.8 mm to (85.8, 68.8), turned to 90 degrees
- moved D1 37.3 mm to (148.8, 56.7), turned to 90 degrees
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- renumbered C16 to C15, C15 to C16, C21 to C22, C22 to C23, C23 to C24, C24 to C25, C25 to C26, C26 to C27, D9 to D10, D11 to D6, J4 to J1, J1 to J2, J2 to J3, J3 to J4, R11 to R10, R28 to R20, R21 to R23, R23 to R25, R10 to R9
Connections:
- D4 pad 1: GND -> Net-(D4-K)
- D4 pad 2: Net-(D4-A) -> +3V3
- D5 pad 1: /STAT -> GND
- D7 pad 1: GND -> Net-(D7-K)
- D7 pad 2: Net-(D7-A) -> +3V3
- D8 pad 1: GND -> Net-(D8-K)
- D8 pad 2: Net-(D8-A) -> +3V3
- R17 pad 1: +3V3 -> Net-(D4-K)
- R17 pad 2: Net-(D4-A) -> /INT_UCON
- R18 pad 1: /INT_UCON -> +3V3
- R18 pad 2: +3V3 -> Net-(D5-A)
- R19 pad 1: +3V3 -> /INT_UCON
- R19 pad 2: Net-(D5-A) -> +3V3
- R22 pad 1: +3V3 -> /STAT
- R22 pad 2: Net-(D6-A) (its old number) -> +3V3
- R24 pad 2: +3V3 -> Net-(D8-K)
- R26 pad 1: /LED_IOXX -> /DSEL
- R26 pad 2: Net-(D8-A) -> +3V3
- U4 pad 12: /SDA -> unconnected-(U4-IO8-Pad12)
- U4 pad 6: unconnected-(U4-IO6-Pad6) -> /SDA
Routing:
- net +3V3: track 22.6 -> 248.0 mm, vias 5 -> 15
- net /SCL: track 9.07 -> 96.0 mm, vias 0 -> 5
- net /SDA: track 9.10 -> 94.2 mm, vias 0 -> 5
- net /GNSS_TX: track 0.00 -> 72.4 mm, vias 0 -> 2
- net /GNSS_RX: track 0.00 -> 71.6 mm, vias 0 -> 2
- net VIN: track 0.00 -> 63.3 mm, vias 0 -> 7
- net +5V: track 0.79 -> 61.3 mm, vias 0 -> 5
- net /D+: track 0.82 -> 39.1 mm, vias 0 -> 2
- net /D-: track 1.40 -> 35.0 mm, vias 1 -> 2
- net /STAT: track 1.41 -> 30.7 mm, vias 1 -> 2
- net /EN: track 4.94 -> 29.2 mm, vias 0 -> 2
- net /DSEL: track 0.84 -> 24.4 mm, vias 1 -> 2
- net /GNSS_WKP: track 0.00 -> 22.3 mm
- net /GNSS_RST: track 0.00 -> 21.3 mm
- net /INT_UCON: track 0.00 -> 17.7 mm, vias 0 -> 2
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- added copper zone on F.Cu, net VOTG

Commit message: i think im depressed again
Parts:
- removed J1: FFC2B28-12-G, gps-compass_brd:GCT_FFC2B28-12-G
- added J8: FFC2B28-12-G, gps-compass_brd:GCT_FFC2B28-12-G, F.Cu at (169.5, 55.8)
- added TP1: TestPoint, TestPoint:TestPoint_Pad_D1.0mm, F.Cu at (77.2, 53.0)
- added TP2: TestPoint, TestPoint:TestPoint_Pad_D1.0mm, F.Cu at (81.0, 69.2)
- added TP3: TestPoint, TestPoint:TestPoint_Pad_D1.0mm, F.Cu at (144.1, 87.8)
- added TP4: TestPoint, TestPoint:TestPoint_Pad_D1.0mm, F.Cu at (118.5, 71.5)
- added TP5: TestPoint, TestPoint:TestPoint_Pad_D1.0mm, F.Cu at (110.8, 86.5)
- added TP6: TestPoint, TestPoint:TestPoint_Pad_D1.0mm, F.Cu at (141.1, 87.8)
- added TP7: TestPoint, TestPoint:TestPoint_Pad_D1.0mm, F.Cu at (138.0, 93.8)
- added TP8: TestPoint, TestPoint:TestPoint_Pad_D1.0mm, F.Cu at (138.0, 90.8)
- added TP9: TestPoint, TestPoint:TestPoint_Pad_D1.0mm, F.Cu at (138.0, 87.8)
- BT1: moved to F.Cu
- moved BT1 87.7 mm to (41.0, 31.5), turned to 180 degrees
- moved D9 43.1 mm to (118.5, 79.0), turned to -90 degrees
- moved D11 38.2 mm to (124.0, 79.1), turned to -90 degrees
- moved R27 37.0 mm to (120.5, 79.0), turned to -90 degrees
- moved R28 32.1 mm to (126.0, 79.1), turned to -90 degrees
- moved R4 5.04 mm to (153.8, 59.5)
- moved R14 4.10 mm to (135.8, 68.2), turned to -90 degrees
- moved D1 4.09 mm to (151.8, 59.5)
- moved C7 2.70 mm to (105.8, 82.2)
- moved C9 2.70 mm to (107.8, 82.2)
- moved L2 2.70 mm to (105.2, 78.8)
- moved R7 2.70 mm to (110.7, 82.2)
- moved C11 2.70 mm to (108.6, 78.9)
- moved C13 2.70 mm to (110.6, 78.8)
- moved C14 2.70 mm to (112.6, 78.8)
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Connections:
- R27 pad 1: /LED_IOXX -> /LED_IO13
- R28 pad 1: /LED_IOXX -> /LED_IO21
- R3 pad 1: Net-(U1-NFAULT) -> /NFAULT
- R4 pad 2: Net-(U1-NFAULT) -> /NFAULT
- U1 pad 13: Net-(U1-NFAULT) -> /NFAULT
- U4 pad 10: unconnected-(U4-IO17-Pad10) -> /INT_UCON
- U4 pad 11: unconnected-(U4-IO18-Pad11) -> /GNSS_WKP
- U4 pad 12: unconnected-(U4-IO8-Pad12) -> /PWM_BZ
- U4 pad 17: unconnected-(U4-IO9-Pad17) -> /GNSS_RST
- U4 pad 21: unconnected-(U4-IO13-Pad21) -> /LED_IO13
- U4 pad 22: unconnected-(U4-IO14-Pad22) -> /PWM_HPTCS
- U4 pad 23: unconnected-(U4-IO21-Pad23) -> /LED_IO21
- U4 pad 24: unconnected-(U4-IO47-Pad24) -> /STEP
- U4 pad 25: unconnected-(U4-IO48-Pad25) -> /DIR
- U4 pad 28: unconnected-(U4-IO35-Pad28) -> /NFAULT
- U4 pad 29: unconnected-(U4-IO36-Pad29) -> /DBNCD_0
- U4 pad 30: unconnected-(U4-IO37-Pad30) -> /DBNCD_1
- U4 pad 31: unconnected-(U4-IO38-Pad31) -> /LED_EXT
- U4 pad 32: unconnected-(U4-IO39-Pad32) -> /DBNCD_2
- U4 pad 33: unconnected-(U4-IO40-Pad33) -> /DBNCD_3
- U4 pad 34: unconnected-(U4-IO41-Pad34) -> /OTG
- U4 pad 35: unconnected-(U4-IO42-Pad35) -> /MOSI
- U4 pad 38: unconnected-(U4-IO2-Pad38) -> /CLK
- U4 pad 39: unconnected-(U4-IO1-Pad39) -> /~{CS}
- U4 pad 4: unconnected-(U4-IO4-Pad4) -> /INT_CHRG
- U4 pad 5: unconnected-(U4-IO5-Pad5) -> /EN_LS
- U4 pad 8: unconnected-(U4-IO15-Pad8) -> /DSEL
- U4 pad 9: unconnected-(U4-IO16-Pad9) -> /STAT
Routing:
- net /GNSS_RST: track 21.3 -> 118.4 mm, vias 0 -> 6
- net /MSW_ON: track 1.88 -> 94.6 mm, vias 0 -> 2
- net /OTG: track 1.61 -> 76.0 mm, vias 1 -> 2
- net /PWM_HPTCS: track 1.98 -> 43.4 mm, vias 0 -> 2
- net /DBNCD_0: track 0.00 -> 40.8 mm
- net /DBNCD_1: track 0.00 -> 40.7 mm
- net /LED_EXT: track 0.00 -> 40.5 mm
- net /DBNCD_2: track 0.00 -> 40.4 mm
- net /DBNCD_3: track 0.00 -> 40.3 mm
- net /EN: track 29.2 -> 67.3 mm, vias 2 -> 4
- net /GNSS_WKP: track 22.3 -> 55.1 mm, vias 0 -> 2
- net /NFAULT: track 0.00 -> 32.4 mm, vias 0 -> 2
- net /PWM_BZ: track 0.00 -> 27.9 mm, vias 0 -> 2
- net /INT_UCON: track 17.7 -> 44.8 mm, vias 2 -> 4
- net /STEP: track 0.00 -> 26.2 mm, vias 0 -> 2
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
Commit message: sdas
Parts:
- removed BT1: LiPo cell, TestPoint:TestPoint_Pad_D2.0mm
- removed the TP8 at (138.0, 90.8)
- added TP1: TestPoint, TestPoint:TestPoint_Pad_D1.0mm, F.Cu at (84.0, 54.8)
- added TP11: TestPoint, TestPoint:TestPoint_Pad_D1.0mm, F.Cu at (132.4, 98.7)
- added TP12: TestPoint, TestPoint:TestPoint_Pad_D1.0mm, F.Cu at (132.4, 101.8)
- added TP13: TestPoint, TestPoint:TestPoint_Pad_D1.0mm, F.Cu at (149.5, 69.8)
- added TP14: TestPoint, TestPoint:TestPoint_Pad_D1.0mm, F.Cu at (81.8, 103.0)
- added TP15: TestPoint, TestPoint:TestPoint_Pad_D1.0mm, F.Cu at (119.6, 79.2)
- added TP16: TestPoint, TestPoint:TestPoint_Pad_D1.0mm, F.Cu at (98.8, 103.2)
- added TP17: TestPoint, TestPoint:TestPoint_Pad_D1.0mm, F.Cu at (120.8, 81.2)
- added TP18: TestPoint, TestPoint:TestPoint_Pad_D1.0mm, F.Cu at (77.8, 55.2)
- added TP19: TestPoint, TestPoint:TestPoint_Pad_D1.0mm, F.Cu at (122.1, 79.2)
- added TP20: TestPoint, TestPoint:TestPoint_Pad_D1.0mm, F.Cu at (75.2, 55.2)
- added TP5: TestPoint, TestPoint:TestPoint_Pad_D1.0mm, F.Cu at (129.3, 98.7)
- moved TP7 34.8 mm to (154.5, 63.2), turned to 0 degrees
- moved TP6 18.2 mm to (129.3, 101.8), turned to 0 degrees
- moved J5 16.9 mm to (82.8, 88.3)
- moved TP3 16.7 mm to (129.3, 95.7), turned to 0 degrees
- moved D11 15.3 mm to (133.8, 79.2)
- moved R28 11.3 mm to (131.8, 79.2)
- moved D10 11.2 mm to (133.8, 73.5)
- moved TP9 9.68 mm to (132.4, 95.7), turned to 0 degrees
- moved R18 8.46 mm to (124.5, 79.2)
- moved R27 8.02 mm to (131.8, 73.5)
- moved D5 5.62 mm to (126.5, 79.2)
- moved C1 2.25 mm to (116.2, 74.5)
- moved C4 2.25 mm to (118.2, 74.5)
- moved L1 2.25 mm to (110.8, 74.5)
- moved U2 2.25 mm to (113.5, 74.5)
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- renumbered C22 to C21, C23 to C22, C24 to C23, C25 to C24, C26 to C25, C27 to C26, D11 to D10, D9 to D11, D10 to D9, J2 to J1, J3 to J2, J4 to J3, J8 to J4, R9 to R10, R10 to R11, R11 to R12, R25 to R24, R24 to R25, R28 to R27, R27 to R28, R12 to R9, TP5 to TP10, TP1 to TP2, TP2 to TP4, TP4 to TP8
Connections:
- TP3 pad 1: 5V_CONV -> /DSEL
- TP6 pad 1: unconnected-(TP6-Pad1) -> VOTG
- TP7 pad 1: unconnected-(TP7-Pad1) -> /NFAULT
- TP9 pad 1: unconnected-(TP9-Pad1) -> /INT_UCON
- U4 pad 18: unconnected-(U4-IO10-Pad18) -> /IO10
- U4 pad 19: unconnected-(U4-IO11-Pad19) -> /IO11
- U4 pad 20: unconnected-(U4-IO12-Pad20) -> /IO12
Routing:
- net /SDA: track 94.1 -> 68.8 mm, vias 5 -> 7
- net /SCL: track 95.4 -> 71.1 mm
- net /GNSS_RST: track 118.4 -> 94.6 mm, vias 6 -> 7
- net /GNSS_WKP: track 55.1 -> 31.6 mm
- net /GNSS_TX: track 73.1 -> 49.7 mm
- net /GNSS_RX: track 72.9 -> 49.8 mm
- net +3V3: track 253.5 -> 232.1 mm
- net /IO11: track 0.00 -> 12.8 mm
- net /IO10: track 0.00 -> 10.8 mm
- net /IO12: track 0.00 -> 10.8 mm
- net /CC2: track 15.8 -> 25.3 mm, vias 2 -> 3
- net /CC1: track 17.5 -> 24.7 mm, vias 2 -> 3
- net GND: track 64.1 -> 69.4 mm, vias 36 -> 75
- net /LED_IO13: track 10.8 -> 15.1 mm
- net VIN: track 64.5 -> 61.5 mm
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