File: GPS-Compass/GPS-Compass.kicad_sch (KiCad schematic)
At the start: 127 parts, among them IC1 TPS565242DRLR, J1 FFC2B28-12-G, J2 Conn_01x02_Pin, J3 Motor_conn, J5 01x10, J6 USB_TypeC, J7 USB_TypeC, J8 Conn_01x02_Pin, M1 Stepper_Motor_bipolar, M2 FAN, Q1 SI2393DS, Q2 SI2393DS, SW1 RESET, SW2 BOOT, SW4 SHIP-MODE, U1 DRV8834RGER, U2 TPS613222ADBV, U3 USBLC6-2SC6, U4 ESP32-S3-WROOM-1, U5 BQ25895RTW, U6 BQ25887

Commit message: no chsanges
Other:
- note added: "FAN"

Commit message: asdasd
Parts:
- removed C17: 100n, Capacitor_SMD:C_0805_2012Metric, symbol Device:C_Small
- removed J7: USB_TypeC, sumec_brd:HRO_TYPE-C-31-M-12, symbol sumec_sch_lib:USB_TypeC
- removed M2: FAN, Connector:FanPinHeader_1x04_P2.54mm_Vertical, symbol Motor:Fan_4pin
- removed Q2: SI2393DS, Package_TO_SOT_SMD:SOT-23-3, symbol Device:Q_PMOS_GSD
- removed R19: 100k, Resistor_SMD:R_0805_2012Metric, symbol Device:R_Small
- removed R21, R24: 36k, Resistor_SMD:R_0805_2012Metric, symbol Device:R_Small
- removed R7: 5.1k, Resistor_SMD:R_0805_2012Metric, symbol Device:R_Small
- added D11: LED, Connector_Wire:SolderWire-0.1sqmm_1x02_P3.6mm_D0.4mm_OD1mm_Relief, symbol Device:LED
- added D12: Schottky, Diode_SMD:D_1206_3216Metric, symbol Device:D_Schottky_Small
- added J9: FFC2B28-12-G, gps-compass_brd:GCT_FFC2B28-12-G, symbol gps-compass_sch:FFC2B28-12-G
- added M2: Motor_DC, Connector_Wire:SolderWire-0.5sqmm_1x02_P4.6mm_D0.9mm_OD2.1mm_Relief, symbol Motor:Motor_DC
- added Q10, Q11, Q9: SI2393DS, Package_TO_SOT_SMD:SOT-23-3, symbol Device:Q_PMOS_GSD
- added Q12, Q13, Q2, Q6, Q8: DMG3406L, Package_TO_SOT_SMD:SOT-23, symbol Transistor_FET:DMG3406L
- added Q14, Q7: SI2365EDS, Package_TO_SOT_SMD:SOT-23, symbol Transistor_FET:Si2319CDS
- added Q3, Q4, Q5: NMOS, Package_TO_SOT_SMD:SOT-23, symbol Transistor_FET:Q_NMOS_GDS
- added R41: 5.1k, Resistor_SMD:R_0805_2012Metric, symbol Device:R_Small
- added R42, R43: 36k, Resistor_SMD:R_0805_2012Metric, symbol Device:R_Small
- added R44: 2.2k, Resistor_SMD:R_0805_2012Metric, symbol Device:R
- added R45, R47: 5.1K, Resistor_SMD:R_0805_2012Metric, symbol Device:R
- added R48, R49: 10k, Resistor_SMD:R_0805_2012Metric, symbol Device:R_Small
- added R50, R51: 36k, Resistor_SMD:R_0805_2012Metric, symbol Device:R
- added SW3: SW_SPDT, Connector_Wire:SolderWire-0.1sqmm_1x02_P3.6mm_D0.4mm_OD1mm_Relief, symbol Switch:SW_SPDT
Connections:
- net +3V3: now also D12.1 (K), J9.2, M2.1 (+), R42.1, R43.1, R50.1, R51.1, SW3.2 (B)
- net +5V: no longer R40.1
- net EN: now also J9.9
- net GND: now also R40.2, D11.1 (K), J9.12, J9.4, Q2.2 (S), Q6.2 (S), Q8.2 (S), R41.1, R48.2, R49.1
- net GNSS_RST: now also J9.10
- net MSW_ON: now also J9.11
- net USB_VBUS: now also Q5.3 (S), Q7.3 (D); no longer J6.A4_B9 (VBUS), J6.B4_A9 (VBUS)
- net VOTG: now also Q14.2 (S)
- net ~{FAN_SW}: no longer R40.2
- net CC2: now reaches J6.B5 (CC2)
- net CC2: now also Q13.2 (S), Q3.2 (D), Q9.3 (D), R47.1
- net at R10.2: now also Q3.3 (S); no longer J6.A5 (CC1)
- new net: D11.2 (A), R44.2
- new net: D12.2 (A), M2.2 (-), Q2.3 (D)
- new net: Q13.3 (D), R51.2
- new net: Q10.2 (S), R42.2
- new net: Q9.2 (S), R43.2
- new net: Q12.3 (D), R50.2
- new net: Q4.3 (S), R41.2
- new net: Q8.3 (D), R47.2
- new net: J9.S1 (SHIELD), J9.S2 (SHIELD)
- new net: Q6.3 (D), R45.2
- new net CC1: J6.A5 (CC1), Q10.3 (D), Q12.2 (S), Q4.2 (D), R45.1
- new net DBNCD_0: J9.8
- new net DBNCD_1: J9.7
- new net DBNCD_2: J9.5
- new net DBNCD_3: J9.3
- new net LED_EXT: J9.6
- new net OTG_ON: J9.1, R44.1
- new net POS_1: Q14.1 (G), Q6.1 (G), Q8.1 (G), R49.2, SW3.1 (A)
- new net POS_2: Q12.1 (G), Q13.1 (G), Q7.1 (G), R48.1, SW3.3 (C)
- new net PWM_HAPTICS: Q2.1 (G), R40.1
- new net SINK: Q3.1 (G), Q4.1 (G), Q5.1 (G)
- new net SOURCE: Q10.1 (G), Q11.1 (G), Q9.1 (G)
- new net USB_VOTG: Q11.2 (S)
- new net VBUS: Q11.3 (D), Q5.2 (D)
- new net VBUS_PIN: J6.A4_B9 (VBUS), J6.B4_A9 (VBUS), Q14.3 (D), Q7.2 (S)
- no-connect marks 20 -> 14
Other:
- note added: "1. UI PCB, accomedate the SINK/SOURCE SW 2. 3. add test points for charger IC 4. 5. 6. 7."
- note added: "CHARGE IND."
- note added: "HAPTICS"
- note added: "OTG SW"
- note added: "SINK"
- note added: "SINK/SOURCE SWITCHING"
- note added: "SOURCE"
- note added: "UI CONN"
- note removed: "1. FUEL GAUGE 2. LiPo/Li-Ion 3. add test points for charger IC 4. 5. 6. 7."
- note removed: "BATT. INDICATOR"
- note removed: "FAN"
- note removed: "USB C OTG CHARGER"
- moved on the sheet: C16, C6, D5, D6, J6, J8, M1, Q1, R10, R12, R13, R22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

Commit message: asdasd
Parts:
- removed J9: FFC2B28-12-G, gps-compass_brd:GCT_FFC2B28-12-G, symbol gps-compass_sch:FFC2B28-12-G
- added J4: FFC2B28-12-G, gps-compass_brd:GCT_FFC2B28-12-G, symbol gps-compass_sch:FFC2B28-12-G
- BZ1: footprint inset:AST0827MW-03BTRQ_MAL -> Buzzer_Beeper:MagneticBuzzer_StarMicronics_QMB-108
- J8: footprint Connector_Wire:SolderWire-0.1sqmm_1x02_P3.6mm_D0.4mm_OD1mm_Relief -> Connector_Wire:SolderWire-0.5sqmm_1x02_P4.6mm_D0.9mm_OD2.1mm_Relief
- R35: value 220R -> 0R
Connections:
- net +3V3: now also J4.2
- net DBNCD_0: now also J4.9
- net DBNCD_1: now also J4.8
- net DBNCD_2: now also J4.6
- net DBNCD_3: now also J4.5
- net EN: now also J4.10
- net GND: now also J4.1
- net GNSS_RST: now also J4.11
- net LED_EXT: now also J4.7
- net MSW_ON: now also J4.12
- new net: J4.S1 (SHIELD), J4.S2 (SHIELD)
- new net SINK-MODE: J4.3
- new net SRC-MODE: J4.4

Commit message: ?sd,.fvsd';
Parts:
- removed D11: LED, Connector_Wire:SolderWire-0.1sqmm_1x02_P3.6mm_D0.4mm_OD1mm_Relief, symbol Device:LED
- removed Q10, Q11, Q9: SI2393DS, Package_TO_SOT_SMD:SOT-23-3, symbol Device:Q_PMOS_GSD
- removed Q3, Q4, Q5: NMOS, Package_TO_SOT_SMD:SOT-23, symbol Transistor_FET:Q_NMOS_GDS
- removed R10, R41: 5.1k, Resistor_SMD:R_0805_2012Metric, symbol Device:R_Small
- removed R42, R43: 36k, Resistor_SMD:R_0805_2012Metric, symbol Device:R_Small
- removed R44: 2.2k, Resistor_SMD:R_0805_2012Metric, symbol Device:R
- removed R48, R49: 10k, Resistor_SMD:R_0805_2012Metric, symbol Device:R_Small
- removed SW3: SW_SPDT, Connector_Wire:SolderWire-0.1sqmm_1x02_P3.6mm_D0.4mm_OD1mm_Relief, symbol Switch:SW_SPDT
Other:
- note removed: "OTG SW"

Commit message: im to tired to write this shi
Parts:
- removed D10: LED, LED_SMD:LED_0805_2012Metric, symbol Device:LED
- removed R32: 220R, Resistor_SMD:R_0805_2012Metric, symbol Device:R
- added C17: 100n, Capacitor_SMD:C_0805_2012Metric, symbol Device:C_Small
- added C18, C19: 330p, Capacitor_SMD:C_0805_2012Metric, symbol Device:C_Small
- added D11: LED, LED_SMD:LED_0805_2012Metric, symbol Device:LED
- added R18: 10k, Resistor_SMD:R_0805_2012Metric, symbol Device:R_Small
- added R28: 2.2k, Resistor_SMD:R_0805_2012Metric, symbol Device:R
- added U5: FUSB302B11MPX, Package_DFN_QFN:WQFN-14-1EP_2.5x2.5mm_P0.5mm_EP1.45x1.45mm, symbol Interface_USB:FUSB302B11MPX
- J7: renamed from J8; footprint Connector_Wire:SolderWire-0.5sqmm_1x02_P4.6mm_D0.9mm_OD2.1mm_Relief -> Connector_Wire:SolderWire-0.1sqmm_1x02_P3.6mm_D0.4mm_OD1mm
- renumbered C18 to C20, C19 to C21, C20 to C22, C21 to C23, C22 to C24, C23 to C25, C24 to C26, C25 to C27, C26 to C28, C27 to C29, C28 to C30, C29 to C31, C30 to C32, C31 to C33, D9 to D10, D12 to D9, Q12 to Q3, Q8 to Q4, Q13 to Q5, Q14 to Q7, Q7 to Q8, R12 to R10, R13 to R11, R14 to R12, R15 to R13, R16 to R14, R17 to R15, R18 to R16, R20 to R17, R22 to R19, R23 to R20, R25 to R21, R27 to R22, R26 to R23, R30 to R24, R28 to R25, R29 to R26, R31 to R27, R33 to R29, R34 to R30, R35 to R31, R40 to R32, R36 to R33, R37 to R34, R38 to R35, R39 to R36, R50 to R37, R47 to R38, R51 to R39, R45 to R40, R8 to R7, R9 to R8, R11 to R9, SW4 to SW3, U5 to U6, U6 to U7
Connections:
- net +8V is gone; now on net +5V: R16.1
- net +3V3: now also C17.1, R18.2, U5.12 (VCONN), U5.13 (VCONN), U5.3 (VDD), U5.4 (VDD)
- net CC1: now also C19.1, U5.10 (CC1), U5.11 (CC1)
- net CC2: now also C18.1, U5.1 (CC2), U5.14 (CC2)
- net CLK: no longer U4.6 (IO6)
- net DIR: no longer U4.4 (IO4)
- net GND: now also C17.2, C18.2, C19.2, D11.1 (K), U5.15 (GND), U5.8 (GND), U5.9 (GND)
- net GNSS_RX: now also U4.37 (IO43)
- net GNSS_TX: now also U4.36 (IO44)
- net MOSI: no longer U4.17 (IO9)
- net SCL: now also U5.6 (SCL)
- net SDA: now also U5.7 (SDA)
- net STEP: no longer U4.38 (IO2)
- net USB_VBUS: now also J6.A4_B9 (VBUS), J6.B4_A9 (VBUS), U5.2 (VBUS)
- net VBUS_PIN: no longer J6.A4_B9 (VBUS), J6.B4_A9 (VBUS)
- net VOTG: now also R28.1
- net ~{CS}: no longer U4.5 (IO5)
- net BZ_PWM renamed PWM_BZ
- net INT renamed INT_CHRG
- net INT_CHRG: no longer U4.39 (IO1)
- net PWM_HAPTICS renamed PWM_HPTCS
- new net: D11.2 (A), R28.2
- new net INT_UCON: R18.1, U5.5 (INT_N)
Other:
- note added: "1. VBUS - OTG backfeed? 2. OTG to VBUS? Check for mosfets on BQ 3. add test points for charger IC 4. 5. 6. 7."
- note removed: "1. UI PCB, accomedate the SINK/SOURCE SW 2. 3. add test points for charger IC 4. 5. 6. 7."
- note removed: "I2C PULLUS"
- note removed: "probs not meant to be connected to the MCU"
- moved on the sheet: D2, D3, D4, Q3, Q4, Q5, Q6, Q7, Q8, R15, R16, R17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

Commit message: cannot bother
Parts:
- removed D8: LED, LED_SMD:LED_0805_2012Metric, symbol Device:LED
- removed R26: 220R, Resistor_SMD:R_0805_2012Metric, symbol Device:R
- added D4: LED, LED_SMD:LED_0805_2012Metric, symbol Device:LED_Small
- added IC2: KTS1605EUB-1-TR, gps-compass_brd:KTS1605EUB1TR, symbol gps-compass_sch:KTS1605EUB-1-TR
- added JP4: Jumper, Jumper:SolderJumper-3_P1.3mm_Open_RoundedPad1.0x1.5mm_NumberLabels, symbol Jumper:SolderJumper_3_Open
- added R17: 2.2K, Resistor_SMD:R_0805_2012Metric, symbol Device:R_Small
- renumbered C16 to C15, C15 to C16, C21 to C22, C22 to C23, C23 to C24, C24 to C25, C25 to C26, C26 to C27, C27 to C29, C28 to C30, C29 to C31, C30 to C32, C31 to C33, C32 to C34, C33 to C35, D9 to D10, D10 to D11, D4 to D5, D11 to D6, D5 to D7, D6 to D8, D7 to D9, J4 to J1, J1 to J2, J2 to J3, J3 to J4, JP4 to JP5, R11 to R10, R9 to R11, R17 to R18, R18 to R19, R28 to R20, R19 to R21, R20 to R22, R21 to R23, R22 to R24, R23 to R25, R24 to R26, R25 to R27, R27 to R28, R10 to R9
Connections:
- net +3V3: now also D7.2 (A), D8.2 (A), D4.2 (A), JP4.1 (A); no longer R21.1, R24.1
- net DSEL: now also R24.1; no longer D8.1 (K)
- net GND: now also IC2.C1 (GND), JP4.3 (B)
- net INT_UCON: now also R17.2
- net SDA: now also U4.6 (IO6); no longer U4.12 (IO8)
- net STAT: now also R21.1; no longer D7.1 (K)
- net USB_VBUS: now also IC2.A1 (OUT_1), IC2.B1 (OUT_2)
- net VOTG: now also IC2.A2 (IN_1), IC2.B2 (IN_2)
- net at R21.2: now also D7.1 (K); no longer D7.2 (A)
- net at R24.2: now also D8.1 (K); no longer D8.2 (A)
- new net: D4.1 (K), R17.1
- new net EN_LS: IC2.C2 (EN), JP4.2 (C)
Other:
- note added: "1. Change the UI PCB 2. 3. add test points for charger IC 4. 5. 6. 7."
- note added: "CHARGE INDICATOR"
- note added: "LOAD SWITCH"
- note added: "USB CC LOGIC"
- note removed: "1. VBUS - OTG backfeed? 2. OTG to VBUS? Check for mosfets on BQ 3. add test points for charger IC 4. 5. 6. 7."
- note removed: "CHARGE IND."
- moved on the sheet: C15, C17, C18, C19, C6, D7, D8, J1, J6, J7, R10, R11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

Commit message: i think im depressed again
Parts:
- removed J1: FFC2B28-12-G, gps-compass_brd:GCT_FFC2B28-12-G, symbol gps-compass_sch:FFC2B28-12-G
- removed JP4: Jumper, Jumper:SolderJumper-3_P1.3mm_Open_RoundedPad1.0x1.5mm_NumberLabels, symbol Jumper:SolderJumper_3_Open
- added J8: FFC2B28-12-G, gps-compass_brd:GCT_FFC2B28-12-G, symbol gps-compass_sch:FFC2B28-12-G
Connections:
- net +3V3: now also J8.11
- net CLK: now also U4.38 (IO2)
- net DBNCD_0: now also U4.29 (IO36), J8.4
- net DBNCD_1: now also U4.30 (IO37), J8.5
- net DBNCD_2: now also U4.32 (IO39), J8.7
- net DBNCD_3: now also U4.33 (IO40), J8.8
- net DIR: now also U4.25 (IO48)
- net DSEL: now also U4.8 (IO15)
- net EN: now also J8.3
- net EN_LS: now also U4.5 (IO5)
- net GND: now also J8.10, J8.12
- net GNSS_RST: now also U4.17 (IO9), J8.2
- net GNSS_WKP: now also U4.11 (IO18)
- net INT_CHRG: now also U4.4 (IO4)
- net INT_UCON: now also U4.10 (IO17)
- net LED_EXT: now also U4.31 (IO38), J8.6
- net MOSI: now also U4.35 (IO42)
- net MSW_ON: now also J8.1
- net OTG: now also U4.34 (IO41), J8.9
- net PWM_BZ: now also U4.12 (IO8)
- net PWM_HPTCS: now also U4.22 (IO14)
- net STAT: now also U4.9 (IO16)
- net STEP: now also U4.24 (IO47)
- net ~{CS}: now also U4.39 (IO1)
- net NFAULT: now reaches R3.1, R4.2, U1.13 (NFAULT)
- net NFAULT: now also U4.28 (IO35)
- net LED_IO13: now reaches U4.21 (IO13)
- net LED_IO13: now also R27.1
- net LED_IO21: now reaches U4.23 (IO21)
- net LED_IO21: now also R28.1
- net 5V_CONV: no longer names the net of TP3.1
- removed net LED_IOXX: R27.1, R28.1
- new net: J8.S1 (SHIELD), J8.S2 (SHIELD)
- no-connect marks 14 -> 11
Other:
- moved on the sheet: D1, R11, R12, R3, R4

Commit message: sdas
Parts:
- added TP1, TP11, TP13, TP15, TP17, TP19, TP20, TP3, TP5, TP7, TP9: TestPoint, TestPoint:TestPoint_Pad_D1.0mm, symbol Connector:TestPoint
- BT1: footprint TestPoint:TestPoint_Pad_D2.0mm -> (none)
- renumbered C22 to C21, C23 to C22, C24 to C23, C25 to C24, C26 to C25, C27 to C26, C29 to C27, C30 to C28, C31 to C29, C32 to C30, C33 to C31, C34 to C32, C35 to C33, D11 to D10, D9 to D11, D10 to D9, J2 to J1, J3 to J2, J4 to J3, J8 to J4, JP5 to JP4, R9 to R10, R10 to R11, R11 to R12, R25 to R24, R24 to R25, R28 to R27, R27 to R28, R12 to R9, TP5 to TP10, TP6 to TP12, TP7 to TP14, TP8 to TP16, TP9 to TP18, TP1 to TP2, TP2 to TP4, TP3 to TP6, TP4 to TP8
Connections:
- net CC1: now also TP18.1
- net CC2: now also TP20.1
- net DIR: now also TP13.1
- net DSEL: now also TP3.1
- net INT_UCON: now also TP9.1
- net NFAULT: now also TP7.1
- net SCL: now also TP16.1
- net SDA: now also TP14.1
- net STAT: now also TP5.1
- net STEP: now also TP11.1
- net VIN: now also TP12.1
- net VOTG: now also TP6.1
- net VSYS: now also TP1.1
- net IO10: now reaches U4.18 (IO10)
- net IO10: now also TP15.1
- net IO11: now reaches U4.19 (IO11)
- net IO11: now also TP17.1
- net IO12: now reaches U4.20 (IO12)
- net IO12: now also TP19.1
Other:
- moved on the sheet: D10, D11, J7, M1, R27, R28, TP10, TP12, TP14, TP16, TP18, TP2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
