File: GPS-Compass/GPS-Compass.kicad_sch (KiCad schematic)
At the start: 149 parts, among them IC1 TPS565242DRLR, IC2 KTS1605EUB-1-TR, J1 FFC2B28-12-G, J2 Conn_01x02_Pin, J3 Motor_conn, J4 FFC2B28-12-G, J5 01x10, J6 USB_TypeC, J7 Conn_01x02_Pin, M1 Stepper_Motor_bipolar, M2 Motor_DC, Q1 SI2393DS, Q2 DMG3406L, Q3 DMG3406L, Q4 DMG3406L, Q5 DMG3406L, Q6 DMG3406L, Q7 SI2365EDS, Q8 SI2365EDS, SW1 RESET, SW2 BOOT, SW3 SHIP-MODE, U1 DRV8834RGER, U2 TPS613222ADBV, U3 USBLC6-2SC6, U4 ESP32-S3-WROOM-1, U5 FUSB302B11MPX, U6 BQ25895RTW, U7 BQ25887

Commit message: asda
Connections:
- net at J3.1 (Pin_1): now also U1.4 (BOUT2); no longer U1.1 (AOUT1)
- net at J3.2 (Pin_2): now also U1.6 (BOUT1); no longer U1.3 (AOUT2)
- net at J3.3 (Pin_3): now also U1.3 (AOUT2); no longer U1.6 (BOUT1)
- net at J3.4 (Pin_4): now also U1.1 (AOUT1); no longer U1.4 (BOUT2)
Changed lines of the file:
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@@
 	)
 	(rectangle
-		(start 436.88 -31.115)
-		(end 463.55 -5.08)
-		(stroke
-			(width 0)
-			(type dash)
-			(color 0 0 0 1)
-		)
-		(fill
-			(type none)
-		)
-	)
-	(rectangle
 		(start 43.18 36.83)
 		(end 85.725 78.74)
@@
 	(symbol
 		(lib_id "Connector:Conn_01x04_Socket")
-		(at 115.57 195.58 0)
+		(at 115.57 198.12 0)
+		(mirror x)
 		(unit 1)
 		(exclude_from_sim no)
@@
 		(dnp no)
 		(property "Reference" "J3"
-			(at 117.475 195.58 0)
+			(at 117.475 198.12 0)
 			(effects
 				(font
@@
 		)
 		(property "Value" "Motor_conn"
-			(at 120.65 197.485 0)
+			(at 120.65 196.215 0)
 			(effects
 				(font
@@
 		)
 		(property "Footprint" "Connector_JST:JST_XH_S4B-XH-SM4-TB_1x04-1MP_P2.50mm_Horizontal"
-			(at 115.57 195.58 0)
+			(at 115.57 198.12 0)
 			(effects
 				(font
@@
 		)
 		(property "Datasheet" "~"
-			(at 115.57 195.58 0)
+			(at 115.57 198.12 0)
 			(effects
 				(font
@@
 		)
 		(property "Description" "Generic connector, single row, 01x04, script generated"
-			(at 115.57 195.58 0)
+			(at 115.57 198.12 0)
 			(effects
 				(font
@@
 		)
 		(instances
-			(project ""
+			(project "GPS-Compass"
 				(path "/944f168e-b689-4be9-b5f1-4ef8c625b176"
 					(reference "J3")

Commit message: changes s
Parts:
- removed J1, J4: FFC2B28-12-G, gps-compass_brd:GCT_FFC2B28-12-G, symbol gps-compass_sch:FFC2B28-12-G
- added J1: Conn_01x10_Socket, Connector_PinSocket_2.54mm:PinSocket_1x10_P2.54mm_Horizontal, symbol Connector:Conn_01x10_Socket
- added J8: FFC2B28-12-G, gps-compass_brd:GCT_FFC2B28-12-G, symbol gps-compass_sch:FFC2B28-12-G
- BZ1: footprint Buzzer_Beeper:MagneticBuzzer_StarMicronics_QMB-108 -> inset:AST0827MW-03BTRQ_MAL
- M2: footprint Connector_Wire:SolderWire-0.5sqmm_1x02_P4.6mm_D0.9mm_OD2.1mm_Relief -> Connector_Wire:SolderWire-0.1sqmm_1x02_P3.6mm_D0.4mm_OD1mm
Connections:
- net +3V3: now also J1.10 (Pin_10)
- net +5V: now also J8.10, J8.11, J8.12
- net CLK: now also J8.7
- net DBNCD_0: now also J1.2 (Pin_2)
- net DBNCD_1: now also J1.3 (Pin_3)
- net DBNCD_2: now also J1.6 (Pin_6)
- net DBNCD_3: now also J1.7 (Pin_7)
- net EN: now also J1.8 (Pin_8)
- net GND: now also J1.9 (Pin_9), J8.4, J8.6, J8.8
- net GNSS_RST: now also J1.1 (Pin_1)
- net LED_EXT: now also J1.4 (Pin_4)
- net MOSI: now also J8.9
- net MSW_ON: now also J1.5 (Pin_5)
- net ~{CS}: now also J8.5
- new net: J8.S1 (SHIELD), J8.S2 (SHIELD)
- no-connect marks 11 -> 10

Commit message: pcb updates
Parts:
- removed M1: Stepper_Motor_bipolar, symbol Motor:Stepper_Motor_bipolar
- renumbered C9 to C10, C10 to C9, J8 to J1, J1 to J4, M2 to M1, IC1 to U3, U3 to U4, U4 to U5, U5 to U6, U6 to U7, IC2 to U8, U7 to U9
Connections:
- net CLK: now also U5.20 (IO12); no longer U5.38 (IO2)
- net DBNCD_0: now also U5.28 (IO35); no longer U5.29 (IO36)
- net DBNCD_1: now also U5.29 (IO36); no longer U5.30 (IO37)
- net DBNCD_2: now also J4.5 (Pin_5), U5.31 (IO38); no longer J4.6 (Pin_6), U5.32 (IO39)
- net DBNCD_3: now also J4.6 (Pin_6), U5.32 (IO39); no longer J4.7 (Pin_7), U5.33 (IO40)
- net DIR: now also U5.34 (IO41); no longer U5.25 (IO48)
- net EN_LS: now also U5.10 (IO17); no longer U5.5 (IO5)
- net GNSS_RST: now also U5.22 (IO14); no longer U5.17 (IO9)
- net GNSS_WKP: now also U5.12 (IO8); no longer U5.11 (IO18)
- net INT_CHRG: now also U5.5 (IO5); no longer U5.4 (IO4)
- net INT_UCON: now also U5.11 (IO18); no longer U5.10 (IO17)
- net LED_EXT: now also U5.30 (IO37); no longer U5.31 (IO38)
- net MOSI: now also U5.21 (IO13); no longer U5.35 (IO42)
- net MSW_ON: now also J4.7 (Pin_7); no longer J4.5 (Pin_5)
- net NFAULT: now also U5.35 (IO42); no longer U5.28 (IO35)
- net OTG: now also U5.4 (IO4); no longer U5.34 (IO41)
- net PWM_BZ: now also U5.18 (IO10); no longer U5.12 (IO8)
- net STEP: now also U5.33 (IO40); no longer U5.24 (IO47)
- net ~{CS}: now also U5.19 (IO11); no longer U5.39 (IO1)
- net IO10 renamed IO01
- net IO01: now also U5.39 (IO1); no longer U5.18 (IO10)
- net IO11 renamed IO02
- net IO02: now also U5.38 (IO2); no longer U5.19 (IO11)
- net IO12 renamed IO48
- net IO48: now also U5.25 (IO48); no longer U5.20 (IO12)
- net LED_IO13 renamed LED_IO47
- net LED_IO47: now also U5.24 (IO47); no longer U5.21 (IO13)
- net PWM_HPTCS renamed PWM_HPTC
- net PWM_HPTC: now also U5.17 (IO9); no longer U5.22 (IO14)
Other:
- note added: "UNUSED"
- note added: "motor link aliexpress"
- moved on the sheet: C27, C28, C29, C30, C31, C32, C33, C8, C9, JP4, L4, Q3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

Commit message: To do list updated
Other:
- note added: "1. Add magnetometer and decide if IMU needed 2. Ferrite bead for motor wires 3. Add EEPROM 4. Add Magnetometer 5. Add 6 axis IMU 6. 7."
- note removed: "1. Change the UI PCB 2. 3. add test points for charger IC 4. 5. 6. 7."
Changed lines of the file:
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@@
 		)
 	)
-	(text "1. Change the UI PCB\n2. \n3. add test points for charger IC\n4. \n5. \n6. \n7."
+	(text "1. Add magnetometer and decide if IMU needed\n2. Ferrite bead for motor wires\n3. Add EEPROM\n4. Add Magnetometer\n5. Add 6 axis IMU\n6. \n7."
 		(exclude_from_sim no)
 		(at 19.685 307.975 0)

Commit message: dunnop
Parts:
- added C34, C35, C36: 100nF, Capacitor_SMD:C_0805_2012Metric_Pad1.18x1.45mm_HandSolder, symbol Device:C
- added U10: BMI088, finca:PQFN50P450X300X100-16N, symbol finca_lib:BMI088
- added U11: ICM-20948, Sensor_Motion:InvenSense_QFN-24_3x3mm_P0.4mm, symbol Sensor_Motion:ICM-20948
- added U12: 24CW1280T-I/OT, Package_TO_SOT_SMD:SOT-23-5, symbol Memory_EEPROM:24AA02-OT
Connections:
- net +3V3: now also C34.2, C35.2, C36.1, U10.10 (SDO2), U10.11 (VDDIO), U10.14 (CSB1), U10.15 (SDO1), U10.3 (VDD), U10.7 (PS), U12.4 (V_{CC})
- net GND: now also C34.1, C35.1, C36.2, U10.4 (GNDA), U10.6 (GNDIO), U12.2 (V_{SS})
- net SCL: now also U10.8 (SCL/SCK), U12.1 (SCL)
- net SDA: now also U10.9 (SDA/SDI), U12.3 (SDA)
- new net: U11.18 (GND), U11.20 (GND)
- new net ACC_INT: U10.16 (INT1)
- new net GYR_INT: U10.12 (INT3)
- no-connect marks 10 -> 15
Other:
- note added: "1. IMPLEMENT ICM-20948, put it away from the motor 2. Ferrite bead for motor wires 3. Add EEPROM 4. Move the GNSS antenna closer to the edge 5. 6. 7."
- note added: "BAD PINOUT"
- note added: "EEPROM"
- note added: "I2C Addr.: 0x50"
- note added: "INERTIAL MEASURMENT UNIT"
- note added: "Memory: 128kbit Ma freq.: 1MHz Vin: 1.6-5.5V Access time: 450ns Max supply curr.: 1mA"
- note added: "SDO pins are I2C adress setting pins, when pulled high: ACCELEROMETER: 0x19 GYROSCOPE: 0x69"
- note removed: "1. Add magnetometer and decide if IMU needed 2. Ferrite bead for motor wires 3. Add EEPROM 4. Add Magnetometer 5. Add 6 axis IMU 6. 7."

Commit message: schematic update
Parts:
- removed U11: ICM-20948, Sensor_Motion:InvenSense_QFN-24_3x3mm_P0.4mm, symbol Sensor_Motion:ICM-20948
- added C37: 10u, Capacitor_SMD:C_0805_2012Metric, symbol Device:C_Small
- added C38: 100n, Capacitor_SMD:C_0805_2012Metric, symbol Device:C_Small
- added C39: 220n, Capacitor_SMD:C_0805_2012Metric, symbol Device:C_Small
- added JP5: Jumper, Jumper:SolderJumper-3_P1.3mm_Open_RoundedPad1.0x1.5mm_NumberLabels, symbol Jumper:SolderJumper_3_Open
- added U13: LIS2MDL, Package_LGA:LGA-12_2x2mm_P0.5mm, symbol Sensor_Magnetic:LIS2MDL
Connections:
- net +3V3: now also C37.1, C38.1, JP5.3 (B), U13.10 (Vdd_IO), U13.9 (Vdd)
- net GND: now also C37.2, C38.2, C39.2, JP5.1 (A), U13.6 (GND), U13.8 (GND)
- net SCL: now also U13.1 (SCL/SPC)
- net SDA: now also U13.4 (SDA/SDI/SDO)
- new net: JP5.2 (C), U13.3 (~{CS})
- new net: C39.1, U13.5 (C1)
- new net INT_MAG: U13.7 (DRDY)
Other:
- note added: "1. Add magnetometer 2. Add IMU 3. Add EEPROM 4. Move the GNSS antenna closer to the edge 5. Pick OLED display 6. 7."
- note removed: "1. IMPLEMENT ICM-20948, put it away from the motor 2. Ferrite bead for motor wires 3. Add EEPROM 4. Move the GNSS antenna closer to the edge 5. 6. 7."
- note removed: "BAD PINOUT"
- moved on the sheet: C2, C3, C36, C5, D1, J3, JP1, JP2, JP3, R1, R2, R3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
