File: GPS-Compass_GNSS/GPS-Compass_GNSS.kicad_pcb (KiCad board)
At the start: 4 copper layers, 96 x 48.7 mm, 55 parts, among them J1 Conn_01x08_Socket, J1 JSTGH, J2 CONUFL001-SMD-T, J2 SMA_F, J3 CONSMA002, Q1 AO3401A, Q2 MMBT3904, Q4 BC337, U1 TESEO-LIV3R, U10 BGA725L6E6327FTSA1, U11 TESEO-LIV3R, U2 MAX2674EWT+T

Commit message: GNSS update
Parts:
- R41: footprint Resistor_SMD:R_0805_2012Metric -> Resistor_SMD:R_0402_1005Metric
- moved AE1 78.4 mm to (210.4, 53.8)
- moved R2 26.6 mm to (128.0, 101.5), turned to 0 degrees
- moved C15 24.1 mm to (130.8, 107.0), turned to 180 degrees
- moved R1 24.0 mm to (128.0, 99.5), turned to 0 degrees
- moved Q4 23.3 mm to (135.0, 112.5), turned to -90 degrees
- moved C33 22.7 mm to (131.7, 109.1), turned to -90 degrees
- moved J2 21.5 mm to (102.5, 107.8)
- moved L5 21.3 mm to (130.2, 108.6), turned to 180 degrees
- moved JP7 20.0 mm to (114.1, 100.5), turned to 90 degrees
- moved R29 19.4 mm to (130.5, 112.0), turned to 180 degrees
- moved C32 18.7 mm to (128.7, 109.1), turned to -90 degrees
- moved JP8 18.1 mm to (116.6, 100.5), turned to 90 degrees
- moved R33 15.9 mm to (135.0, 109.0), turned to 180 degrees
- moved D6 14.3 mm to (135.0, 107.0), turned to 180 degrees
- moved JP6 13.5 mm to (120.8, 100.5), turned to 90 degrees
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Routing:
- net Net-(Q4-C): track 3.36 -> 0.00 mm
- net Net-(D6-K): track 2.01 -> 0.00 mm
- net Net-(FL1-INPUT): track 0.00 -> 1.45 mm
- net Net-(Q4-B): track 3.67 -> 4.31 mm

Commit message: GNSS update
Parts:
- removed U1: TESEO-LIV3R, TESEO-LIV3R:TESEOLIV3R
- moved JP7 10.9 mm to (124.8, 98.2), turned to -90 degrees
- moved JP5 8.59 mm to (115.2, 98.2)
- moved JP8 6.08 mm to (122.2, 98.2), turned to -90 degrees
- moved R1 4.31 mm to (130.8, 102.8)
- moved R2 4.31 mm to (130.8, 104.8)
- moved JP6 3.37 mm to (118.2, 98.2)
- moved C29 0.48 mm to (112.8, 109.2)
- moved R41 0.43 mm to (110.8, 109.2)
- moved FL1 0.07 mm to (113.5, 107.8)
- moved U10 0.07 mm to (111.5, 107.8)
Connections:
- J1 pad 1: GND -> +3V3
- J1 pad 2: +3V3 -> GNSS_TX
- J1 pad 3: SCL -> GNSS_RX
- J1 pad 5: GNSS_TX -> SCL
- J1 pad 6: GNSS_RX -> GNSS_WKP
- J1 pad 7: GNSS_WKP -> GNSS_RST
- J1 pad 8: GNSS_RST -> GND
Routing:
- net GNSS_RX: track 0.00 -> 4.54 mm
- net VCC_RF: track 3.26 -> 5.11 mm
- net RF_IN: track 0.00 -> 1.62 mm
- net Net-(U10-AI): track 0.00 -> 1.09 mm
- net ANT_OFF: track 0.00 -> 1.06 mm
- net Net-(FL1-OUTPUT): track 0.00 -> 1.02 mm

Commit message: gnss module
Parts:
- removed AE1: Antenna, gps-compass_brd:ANT2525B00DT1516S
- removed C1: 2u2, Capacitor_SMD:C_0603_1608Metric
- removed C2: 100n, Capacitor_SMD:C_0402_1005Metric
- removed C3: 10n, Capacitor_SMD:C_0402_1005Metric
- removed C4, C5: 56p, Capacitor_SMD:C_0402_1005Metric
- removed C6: 10p, Capacitor_SMD:C_0402_1005Metric
- removed C7, C8: 100p, Capacitor_SMD:C_0402_1005Metric
- removed the D1 at (74.8, 116.0)
- removed D2: BLUE, LED_SMD:LED_0603_1608Metric
- removed the J1 at (84.8, 122.5)
- removed the J2 at (54.3, 115.8)
- removed J3: CONSMA002, CONSMA002:CONSMA002
- removed L1: 27n, Inductor_SMD:L_0402_1005Metric
- removed L2: 88n, Inductor_SMD:L_0402_1005Metric
- removed Q1: AO3401A, Package_TO_SOT_SMD:SOT-23
- removed Q2: MMBT3904, Package_TO_SOT_SMD:SOT-23
- removed the R1 at (78.0, 116.0)
- removed the R2 at (74.4, 119.2)
- removed the R3 at (75.0, 123.2)
- removed R4: 10k, Resistor_SMD:R_0603_1608Metric
- removed R5, R6: 22, Resistor_SMD:R_0402_1005Metric
- removed R7: 1k, Resistor_SMD:R_0402_1005Metric
- removed R8: 2k2, Resistor_SMD:R_0603_1608Metric
- removed U2: MAX2674EWT+T, SchmillipKiCADLibrary:MAX2674EWT+T
- moved JP5 4.81 mm to (120.0, 97.5)
- moved D6 4.00 mm to (135.0, 103.0)
- moved R33 4.00 mm to (135.0, 105.0)
- moved R2 3.75 mm to (130.8, 101.0)
- moved JP8 2.95 mm to (125.1, 97.5)
- moved Q4 2.88 mm to (135.0, 109.6)
- moved D1 2.40 mm to (135.0, 97.6)
- moved R3 2.40 mm to (135.0, 99.6)
- moved JP7 2.28 mm to (122.6, 97.5)
- moved R29 2.10 mm to (130.6, 109.9)
- moved C15 2.00 mm to (130.8, 105.0)
- moved C28 2.00 mm to (107.8, 105.8)
- moved C30 2.00 mm to (115.5, 105.5)
- moved C31 2.00 mm to (116.1, 109.3)
- moved C32 2.00 mm to (128.7, 107.1)
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Connections:
- J1 pad 2: GNSS_TX -> GNSS_RX
- J1 pad 3: GNSS_RX -> GNSS_TX
- J1 pad 4: SDA -> SCL
- J1 pad 5: SCL -> SDA
Routing:
- net +3V3: track 43.7 -> 4.20 mm, vias 9 -> 0
- net GND: track 45.8 -> 10.6 mm, vias 26 -> 37
- net GNSS_WKP: track 0.00 -> 31.8 mm, vias 0 -> 1
- net GNSS_RST: track 0.00 -> 26.7 mm, vias 0 -> 3
- net GPS_!RST: track 23.6 -> 0.00 mm, vias 2 -> 0
- net Net-(JP5-A): track 0.00 -> 16.7 mm
- net Net-(JP7-B): track 0.00 -> 16.5 mm
- net UART_TX: track 16.5 -> 0.00 mm
- net Net-(JP6-A): track 0.00 -> 16.0 mm
- net Net-(JP8-B): track 0.00 -> 14.5 mm
- net GPS_WAKEUP: track 12.8 -> 0.00 mm, vias 2 -> 0
- net GPS_PPS: track 11.7 -> 0.00 mm
- net UART_RX: track 9.70 -> 0.00 mm
- net ANT_OFF: track 1.06 -> 9.78 mm, vias 0 -> 2
- net ANT_ACTIVE: track 8.13 -> 0.00 mm
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- added copper zone on F.Cu, net +3V3
- added copper zone on F.Cu, net /VCC_GNSS
- added copper zone on B.Cu, net GND
- added copper zone on F.Cu, net GND
- removed copper zone on In1.Cu, net GND
- removed copper zone on In2.Cu, net GND
Other:
- board size 96 x 48.7 mm -> 40.5 x 34.4 mm

Commit message: GNSS and Mian ocb
Parts:
- removed J1: Conn_01x08_Socket, Connector_PinSocket_2.54mm:PinSocket_1x08_P2.54mm_Horizontal
- added C1: 100n, Capacitor_SMD:C_0805_2012Metric, F.Cu at (169.9, 110.5)
- added C10: 10uF, Capacitor_SMD:C_0805_2012Metric, F.Cu at (108.2, 33.2)
- added C11: 22uF, Capacitor_SMD:C_0805_2012Metric, F.Cu at (102.2, 22.3)
- added C12: 22uF, Capacitor_SMD:C_0805_2012Metric, F.Cu at (104.2, 22.3)
- added C13: 1uF, Capacitor_SMD:C_0805_2012Metric, F.Cu at (116.2, 9.47)
- added C14: 47nF, Capacitor_SMD:C_0805_2012Metric, F.Cu at (109.7, 7.47)
- added C15: 4.7uF, Capacitor_SMD:C_0805_2012Metric, F.Cu at (111.0, -0.03)
- added C16: 10uF, Capacitor_SMD:C_0805_2012Metric, F.Cu at (112.7, 11.5)
- added C17: 10uF, Capacitor_SMD:C_0805_2012Metric, F.Cu at (110.4, 2.73)
- added C18: 22uF, Capacitor_SMD:C_0805_2012Metric, F.Cu at (125.7, 20.1)
- added C20: 10nF, Capacitor_SMD:C_0402_1005Metric, F.Cu at (108.2, 35.5)
- added C21: 100nF, Capacitor_SMD:C_0805_2012Metric, F.Cu at (110.2, 33.2)
- added C22: 100nF, Capacitor_SMD:C_0805_2012Metric, F.Cu at (112.7, 9.47)
- added C23: 44uF, Capacitor_SMD:C_0805_2012Metric, F.Cu at (109.7, 5.47)
- added C26: 100nF, Capacitor_SMD:C_0805_2012Metric, F.Cu at (101.5, -7.15)
- added C27: 100nF, Capacitor_SMD:C_0805_2012Metric, F.Cu at (110.8, -8.95)
- added C3: 10uF, Capacitor_SMD:C_0805_2012Metric, F.Cu at (125.3, 24.2)
- added C4: 10uF, Capacitor_SMD:C_0805_2012Metric, F.Cu at (107.0, 18.9)
- added C5: 100nF, Capacitor_SMD:C_0805_2012Metric, F.Cu at (120.6, 25.9)
- added C6: 100nF, Capacitor_SMD:C_0805_2012Metric, F.Cu at (123.3, 24.2)
- added C7: 100nF, Capacitor_SMD:C_0805_2012Metric, F.Cu at (106.2, 22.3)
- added C8: 22uF, Capacitor_SMD:C_0805_2012Metric, F.Cu at (127.7, 20.1)
- added C9: 100nF, Capacitor_SMD:C_0805_2012Metric, F.Cu at (109.0, 18.9)
- added D3: LED, LED_SMD:LED_0805_2012Metric, F.Cu at (124.8, 4.47)
- added D4: LED, LED_SMD:LED_0805_2012Metric, F.Cu at (124.8, 0.47)
- added D5: LED, LED_SMD:LED_0805_2012Metric, F.Cu at (124.8, 8.47)
- added H1: MountingHole_Pad, MountingHole:MountingHole_2.2mm_M2_Pad_Via, F.Cu at (86.0, 124.0)
- added H1: Mounting Hole M3, MountingHole:MountingHole_3.2mm_M3_Pad, F.Cu at (96.8, 45.6)
- added H2: Mounting Hole M3, MountingHole:MountingHole_3.2mm_M3_Pad, F.Cu at (130.8, 45.6)
- added H2: MountingHole_Pad, MountingHole:MountingHole_2.2mm_M2_Pad_Via, F.Cu at (86.2, 88.8)
- added H3: MountingHole_Pad, MountingHole:MountingHole_2.2mm_M2_Pad_Via, F.Cu at (136.5, 113.9)
- added H3: Mounting Hole M3, MountingHole:MountingHole_3.2mm_M3_Pad_Via, F.Cu at (187.8, -26.4)
- added H4: Mounting Hole M3, MountingHole:MountingHole_3.2mm_M3_Pad_Via, F.Cu at (96.8, -26.4)
- added H4: MountingHole_Pad, MountingHole:MountingHole_2.2mm_M2_Pad_Via, F.Cu at (101.1, 113.9)
- added IC1: TPS565242DRLR, Package_TO_SOT_SMD:SOT-563, F.Cu at (111.0, 19.4)
- added J2: USB_TypeC, sumec_brd:HRO_TYPE-C-31-M-12, F.Cu at (93.3, -10.2)
- added J3: Conn_01x10_Socket, Connector_PinSocket_2.54mm:PinSocket_1x10_P2.54mm_Horizontal, F.Cu at (130.2, 93.2)
- added JP1: Jumper, Jumper:SolderJumper-3_P1.3mm_Open_RoundedPad1.0x1.5mm_NumberLabels, F.Cu at (166.8, -6.90)
- added JP1: Jumper_2_Small_Open, Jumper:SolderJumper-2_P1.3mm_Open_RoundedPad1.0x1.5mm, F.Cu at (167.7, 103.2)
- added JP3: Jumper, Jumper:SolderJumper-2_P1.3mm_Open_RoundedPad1.0x1.5mm, F.Cu at (105.8, 5.72)
- added JP4: Jumper, Jumper:SolderJumper-3_P1.3mm_Open_RoundedPad1.0x1.5mm_NumberLabels, F.Cu at (113.5, 34.0)
- added L1: 1.5uH, Inductor_SMD:L_Vishay_IHLP-1212, F.Cu at (109.7, 22.4)
- added L2: 3.3uH, Inductor_SMD:L_Vishay_IHLP-1616, F.Cu at (121.5, 20.1)
- added L3: 1uH, Inductor_SMD:L_Walsin_WLFM201609x, F.Cu at (112.4, 13.6)
- added Q3: Q_NMOS_GSD, Package_TO_SOT_SMD:SOT-23-3, F.Cu at (109.3, 29.6)
- added R10: 10k, Resistor_SMD:R_0805_2012Metric, F.Cu at (120.8, 9.72)
- added R11: 383R, Resistor_SMD:R_0805_2012Metric, F.Cu at (117.6, 0.28)
- added R12: 300R, Resistor_SMD:R_0805_2012Metric, F.Cu at (115.7, 0.28)
- added R13: 9.5R, Resistor_SMD:R_0805_2012Metric, F.Cu at (113.8, 0.28)
- added R15: 5.23k, Resistor_SMD:R_0805_2012Metric, F.Cu at (119.8, 3.88)
- added R16: 30.1k, Resistor_SMD:R_0805_2012Metric, F.Cu at (119.8, 5.78)
- added R17: R(SET), Resistor_SMD:R_0805_2012Metric, F.Cu at (102.8, 30.1)
- added R18: R(SET), Resistor_SMD:R_0805_2012Metric, F.Cu at (104.8, 30.1)
- added R19: 10k, Resistor_SMD:R_0805_2012Metric, F.Cu at (112.3, 29.7)
- added R23: 100k, Resistor_SMD:R_0805_2012Metric, F.Cu at (101.5, -13.2)
- added R27: 15R, Resistor_SMD:R_0805_2012Metric, F.Cu at (101.5, -11.2)
- added R28: 15R, Resistor_SMD:R_0805_2012Metric, F.Cu at (101.5, -9.15)
- added R3: 45k, Resistor_SMD:R_0805_2012Metric, F.Cu at (104.2, 18.9)
- added R30: 2.2k, Resistor_SMD:R_0805_2012Metric, F.Cu at (128.3, 4.47)
- added R31: 2.2k, Resistor_SMD:R_0805_2012Metric, F.Cu at (128.3, 0.47)
- added R32: 2.2k, Resistor_SMD:R_0805_2012Metric, F.Cu at (128.3, 8.47)
- added R34: 10k, Resistor_SMD:R_0805_2012Metric, F.Cu at (128.3, 6.47)
- added R35: 10k, Resistor_SMD:R_0805_2012Metric, F.Cu at (128.3, 2.48)
- added R36: 10k, Resistor_SMD:R_0805_2012Metric, F.Cu at (128.3, 10.5)
- added R4: 100k, Resistor_SMD:R_0805_2012Metric, F.Cu at (124.3, 26.9)
- added R4: 10k, Resistor_SMD:R_0805_2012Metric, F.Cu at (167.7, 100.0)
- added R5: 52.3k, Resistor_SMD:R_0805_2012Metric, F.Cu at (124.3, 28.8)
- added R6: 10k, Resistor_SMD:R_0805_2012Metric, F.Cu at (102.2, 18.9)
- added R8: 52.3k, Resistor_SMD:R_0805_2012Metric, F.Cu at (120.7, 29.9)
- added R9: 10k, Resistor_SMD:R_0805_2012Metric, F.Cu at (120.6, 27.9)
- added REF**: PinHeader_1x10_P2.54mm_Horizontal, Connector_PinHeader_2.54mm:PinHeader_1x10_P2.54mm_Horizontal, F.Cu at (125.1, 44.7)
- added SW1: GNSS_RST, Button_Switch_SMD:SW_SPST_B3U-1000P, F.Cu at (156.0, 102.8)
- added TH1: 10k NTC, Resistor_SMD:R_0402_1005Metric, F.Cu at (119.8, 1.88)
- added TP1: TestPoint, TestPoint:TestPoint_Pad_D1.0mm, F.Cu at (164.0, 100.0)
- added TP2: TestPoint, TestPoint:TestPoint_Pad_D1.0mm, F.Cu at (164.0, 103.1)
- added TP3: TestPoint, TestPoint:TestPoint_Pad_D1.0mm, F.Cu at (164.0, 106.1)
- added TP4: TestPoint, TestPoint:TestPoint_Pad_D1.0mm, F.Cu at (164.0, 109.2)
- added U1: ESP32-S3-WROOM-1, PCM_Espressif:ESP32-S3-WROOM-1, F.Cu at (139.8, -13.7)
- added U2: AP62300Z6, Package_TO_SOT_SMD:SOT-563, F.Cu at (121.3, 23.7)
- added U3: BQ25887, Package_DFN_QFN:VQFN-24-1EP_4x4mm_P0.5mm_EP2.5x2.5mm, F.Cu at (114.1, 5.85)
- added U4: DRV8834RGER, gps-compass_brd:DRIVER_DRV8834RGER, F.Cu at (104.8, 34.5)
- added U9: USBLC6-2SC6, Package_TO_SOT_SMD:TSOT-23-6_HandSoldering, F.Cu at (106.3, -10.2)
- C15: value 100nF -> 100n
- C28, C30: value 120pF -> 120p
- C29: value 1nF -> 1n
- C31, C32: value 56nF -> 56n
- C33: value 10nF -> 10n
- L4: value 5.6nH -> 5.6n
- moved Q4 2.37 mm to (135.0, 107.2)
- moved D6 0.23 mm to (135.0, 102.8)
- moved R33 0.23 mm to (135.0, 104.8)
Connections:
- C32 pad 1: /VCC_GNSS -> Net-(JP1-A)
- L5 pad 2: /VCC_GNSS -> Net-(JP1-A)
- U11 pad 6: /VCC_GNSS -> Net-(JP1-B)
- U11 pad 7: /VCC_GNSS -> Net-(JP1-A)
- U11 pad 8: /VCC_GNSS -> Net-(JP1-A)
Routing:
- net SWC: track 0.00 -> 8.49 mm
- net SNS: track 0.00 -> 7.26 mm
- net D- IN: track 0.00 -> 6.28 mm
- net VBATT: track 0.00 -> 5.77 mm
- net D+ IN: track 0.00 -> 4.76 mm
- net LDO: track 0.00 -> 4.51 mm
- net Net-(U3-ILIM): track 0.00 -> 4.47 mm
- net /POWER/SW: track 0.00 -> 4.14 mm
- net TS: track 0.00 -> 3.61 mm
- net Net-(U3-MID): track 0.00 -> 3.43 mm
- net Net-(U3-CBSET): track 0.00 -> 2.75 mm
- net Net-(R27-Pad2): track 0.00 -> 2.15 mm
- net Net-(R28-Pad2): track 0.00 -> 2.15 mm
- net VM: track 0.00 -> 2.09 mm
- net Net-(Q4-C): track 4.88 -> 3.07 mm
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- added copper zone on F.Cu, net Net-(JP1-A)
- removed copper zone on F.Cu, net /VCC_GNSS
Other:
- board size 40.5 x 34.4 mm -> 100 x 146.2 mm
- board text added: "MOTOR"
