File: GPS-Compass_GNSS/GPS-Compass_GNSS.kicad_pcb (KiCad board)
At the start: 2 copper layers, 40.5 x 29.6 mm, 38 parts, among them J3 01x10, J4 636101112001, Q1 MMBT3904, SW1 GNSS_RST, U1 BGA725L6E6327FTSA1, U2 TESEO-LIV3R

Commit message: PCB updates
Other:
- board text added: "u.fl - F"
- board text removed: "SMA-F"
Changed lines of the file:
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@@
 		)
 	)
-	(gr_text "SMA-F"
-		(at 103 113.9 0)
+	(gr_text "u.fl - F"
+		(at 102.909393 113.906006 0)
 		(layer "F.SilkS")
 		(effects
@@
 			)
 		)
-		(render_cache "SMA-F" 0
-			(polygon
-				(pts
-					(xy 101.289751 114.325746) (xy 101.219263 114.322139) (xy 101.150715 114.311397) (xy 101.084435 114.293574)
-					(xy 101.023282 114.269387) (xy 100.966376 114.238657) (xy 100.916059 114.20277) (xy 101.002826 114.048286)
-					(xy 101.064123 114.089868) (xy 101.135328 114.121254) (xy 101.211538 114.140537) (xy 101.289751 114.14696)
-					(xy 101.350293 114.142932) (xy 101.396678 114.132092) (xy 101.431839 114.115819) (xy 101.460328 114.091726)
-					(xy 101.476755 114.062943) (xy 101.482397 114.027831) (xy 101.482397 114.027098) (xy 101.475683 113.98808)
-					(xy 101.457118 113.961153) (xy 101.428776 113.941734) (xy 101.390501 113.927325) (xy 101.30068 113.908885)
-					(xy 101.183139 113.88672) (xy 101.125752 113.869301) (xy 101.07384 113.844344) (xy 101.029223 113.809417)
-					(xy 100.993606 113.761301) (xy 100.977575 113.724041) (xy 100.967052 113.676764) (xy 100.963198 113.617137)
-					(xy 100.963198 113.616404) (xy 100.969702 113.544962) (xy 100.988108 113.485003) (xy 101.017654 113.434287)
-					(xy 101.058819 113.391273) (xy 101.108249 113.358202) (xy 101.168317 113.333368) (xy 101.241157 113.317393)
-					(xy 101.329379 113.31165) (xy 101.409825 113.318262) (xy 101.493266 113.338639) (xy 101.573737 113.371364)
-					(xy 101.64836 113.415514) (xy 101.569103 113.574028) (xy 101.510042 113.538102) (xy 101.449241 113.512051)
-					(xy 101.386946 113.495649) (xy 101.329379 113.490436) (xy 101.272362 113.494134) (xy 101.228891 113.504057)
-					(xy 101.196145 113.51889) (xy 101.16948 113.54092) (xy 101.15422 113.567018) (xy 101.149006 113.598635)
-					(xy 101.149006 113.599368) (xy 101.152437 113.630015) (xy 101.161899 113.653597) (xy 101.176971 113.671786)
-					(xy 101.208226 113.692713) (xy 101.250061 113.708361) (xy 101.347087 113.730526) (xy 101.461148 113.757515)
-					(xy 101.515807 113.777232) (xy 101.565012 113.803677) (xy 101.607073 113.839038) (xy 101.640178 113.886353)
-					(xy 101.655024 113.922503) (xy 101.664692 113.96742) (xy 101.668205 114.023007) (xy 101.668205 114.024412)
-					(xy 101.661538 114.094504) (xy 101.642605 114.153601) (xy 101.612028 114.203898) (xy 101.569103 114.246856)
-					(xy 101.518162 114.279529) (xy 101.456168 114.304155) (xy 101.380919 114.320032)
-				)
-			)
-			(polygon
-				(pts
-					(xy 102.26141 113.991439) (xy 102.450637 113.322397) (xy 102.6972 113.322397) (xy 102.6972 114.315)
-					(xy 102.527146 114.315) (xy 102.527146 113.544291) (xy 102.533924 113.58795) (xy 102.344025 114.204419)
-					(xy 102.178733 114.204419) (xy 101.988835 113.601627) (xy 101.995673 113.544291) (xy 101.995673 114.315)
-					(xy 101.825558 114.315) (xy 101.825558 113.322397) (xy 102.072183 113.322397)
-				)
-			)
-			(polygon
-				(pts
-					(xy 102.80656 114.315) (xy 103.186357 113.322397) (xy 103.305243 113.322397) (xy 103.68504 114.315)
-					(xy 103.48354 114.315) (xy 103.245769 113.637103) (xy 103.00806 114.315)
-				)
-			)
-			(polygon
-				(pts
-					(xy 102.988948 114.154776) (xy 102.988948 113.974036) (xy 103.511506 113.974036) (xy 103.511506 114.154776)
-				)
-			)
-			(polygon
-				(pts
-					(xy 103.773639 113.869501) (xy 104.260049 113.869501) (xy 104.260049 114.05024) (xy 103.773639 114.05024)
-				)
-			)
-			(polygon
-				(pts
-					(xy 104.458496 114.315) (xy 104.458496 113.322397) (xy 104.645647 113.322397) (xy 104.645647 114.315)
-				)
-			)
-			(polygon
-				(pts
-					(xy 104.526823 113.920303) (xy 104.526823 113.739563) (xy 105.035703 113.739563) (xy 105.035703 113.920303)
-				)
-			)
-			(polygon
-				(pts
-					(xy 104.526823 113.503136) (xy 104.526823 113.322397) (xy 105.110869 113.322397) (xy 105.110869 113.503136)
+		(render_cache "u.fl - F" 0
+			(polygon
+				(pts
+					(xy 101.339033 114.321006) (xy 101.339033 113.613678) (xy 101.525513 113.613678) (xy 101.525513 114.321006)
+				)
+			)
+			(polygon
+				(pts
+					(xy 101.119093 113.613678) (xy 101.119093 114.043424) (xy 101.122621 114.076262) (xy 101.132428 114.102179)
+					(xy 101.148097 114.122741) (xy 101.169118 114.137946) (xy 101.195787 114.147543) (xy 101.229735 114.151012)
+					(xy 101.263609 114.14745) (xy 101.290008 114.137611) (xy 101.31064 114.122009) (xy 101.325858 114.100951)
+					(xy 101.335521 114.073878) (xy 101.339033 114.039027) (xy 101.34862 114.194671) (xy 101.32451 114.244016)
+					(xy 101.286094 114.289498) (xy 101.254021 114.312611) (xy 101.215986 114.326772) (xy 101.170323 114.331752)
+					(xy 101.114222 114.326723) (xy 101.067227 114.31251) (xy 101.027576 114.289745) (xy 100.99404 114.258113)
+					(xy 100.968158 114.220003) (xy 100.948779 114.173876) (xy 100.936344 114.118135) (xy 100.931881 114.050812)
+					(xy 100.931881 113.613678)
+				)
+			)
+			(polygon
+				(pts
+					(xy 101.678836 114.321006) (xy 101.678836 114.133427) (xy 101.865987 114.133427) (xy 101.865987 114.321006)
+				)
+			)
+			(polygon
+				(pts
+					(xy 102.046605 114.321006) (xy 102.046605 113.516164) (xy 102.052109 113.455209) (xy 102.066941 113.409525)
+					(xy 102.089653 113.375541) (xy 102.121483 113.350537) (xy 102.164846 113.33439) (xy 102.223498 113.328403)
+					(xy 102.353313 113.328403) (xy 102.353313 113.495465) (xy 102.274056 113.495465) (xy 102.255558 113.499615)
+					(xy 102.243343 113.511524) (xy 102.236249 113.528611) (xy 102.233756 113.549381) (xy 102.233756 114.321006)
+				)
+			)
+			(polygon
+				(pts
+					(xy 101.971439 113.773902) (xy 101.971439 113.613678) (xy 102.353313 113.613678) (xy 102.353313 113.773902)
+				)
+			)
+			(polygon
+				(pts
+					(xy 102.656846 113.328403) (xy 102.656846 114.086349) (xy 102.660754 114.109419) (xy 102.671683 114.125978)
+					(xy 102.688823 114.136437) (xy 102.71351 114.140266) (xy 102.744956 114.140266) (xy 102.744956 114.321006)
+					(xy 102.649335 114.321006) (xy 102.594435 114.315033) (xy 102.551127 114.298426) (xy 102.516772 114.271852)
+					(xy 102.49147 114.236343) (xy 102.475442 114.191078) (xy 102.469634 114.133244) (xy 102.469634 113.328403)
+				)
+			)
+			(polygon
+				(pts
+					(xy 103.249257 113.875507) (xy 103.735666 113.875507) (xy 103.735666 114.056246) (xy 103.249257 114.056246)
+				)
+			)
+			(polygon
+				(pts
+					(xy 104.309271 114.321006) (xy 104.309271 113.328403) (xy 104.496422 113.328403) (xy 104.496422 114.321006)
+				)
+			)
+			(polygon
+				(pts
+					(xy 104.377598 113.926309) (xy 104.377598 113.745569) (xy 104.886478 113.745569) (xy 104.886478 113.926309)
+				)
+			)
+			(polygon
+				(pts
+					(xy 104.377598 113.509142) (xy 104.377598 113.328403) (xy 104.961643 113.328403) (xy 104.961643 113.509142)
 				)
 			)
@@
 			(keep_text_aligned yes)
 		)
-		(gr_text "40,5"
+		(gr_text "40.5"
 			(at 118.889668 129.351494 0)
 			(layer "Dwgs.User")
@@
 			(keep_text_aligned yes)
 		)
-		(gr_text "33,8"
+		(gr_text "33.8"
 			(at 118.8897 126.351494 0)
 			(layer "Dwgs.User")
@@
 			(keep_text_aligned yes)
 		)
-		(gr_text "29,75"
+		(gr_text "29.75"
 			(at 144.489668 108.376494 90)
 			(layer "Dwgs.User")

Commit message: 3d and PCB
Other:
- outline, holes or cut-outs redrawn

Commit message: UPDATES
Parts:
- moved H2 33.8 mm to (102.0, 119.8)
- moved H1 33.7 mm to (135.7, 119.8)
- moved G*** 1.07 mm to (119.6, 109.0)
- moved J3 0.18 mm to (107.5, 97.6)
Other:
- outline, holes or cut-outs redrawn
- board text added: "OwO"
- board text added: "made by a good boy :3"
- board text removed: "made by bismarx"
