File: GPS-Compass_GNSS/GPS-Compass_GNSS.kicad_pcb (KiCad board)
At the start: 2 copper layers, 40.5 x 29.6 mm, 38 parts, among them J3 01x10, J4 636101112001, Q1 MMBT3904, SW1 GNSS_RST, U1 BGA725L6E6327FTSA1, U2 TESEO-LIV3R

Commit message: pls dont break
Routing:
- net /GNSS_RX: track 4.94 -> 5.74 mm
- net /GNSS_TX: track 4.65 -> 5.42 mm
Changed lines of the file:
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@@
+	)
+	(segment
+		(start 122.088174 99.5)
+		(end 123 99.5)
+		(width 0.2)
+		(layer "F.Cu")
+		(net 12)
+	)
+	(segment
+		(start 123.75 100.25)
+		(end 123.75 101.1)
+		(width 0.2)
+		(layer "F.Cu")
+		(net 12)
 	)
 	(segment
@@
 	)
 	(segment
-		(start 120.238174 97.75)
-		(end 123.588174 101.1)
-		(width 0.25)
+		(start 123 99.5)
+		(end 123.75 100.25)
+		(width 0.2)
+		(layer "F.Cu")
+		(net 12)
+	)
+	(segment
+		(start 120.164668 97.576494)
+		(end 122.088174 99.5)
+		(width 0.2)
 		(layer "F.Cu")
 		(net 12)
@@
 	)
 	(segment
+		(start 120.75 101.1)
+		(end 120.75 100.25)
+		(width 0.2)
+		(layer "F.Cu")
+		(net 14)
+	)
+	(segment
+		(start 120.75 100.25)
+		(end 120.25 99.75)
+		(width 0.2)
+		(layer "F.Cu")
+		(net 14)
+	)
+	(segment
 		(start 120.75 100.801826)
 		(end 120.75 101.1)
@@
 	)
 	(segment
+		(start 120.25 99.75)
+		(end 119.798174 99.75)
+		(width 0.2)
+		(layer "F.Cu")
+		(net 14)
+	)
+	(segment
+		(start 119.798174 99.75)
+		(end 117.624668 97.576494)
+		(width 0.2)
+		(layer "F.Cu")
+		(net 14)
+	)
+	(segment
 		(start 117.66 97.75)
 		(end 117.698174 97.75)
-		(width 0.25)
-		(layer "F.Cu")
-		(net 14)
-	)
-	(segment
-		(start 117.698174 97.75)
-		(end 120.75 100.801826)
 		(width 0.25)
 		(layer "F.Cu")
@@
 	)
 	(zone
+		(net 4)
+		(net_name "/VCC_RF")
+		(layer "F.Cu")
+		(name "$teardrop_padvia$")
+		(hatch none 0.1)
+		(priority 30002)
+		(attr
+			(teardrop
+				(type padvia)
+			)
+		)
+		(connect_pads yes
+			(clearance 0)
+		)
+		(min_thickness 0.0254)
+		(filled_areas_thickness no)
+		(fill yes
+			(thermal_gap 0.5)
+			(thermal_bridge_width 0.5)
+			(island_removal_mode 1)
+			(island_area_min 10)
+		)
+		(polygon
+			(pts
+				(xy 112.189668 109.15) (xy 112.189668 108.95) (xy 112.064668 108.925) (xy 111.938668 109.05) (xy 112.064668 109.175)
+			)
+		)
+	)
+	(zone
 		(net 3)
 		(net_name "GND")
@@
 			(pts
 				(xy 132.535547 102.328884) (xy 132.535547 103.828884) (xy 129.69766 101.412441) (xy 129.69766 99.912441)
+			)
+		)
+	)
+	(zone
+		(net 28)
+		(net_name "Net-(U2-VBATT)")
+		(layer "F.Cu")
+		(hatch edge 0.5)
+		(priority 1)
+		(connect_pads yes
+			(clearance 0.2)
+		)
+		(min_thickness 0.25)
+		(filled_areas_thickness no)
+		(fill yes
+			(thermal_gap 0.5)
+			(thermal_bridge_width 0.5)
+		)
+		(polygon
+			(pts
+				(xy 128.139668 108.35) (xy 128.139668 109.45) (xy 130.252418 109.45) (xy 130.252418 110.25018) (xy 128.14263 110.254546)
+				(xy 128.139668 110.33) (xy 128.139668 111.35) (xy 126.439668 111.35) (xy 126.439668 108.35)
+			)
+		)
+	)
+	(zone
+		(net 0)
+		(net_name "")
+		(layer "F.Cu")
+		(hatch edge 0.5)
+		(connect_pads
+			(clearance 0)
+		)
+		(min_thickness 0.25)
+		(filled_areas_thickness no)
+		(keepout
+			(tracks allowed)
+			(vias allowed)
+			(pads allowed)
+			(copperpour not_allowed)
+			(footprints allowed)
+		)
+		(placement
+			(enabled no)
+			(sheetname "/")
+		)
+		(fill
+			(thermal_gap 0.5)
+			(thermal_bridge_width 0.5)
+		)
+		(polygon
+			(pts
+				(xy 127.239668 115.55) (xy 127.239668 116) (xy 128.689668 116) (xy 128.689668 118) (xy 124.639668 118)
+				(xy 124.639668 116) (xy 127.239668 116) (xy 127.239668 115.55) (xy 124.139668 115.55) (xy 124.139668 118.45)
+				(xy 129.139668 118.45) (xy 129.139668 115.55)
 			)
 		)
@@
 	)
 	(zone
-		(net 28)
-		(net_name "Net-(U2-VBATT)")
-		(layer "F.Cu")
-		(hatch edge 0.5)
-		(priority 1)
-		(connect_pads yes
-			(clearance 0.2)
-		)
-		(min_thickness 0.25)
-		(filled_areas_thickness no)
-		(fill yes
-			(thermal_gap 0.5)
-			(thermal_bridge_width 0.5)
-		)
-		(polygon
-			(pts
-				(xy 128.139668 108.35) (xy 128.139668 109.45) (xy 130.252418 109.45) (xy 130.252418 110.25018) (xy 128.14263 110.254546)
-				(xy 128.139668 110.33) (xy 128.139668 111.35) (xy 126.439668 111.35) (xy 126.439668 108.35)
-			)
-		)
-	)
-	(zone
-		(net 0)
-		(net_name "")
-		(layer "F.Cu")
-		(hatch edge 0.5)
-		(connect_pads
+		(net 6)
+		(net_name "Net-(FL1-OUTPUT)")
+		(layer "F.Cu")
+		(name "$teardrop_padvia$")
+		(hatch none 0.1)
+		(priority 30001)
+		(attr
+			(teardrop
+				(type padvia)
+			)
+		)
+		(connect_pads yes
 			(clearance 0)
 		)
-		(min_thickness 0.25)
-		(filled_areas_thickness no)
-		(keepout
-			(tracks allowed)
-			(vias allowed)
-			(pads allowed)
-			(copperpour not_allowed)
-			(footprints allowed)
-		)
-		(placement
-			(enabled no)
-			(sheetname "/")
-		)
-		(fill
-			(thermal_gap 0.5)
-			(thermal_bridge_width 0.5)
-		)
-		(polygon
-			(pts
-				(xy 127.239668 115.55) (xy 127.239668 116) (xy 128.689668 116) (xy 128.689668 118) (xy 124.639668 118)
-				(xy 124.639668 116) (xy 127.239668 116) (xy 127.239668 115.55) (xy 124.139668 115.55) (xy 124.139668 118.45)
-				(xy 129.139668 118.45) (xy 129.139668 115.55)
+		(min_thickness 0.0254)
+		(filled_areas_thickness no)
+		(fill yes
+			(thermal_gap 0.5)
+			(thermal_bridge_width 0.5)
+			(island_removal_mode 1)
+			(island_area_min 10)
+		)
+		(polygon
+			(pts
+				(xy 114.699668 108.6) (xy 114.699668 108.9) (xy 115.037143 109.03) (xy 115.260668 108.75) (xy 115.037143 108.47)
+			)
+		)
+	)
+	(zone
+		(net 8)
+		(net_name "Net-(FL1-INPUT)")
+		(layer "F.Cu")
+		(name "$teardrop_padvia$")
+		(hatch none 0.1)
+		(priority 30003)
+		(attr
+			(teardrop
+				(type padvia)
+			)
+		)
+		(connect_pads yes
+			(clearance 0)
+		)
+		(min_thickness 0.0254)
+		(filled_areas_thickness no)
+		(fill yes
+			(thermal_gap 0.5)
+			(thermal_bridge_width 0.5)
+			(island_removal_mode 1)
+			(island_area_min 10)
+		)
+		(polygon
+			(pts
+				(xy 112.189668 108.75) (xy 112.189668 108.55) (xy 112.064668 108.525) (xy 111.938668 108.65) (xy 112.064668 108.775)
 			)
 		)
@@
 			)
 		)
-	)
-	(zone
-		(net 6)
-		(net_name "Net-(FL1-OUTPUT)")
-		(layer "F.Cu")
-		(name "$teardrop_padvia$")
-		(hatch none 0.1)
-		(priority 30001)
-		(attr
-			(teardrop
-				(type padvia)
-			)
-		)
-		(connect_pads yes
-			(clearance 0)
-		)
-		(min_thickness 0.0254)
-		(filled_areas_thickness no)
-		(fill yes
-			(thermal_gap 0.5)
-			(thermal_bridge_width 0.5)
-			(island_removal_mode 1)
-			(island_area_min 10)
-		)
-		(polygon
-			(pts
-				(xy 114.699668 108.6) (xy 114.699668 108.9) (xy 115.037143 109.03) (xy 115.260668 108.75) (xy 115.037143 108.47)
-			)
-		)
-	)
-	(zone
-		(net 4)
-		(net_name "/VCC_RF")
-		(layer "F.Cu")
-		(name "$teardrop_padvia$")
-		(hatch none 0.1)
-		(priority 30002)
-		(attr
-			(teardrop
-				(type padvia)
-			)
-		)
-		(connect_pads yes
-			(clearance 0)
-		)
-		(min_thickness 0.0254)
-		(filled_areas_thickness no)
-		(fill yes
-			(thermal_gap 0.5)
-			(thermal_bridge_width 0.5)
-			(island_removal_mode 1)
-			(island_area_min 10)
-		)
-		(polygon
-			(pts
-				(xy 112.189668 109.15) (xy 112.189668 108.95) (xy 112.064668 108.925) (xy 111.938668 109.05) (xy 112.064668 109.175)
-			)
-		)
-	)
-	(zone
-		(net 8)
-		(net_name "Net-(FL1-INPUT)")
-		(layer "F.Cu")
-		(name "$teardrop_padvia$")
-		(hatch none 0.1)
-		(priority 30003)
-		(attr
-			(teardrop
-				(type padvia)
-			)
-		)
-		(connect_pads yes
-			(clearance 0)
-		)
-		(min_thickness 0.0254)
-		(filled_areas_thickness no)
-		(fill yes
-			(thermal_gap 0.5)
-			(thermal_bridge_width 0.5)
-			(island_removal_mode 1)
-			(island_area_min 10)
-		)
-		(polygon
-			(pts
-				(xy 112.189668 108.75) (xy 112.189668 108.55) (xy 112.064668 108.525) (xy 111.938668 108.65) (xy 112.064668 108.775)
-			)
-		)

Commit message: lots of updates
Parts:
- moved G*** 0.11 mm to (108.4, 121.7)
Other:
- board text added: "made by bismarx"
- board text added: "u.fl - M"
- board text removed: "OwO"
- board text removed: "made by a good boy :3"
- board text removed: "u.fl - F"
