File: GPS-Compass/sub-sch/DRAWING.kicad_sch (KiCad schematic)
At the start: 0 parts

Commit message: UI changes
Other:
- note added: "BATTERY CHARGE"
- note added: "DEBOUNCED_GPIO"
- note added: "DISTANCE TO OBJ"
- note added: "ESP32_RESET"
- note added: "EXTERNAL_LED"
- note added: "GNSS_ANT"
- note added: "GNSS_RESET"
- note added: "MAIN USB PORT BATTERY CAHRGING DATA"
- note added: "MAIN_SWITCH"
- note added: "OTG_LED"
- note added: "OTG_SWITCH"
- note added: "POINTING ARROW"
- note added: "POWER_ON_LED"
- note added: "USB OTG CHARGER"

Commit message: jkolsd
Other:
- note added: "GPIO ACTIVATED FAN"
Changed lines of the file:
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@@
+		)
+	)
+	(rectangle
+		(start 153.67 111.125)
+		(end 166.37 122.555)
+		(stroke
+			(width 0)
+			(type solid)
+			(color 132 132 132 1)
+		)
+		(fill
+			(type none)
 		)
 	)
@@
 		)
 	)
+	(text "GPIO ACTIVATED FAN"
+		(exclude_from_sim no)
+		(at 160.02 110.49 0)
+		(effects
+			(font
+				(face "Bahnschrift")
+				(size 1 1)
+				(color 0 0 0 1)
+			)
+		)
+	)
