File: GPS-Compass/sub-sch/DRAWING.kicad_sch (KiCad schematic)
At the start: 0 parts

Commit message: asdasd
Other:
- note removed: "GPIO ACTIVATED FAN"
Changed lines of the file:
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@@
-		)
-	)
-	(rectangle
-		(start 153.67 111.125)
-		(end 166.37 122.555)
-		(stroke
-			(width 0)
-			(type solid)
-			(color 132 132 132 1)
-		)
-		(fill
-			(type none)
 		)
 	)
@@
 		)
 	)
-	(text "GPIO ACTIVATED FAN"
-		(exclude_from_sim no)
-		(at 160.02 110.49 0)
-		(effects
-			(font
-				(face "Bahnschrift")
-				(size 1 1)
-				(color 0 0 0 1)
-			)
-		)
-	)

Commit message: i think im depressed again
Other:
- note added: "USB SINK/SOURCE"
- note removed: "MAIN USB PORT BATTERY CAHRGING DATA"
- note removed: "OTG_SWITCH"
- note removed: "USB OTG CHARGER"
Changed lines of the file:
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@@
 	)
 	(rectangle
-		(start 190.5 72.39)
-		(end 191.77 74.93)
+		(start 190.5 74.295)
+		(end 191.77 76.835)
 		(stroke
 			(width 0)
@@
 	)
 	(rectangle
-		(start 125.73 80.645)
-		(end 127 83.82)
-		(stroke
-			(width 0)
-			(type solid)
-			(color 132 132 132 1)
-		)
-		(fill
-			(type color)
-			(color 132 132 132 1)
-		)
-	)
-	(rectangle
 		(start 152.4 88.9)
 		(end 165.1 101.6)
@@
 			(type color)
 			(color 132 132 132 1)
-		)
-	)
-	(rectangle
-		(start 190.5 68.58)
-		(end 191.77 72.39)
-		(stroke
-			(width 0)
-			(type solid)
-			(color 255 0 255 1)
-		)
-		(fill
-			(type color)
-			(color 255 0 255 1)
 		)
 	)
@@
 		)
 	)
-	(text "USB OTG CHARGER"
-		(exclude_from_sim no)
-		(at 111.125 76.835 0)
-		(effects
-			(font
-				(face "Bahnschrift")
-				(size 1 1)
-				(color 0 0 0 1)
-			)
-			(justify left)
-		)
-	)
-	(text "OTG_SWITCH"
-		(exclude_from_sim no)
-		(at 193.04 70.485 0)
+	(text "USB SINK/SOURCE"
+		(exclude_from_sim no)
+		(at 111.76 77.47 0)
 		(effects
 			(font
@@
 	(text "POINTING ARROW"
 		(exclude_from_sim no)
-		(at 150.495 88.265 0)
-		(effects
-			(font
-				(face "Bahnschrift")
-				(size 1 1)
-				(color 0 0 0 1)
-			)
-			(justify left)
-		)
-	)
-	(text "MAIN USB PORT\nBATTERY CAHRGING\nDATA"
-		(exclude_from_sim no)
-		(at 111.125 82.55 0)
+		(at 152.4 88.265 0)
 		(effects
 			(font
@@
 	(text "OTG_LED"
 		(exclude_from_sim no)
-		(at 193.04 73.66 0)
+		(at 193.04 75.565 0)
 		(effects
 			(font
@@
 		)
 	)
-	(polyline
-		(pts
-			(xy 191.77 70.485) (xy 193.04 71.755)
-		)
-		(stroke
-			(width 0)
-			(type solid)
-			(color 0 0 0 1)
-		)
-	)

Commit message: sdas
Other:
- note added: "v1.0.0"

Commit message: asda
Other:
- note added: "28mm"
Changed lines of the file:
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@@
 		)
 	)
+	(circle
+		(center 132.715 88.9)
+		(radius 1.27)
+		(stroke
+			(width 1)
+			(type solid)
+			(color 72 72 72 1)
+		)
+		(fill
+			(type color)
+			(color 72 72 72 1)
+		)
+	)
 	(rectangle
 		(start 198.755 32.385)
@@
 	)
 	(rectangle
-		(start 196.85 71.755)
-		(end 200.025 73.66)
+		(start 95.885 78.74)
+		(end 99.06 80.645)
 		(stroke
 			(width 0)
@@
 	)
 	(rectangle
+		(start 126.365 82.55)
+		(end 139.065 95.25)
+		(stroke
+			(width 0)
+			(type solid)
+			(color 132 132 132 1)
+		)
+		(fill
+			(type color)
+			(color 132 132 132 1)
+		)
+	)
+	(rectangle
 		(start 200.025 20.32)
 		(end 263.525 83.82)
@@
 		)
 	)
+	(text "28mm"
+		(exclude_from_sim no)
+		(at 133.35 98.425 0)
+		(effects
+			(font
+				(size 1.27 1.27)
+			)
+		)
+	)
 	(text "USB SINK/SOURCE"
 		(exclude_from_sim no)
@@
 	(text "GNSS_ANT"
 		(exclude_from_sim no)
-		(at 188.595 73.025 0)
+		(at 87.63 80.01 0)
 		(effects
 			(font
@@
 	(polyline
 		(pts
+			(xy 132.715 88.9) (xy 145.415 76.2)
+		)
+		(stroke
+			(width 1)
+			(type solid)
+			(color 0 0 0 1)
+		)
+	)
+	(polyline
+		(pts
 			(xy 214.63 28.575) (xy 214.63 26.035)
 		)
@@
 	(polyline
 		(pts
+			(xy 164.465 71.12) (xy 150.495 57.15)
+		)
+		(stroke
+			(width 2)
+			(type solid)
+			(color 128 77 0 1)
+		)
+	)
+	(polyline
+		(pts
 			(xy 259.715 30.48) (xy 259.715 28.575)
 		)
@@
 	(polyline
 		(pts
+			(xy 164.465 107.315) (xy 164.465 71.12)
+		)
+		(stroke
+			(width 2)
+			(type solid)
+			(color 128 77 0 1)
+		)
+	)
+	(polyline
+		(pts
+			(xy 100.33 71.12) (xy 114.3 57.15)
+		)
+		(stroke
+			(width 2)
+			(type solid)
+			(color 128 77 0 1)
+		)
+	)
+	(polyline
+		(pts
+			(xy 100.33 107.315) (xy 100.33 71.12)
+		)
+		(stroke
+			(width 2)
+			(type solid)
+			(color 128 77 0 1)
+		)
+	)
+	(polyline
+		(pts
 			(xy 208.915 28.575) (xy 208.915 26.035)
 		)
@@
 	(polyline
 		(pts
+			(xy 100.33 107.315) (xy 114.3 121.285)
+		)
+		(stroke
+			(width 2)
+			(type solid)
+			(color 128 77 0 1)
+		)
+	)
+	(polyline
+		(pts
 			(xy 257.81 27.94) (xy 259.715 27.94)
 		)
@@
 	(polyline
 		(pts
+			(xy 150.495 121.285) (xy 164.465 107.315)
+		)
+		(stroke
+			(width 2)
+			(type solid)
+			(color 128 77 0 1)
+		)
+	)
+	(polyline
+		(pts
 			(xy 259.715 31.115) (xy 257.81 31.115)
 		)
@@
 	(polyline
 		(pts
+			(xy 126.365 96.52) (xy 139.065 96.52)
+		)
+		(stroke
+			(width 0)
+			(type default)
+		)
+	)
+	(polyline
+		(pts
 			(xy 254 27.305) (xy 254 25.4)
 		)
@@
 	(polyline
 		(pts
+			(xy 114.3 121.285) (xy 150.495 121.285)
+		)
+		(stroke
+			(width 2)
+			(type solid)
+			(color 128 77 0 1)
+		)
+	)
+	(polyline
+		(pts
+			(xy 114.3 57.15) (xy 150.495 57.15)
+		)
+		(stroke
+			(width 2)
+			(type solid)
+			(color 128 77 0 1)
+		)
+	)
+	(polyline
+		(pts
 			(xy 254 31.115) (xy 252.095 31.115)
 		)
@@
 	)
 	(image
-		(at 66.04 111.76)
+		(at 52.705 106.045)
 		(scale 0.642065)
 		(data "iVBORw0KGgoAAAANSUhEUgAAAuAAAALgCAIAAABavFVeAAAAA3NCSVQICAjb4U/gAAAgAElEQVR4"
@@
 	)
 	(image
-		(at 63.5 62.23)
+		(at 52.705 60.96)
 		(scale 0.42532)
 		(data "iVBORw0KGgoAAAANSUhEUgAABCEAAASwCAIAAABKKsdPAAAAA3NCSVQICAjb4U/gAAAgAElEQVR4"
