File: GPS-Compass_UI/GPS-Compass_UI.kicad_sch (KiCad schematic)
At the start: 24 parts, among them J4 Conn_01x10_Socket, SW1 SPDT, SW3 RESET, SW4 EXT, SW5 RESET, SW6 EXT, SW7 EXT, SW8 EXT

Commit message: updates on different boards
Parts:
- removed C4: 100nF, Capacitor_SMD:C_0805_2012Metric, symbol Device:C
- removed R10: 1k, Resistor_SMD:R_0805_2012Metric, symbol Device:R
- removed R11: 10k, Resistor_SMD:R_0805_2012Metric, symbol Device:R
- removed SW8: EXT, Connector_Wire:SolderWire-0.1sqmm_1x02_P3.6mm_D0.4mm_OD1mm_Relief, symbol Switch:SW_Push
- added H1, H3: M2.5, MountingHole:MountingHole_2.5mm, symbol Mechanical:MountingHole
Connections:
- net DBNCD_3 is gone; now on net GND: J4.6 (Pin_6)
Other:
- note added: "AUX"
- note removed: "EXT. BUTTONS"
- moved on the sheet: D2, D3, R1, R7, SW1

Commit message: 3D updates
Parts:
- added J1: Conn_01x02_Pin, Connector_Wire:SolderWire-0.1sqmm_1x02_P3.6mm_D0.4mm_OD1mm_Relief, symbol Connector:Conn_01x02_Pin
Connections:
- net +3V3: now also J1.2 (Pin_2)
- net GND: now also J1.1 (Pin_1)
Other:
- moved on the sheet: D3, R7
