File: GPS-Compass_Arrow/GPS-Compass_Arrow.kicad_pcb (KiCad board)
At the start: 2 copper layers, 73.9 x 73.9 mm, 72 parts, among them J2 FFC2B28-12-G, U1 OSK3056A-LR, U2 MAX7219

Commit message: arrow pcb update
Parts:
- removed H1, H2: M2.5, MountingHole:MountingHole_2.7mm_M2.5_Pad_Via
- removed J2: FFC2B28-12-G, gps-compass_brd:GCT_FFC2B28-12-G
- added C10: 100nF, Capacitor_SMD:C_0805_2012Metric, F.Cu at (58.4, 138.3)
- added C3: 100nF, Capacitor_SMD:C_0805_2012Metric, F.Cu at (53.9, 132.3)
- added C4: 100nF, Capacitor_SMD:C_0805_2012Metric, F.Cu at (53.9, 135.3)
- added C5: 100nF, Capacitor_SMD:C_0805_2012Metric, F.Cu at (53.9, 138.3)
- added C6: 100nF, Capacitor_SMD:C_0805_2012Metric, F.Cu at (58.4, 126.2)
- added C7: 100nF, Capacitor_SMD:C_0805_2012Metric, F.Cu at (58.4, 129.3)
- added C8: 100nF, Capacitor_SMD:C_0805_2012Metric, F.Cu at (58.4, 132.3)
- added C9: 10uF, Capacitor_SMD:C_0805_2012Metric, F.Cu at (58.4, 135.3)
- added IC1: 74VHC9595FT, gps-compass_brd:SOP65P640X120-16N, F.Cu at (24.3, 89.4)
- added IC2: 74VHC9595FT, gps-compass_brd:SOP65P640X120-16N, F.Cu at (24.3, 96.2)
- added IC3: 74VHC9595FT, gps-compass_brd:SOP65P640X120-16N, F.Cu at (24.3, 102.9)
- added IC4: 74VHC9595FT, gps-compass_brd:SOP65P640X120-16N, F.Cu at (24.3, 109.7)
- added IC5: 74VHC9595FT, gps-compass_brd:SOP65P640X120-16N, F.Cu at (24.3, 116.5)
- added IC6: 74VHC9595FT, gps-compass_brd:SOP65P640X120-16N, F.Cu at (33.2, 89.4)
- added IC7: 74VHC9595FT, gps-compass_brd:SOP65P640X120-16N, F.Cu at (33.2, 96.2)
- added IC8: 74VHC9595FT, gps-compass_brd:SOP65P640X120-16N, F.Cu at (33.2, 102.9)
- added J1: FFC2B28-12-G, gps-compass_brd:GCT_FFC2B28-12-G, F.Cu at (24.6, 122.9)
- added R10: 220, Resistor_SMD:R_0805_2012Metric, B.Cu at (166.2, 91.6)
- added R11: 220, Resistor_SMD:R_0805_2012Metric, B.Cu at (169.2, 91.6)
- added R12: 220, Resistor_SMD:R_0805_2012Metric, F.Cu at (136.4, 57.0)
- added R13: 220, Resistor_SMD:R_0805_2012Metric, F.Cu at (139.4, 57.0)
- added R14: 220, Resistor_SMD:R_0805_2012Metric, F.Cu at (142.3, 57.0)
- added R15: 220, Resistor_SMD:R_0805_2012Metric, F.Cu at (145.3, 57.0)
- added R16: 220, Resistor_SMD:R_0805_2012Metric, F.Cu at (148.2, 57.0)
- added R17: 220, Resistor_SMD:R_0805_2012Metric, F.Cu at (151.2, 57.0)
- added R18: 220, Resistor_SMD:R_0805_2012Metric, F.Cu at (154.2, 57.0)
- added R19: 220, Resistor_SMD:R_0805_2012Metric, F.Cu at (157.1, 57.0)
- added R2: 220, Resistor_SMD:R_0805_2012Metric, B.Cu at (142.7, 91.6)
- added R20: 220, Resistor_SMD:R_0805_2012Metric, F.Cu at (160.1, 57.0)
- added R21: 220, Resistor_SMD:R_0805_2012Metric, F.Cu at (163.0, 57.0)
- added R22: 220, Resistor_SMD:R_0805_2012Metric, F.Cu at (165.9, 57.0)
- added R23: 220, Resistor_SMD:R_0805_2012Metric, F.Cu at (136.4, 52.6)
- added R24: 220, Resistor_SMD:R_0805_2012Metric, F.Cu at (139.4, 52.6)
- added R25: 220, Resistor_SMD:R_0805_2012Metric, F.Cu at (142.3, 52.6)
- added R26: 220, Resistor_SMD:R_0805_2012Metric, F.Cu at (145.3, 52.6)
- added R27: 220, Resistor_SMD:R_0805_2012Metric, F.Cu at (148.2, 52.6)
- added R28: 220, Resistor_SMD:R_0805_2012Metric, F.Cu at (151.2, 52.6)
- added R29: 220, Resistor_SMD:R_0805_2012Metric, F.Cu at (154.2, 52.6)
- added R3: 220, Resistor_SMD:R_0805_2012Metric, B.Cu at (145.6, 91.6)
- added R30: 220, Resistor_SMD:R_0805_2012Metric, F.Cu at (157.1, 52.6)
- added R31: 220, Resistor_SMD:R_0805_2012Metric, F.Cu at (160.1, 52.6)
- added R32: 220, Resistor_SMD:R_0805_2012Metric, F.Cu at (163.0, 52.6)
- added R33: 220, Resistor_SMD:R_0805_2012Metric, F.Cu at (205.0, 97.5)
- added R34: 220, Resistor_SMD:R_0805_2012Metric, F.Cu at (209.4, 68.0)
- added R35: 220, Resistor_SMD:R_0805_2012Metric, F.Cu at (209.4, 70.9)
- added R36: 220, Resistor_SMD:R_0805_2012Metric, F.Cu at (209.4, 73.8)
- added R37: 220, Resistor_SMD:R_0805_2012Metric, F.Cu at (209.4, 76.8)
- added R38: 220, Resistor_SMD:R_0805_2012Metric, F.Cu at (209.4, 79.8)
- added R39: 220, Resistor_SMD:R_0805_2012Metric, F.Cu at (209.4, 82.7)
- added R4: 220, Resistor_SMD:R_0805_2012Metric, B.Cu at (148.6, 91.6)
- added R40: 220, Resistor_SMD:R_0805_2012Metric, F.Cu at (209.4, 85.7)
- added R41: 220, Resistor_SMD:R_0805_2012Metric, F.Cu at (209.4, 88.6)
- added R42: 220, Resistor_SMD:R_0805_2012Metric, F.Cu at (209.4, 91.5)
- added R43: 220, Resistor_SMD:R_0805_2012Metric, F.Cu at (209.4, 94.5)
- added R44: 220, Resistor_SMD:R_0805_2012Metric, F.Cu at (209.4, 97.5)
- added R45: 220, Resistor_SMD:R_0805_2012Metric, F.Cu at (213.8, 68.0)
- added R46: 220, Resistor_SMD:R_0805_2012Metric, F.Cu at (213.8, 70.9)
- added R47: 220, Resistor_SMD:R_0805_2012Metric, F.Cu at (213.8, 73.8)
- added R48: 220, Resistor_SMD:R_0805_2012Metric, F.Cu at (213.8, 76.8)
- added R49: 220, Resistor_SMD:R_0805_2012Metric, F.Cu at (213.8, 79.8)
- added R5: 220, Resistor_SMD:R_0805_2012Metric, B.Cu at (151.5, 91.6)
- added R50: 220, Resistor_SMD:R_0805_2012Metric, F.Cu at (213.8, 82.7)
- added R51: 220, Resistor_SMD:R_0805_2012Metric, F.Cu at (213.8, 85.7)
- added R52: 220, Resistor_SMD:R_0805_2012Metric, F.Cu at (213.8, 88.6)
- added R53: 220, Resistor_SMD:R_0805_2012Metric, F.Cu at (213.8, 91.5)
- added R54: 220, Resistor_SMD:R_0805_2012Metric, F.Cu at (213.8, 94.5)
- added R55: 220, Resistor_SMD:R_0805_2012Metric, F.Cu at (213.8, 97.5)
- added R56: 220, Resistor_SMD:R_0805_2012Metric, F.Cu at (218.2, 68.0)
- added R57: 220, Resistor_SMD:R_0805_2012Metric, F.Cu at (218.2, 70.9)
- added R58: 220, Resistor_SMD:R_0805_2012Metric, F.Cu at (218.2, 73.8)
- added R59: 220, Resistor_SMD:R_0805_2012Metric, F.Cu at (218.2, 76.8)
- added R6: 220, Resistor_SMD:R_0805_2012Metric, B.Cu at (154.4, 91.6)
- added R60: 220, Resistor_SMD:R_0805_2012Metric, F.Cu at (218.2, 79.8)
- added R61: 220, Resistor_SMD:R_0805_2012Metric, F.Cu at (218.2, 82.7)
- added R62: 220, Resistor_SMD:R_0805_2012Metric, F.Cu at (218.2, 85.7)
- added R63: 220, Resistor_SMD:R_0805_2012Metric, F.Cu at (218.2, 88.6)
- added R64: 220, Resistor_SMD:R_0805_2012Metric, F.Cu at (218.2, 91.5)
- added R65: 10k, Resistor_SMD:R_0805_2012Metric, F.Cu at (218.2, 94.5)
- added R7: 220, Resistor_SMD:R_0805_2012Metric, B.Cu at (157.4, 91.6)
- added R8: 220, Resistor_SMD:R_0805_2012Metric, B.Cu at (160.3, 91.6)
- added R9: 220, Resistor_SMD:R_0805_2012Metric, B.Cu at (163.3, 91.6)
- C1: value 10uF -> 100nF; moved to F.Cu
- C2, U2: moved to F.Cu
- R1: value 10k -> 220
- moved U2 109.5 mm to (44.4, 132.5), turned to 0 degrees
- moved C2 103.8 mm to (53.9, 129.3), turned to 0 degrees
- moved C1 99.7 mm to (53.9, 126.2), turned to 0 degrees
- moved D41 70.0 mm to (120.4, 130.7), turned to 135 degrees
- moved D9 70.0 mm to (169.8, 81.3), turned to -45 degrees
- moved D42 69.7 mm to (118.0, 128.2), turned to 129.375 degrees
- moved D40 69.7 mm to (122.9, 133.1), turned to 140.625 degrees
- moved D10 69.7 mm to (172.2, 83.8), turned to -50.625 degrees
- moved D8 69.7 mm to (167.3, 78.9), turned to -39.375 degrees
- moved D43 68.7 mm to (116.0, 125.4), turned to 123.75 degrees
- moved D11 68.7 mm to (174.2, 86.6), turned to -56.25 degrees
- moved D39 68.7 mm to (125.7, 135.1), turned to 146.25 degrees
- moved D7 68.7 mm to (164.5, 76.9), turned to -33.75 degrees
- moved D44 67.0 mm to (114.2, 122.5), turned to 118.125 degrees
- moved D12 67.0 mm to (176.0, 89.5), turned to -61.875 degrees
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Connections:
- C1 pad 1: +5V -> GND
- C1 pad 2: GND -> +3V3
- C2 pad 1: +5V -> GND
- C2 pad 2: GND -> +3V3
- D1 pad 1: unconnected-(D1-K-Pad1) -> GND
- D1 pad 2: unconnected-(D1-A-Pad2) -> Net-(D1-A)
- D10 pad 1: unconnected-(D1-K-Pad1) -> GND
- D10 pad 2: unconnected-(D1-A-Pad2) -> Net-(D10-A)
- D11 pad 1: unconnected-(D1-K-Pad1) -> GND
- D11 pad 2: unconnected-(D1-A-Pad2) -> Net-(D11-A)
- D12 pad 1: unconnected-(D1-K-Pad1) -> GND
- D12 pad 2: unconnected-(D1-A-Pad2) -> Net-(D12-A)
- D13 pad 1: unconnected-(D1-K-Pad1) -> GND
- D13 pad 2: unconnected-(D1-A-Pad2) -> Net-(D13-A)
- D14 pad 1: unconnected-(D1-K-Pad1) -> GND
- D14 pad 2: unconnected-(D1-A-Pad2) -> Net-(D14-A)
- D15 pad 1: unconnected-(D1-K-Pad1) -> GND
- D15 pad 2: unconnected-(D1-A-Pad2) -> Net-(D15-A)
- D16 pad 1: unconnected-(D1-K-Pad1) -> GND
- D16 pad 2: unconnected-(D1-A-Pad2) -> Net-(D16-A)
- D17 pad 1: unconnected-(D1-K-Pad1) -> GND
- D17 pad 2: unconnected-(D1-A-Pad2) -> Net-(D17-A)
- D18 pad 1: unconnected-(D1-K-Pad1) -> GND
- D18 pad 2: unconnected-(D1-A-Pad2) -> Net-(D18-A)
- D19 pad 1: unconnected-(D1-K-Pad1) -> GND
- D19 pad 2: unconnected-(D1-A-Pad2) -> Net-(D19-A)
- D2 pad 1: unconnected-(D1-K-Pad1) -> GND
- D2 pad 2: unconnected-(D1-A-Pad2) -> Net-(D2-A)
- D20 pad 1: unconnected-(D1-K-Pad1) -> GND
- D20 pad 2: unconnected-(D1-A-Pad2) -> Net-(D20-A)
- D21 pad 1: unconnected-(D1-K-Pad1) -> GND
- D21 pad 2: unconnected-(D1-A-Pad2) -> Net-(D21-A)
- D22 pad 1: unconnected-(D1-K-Pad1) -> GND
- D22 pad 2: unconnected-(D1-A-Pad2) -> Net-(D22-A)
- D23 pad 1: unconnected-(D1-K-Pad1) -> GND
- D23 pad 2: unconnected-(D1-A-Pad2) -> Net-(D23-A)
- D24 pad 1: unconnected-(D1-K-Pad1) -> GND
- D24 pad 2: unconnected-(D1-A-Pad2) -> Net-(D24-A)
- D25 pad 1: unconnected-(D1-K-Pad1) -> GND
- D25 pad 2: unconnected-(D1-A-Pad2) -> Net-(D25-A)
- D26 pad 1: unconnected-(D1-K-Pad1) -> GND
- D26 pad 2: unconnected-(D1-A-Pad2) -> Net-(D26-A)
- D27 pad 1: unconnected-(D1-K-Pad1) -> GND
- D27 pad 2: unconnected-(D1-A-Pad2) -> Net-(D27-A)
- D28 pad 1: unconnected-(D1-K-Pad1) -> GND
- D28 pad 2: unconnected-(D1-A-Pad2) -> Net-(D28-A)
- D29 pad 1: unconnected-(D1-K-Pad1) -> GND
- D29 pad 2: unconnected-(D1-A-Pad2) -> Net-(D29-A)
- D3 pad 1: unconnected-(D1-K-Pad1) -> GND
- D3 pad 2: unconnected-(D1-A-Pad2) -> Net-(D3-A)
- D30 pad 1: unconnected-(D1-K-Pad1) -> GND
- D30 pad 2: unconnected-(D1-A-Pad2) -> Net-(D30-A)
- D31 pad 1: unconnected-(D1-K-Pad1) -> GND
- D31 pad 2: unconnected-(D1-A-Pad2) -> Net-(D31-A)
- D32 pad 1: unconnected-(D1-K-Pad1) -> GND
- D32 pad 2: unconnected-(D1-A-Pad2) -> Net-(D32-A)
- D33 pad 1: unconnected-(D1-K-Pad1) -> GND
- D33 pad 2: unconnected-(D1-A-Pad2) -> Net-(D33-A)
- D34 pad 1: unconnected-(D1-K-Pad1) -> GND
- D34 pad 2: unconnected-(D1-A-Pad2) -> Net-(D34-A)
- D35 pad 1: unconnected-(D1-K-Pad1) -> GND
- D35 pad 2: unconnected-(D1-A-Pad2) -> Net-(D35-A)
- D36 pad 1: unconnected-(D1-K-Pad1) -> GND
- D36 pad 2: unconnected-(D1-A-Pad2) -> Net-(D36-A)
- D37 pad 1: unconnected-(D1-K-Pad1) -> GND
- D37 pad 2: unconnected-(D1-A-Pad2) -> Net-(D37-A)
- D38 pad 1: unconnected-(D1-K-Pad1) -> GND
- D38 pad 2: unconnected-(D1-A-Pad2) -> Net-(D38-A)
- D39 pad 1: unconnected-(D1-K-Pad1) -> GND
- D39 pad 2: unconnected-(D1-A-Pad2) -> Net-(D39-A)
- D4 pad 1: unconnected-(D1-K-Pad1) -> GND
- D4 pad 2: unconnected-(D1-A-Pad2) -> Net-(D4-A)
- D40 pad 1: unconnected-(D1-K-Pad1) -> GND
- D40 pad 2: unconnected-(D1-A-Pad2) -> Net-(D40-A)
- D41 pad 1: unconnected-(D1-K-Pad1) -> GND
- D41 pad 2: unconnected-(D1-A-Pad2) -> Net-(D41-A)
- D42 pad 1: unconnected-(D1-K-Pad1) -> GND
- D42 pad 2: unconnected-(D1-A-Pad2) -> Net-(D42-A)
- D43 pad 1: unconnected-(D1-K-Pad1) -> GND
- D43 pad 2: unconnected-(D1-A-Pad2) -> Net-(D43-A)
- D44 pad 1: unconnected-(D1-K-Pad1) -> GND
- D44 pad 2: unconnected-(D1-A-Pad2) -> Net-(D44-A)
- D45 pad 1: unconnected-(D1-K-Pad1) -> GND
- D45 pad 2: unconnected-(D1-A-Pad2) -> Net-(D45-A)
- D46 pad 1: unconnected-(D1-K-Pad1) -> GND
- D46 pad 2: unconnected-(D1-A-Pad2) -> Net-(D46-A)
- D47 pad 1: unconnected-(D1-K-Pad1) -> GND
- D47 pad 2: unconnected-(D1-A-Pad2) -> Net-(D47-A)
- D48 pad 1: unconnected-(D1-K-Pad1) -> GND
- D48 pad 2: unconnected-(D1-A-Pad2) -> Net-(D48-A)
- D49 pad 1: unconnected-(D1-K-Pad1) -> GND
- D49 pad 2: unconnected-(D1-A-Pad2) -> Net-(D49-A)
- D5 pad 1: unconnected-(D1-K-Pad1) -> GND
- D5 pad 2: unconnected-(D1-A-Pad2) -> Net-(D5-A)
- D50 pad 1: unconnected-(D1-K-Pad1) -> GND
- D50 pad 2: unconnected-(D1-A-Pad2) -> Net-(D50-A)
- D51 pad 1: unconnected-(D1-K-Pad1) -> GND
- D51 pad 2: unconnected-(D1-A-Pad2) -> Net-(D51-A)
- D52 pad 1: unconnected-(D1-K-Pad1) -> GND
- D52 pad 2: unconnected-(D1-A-Pad2) -> Net-(D52-A)
- D53 pad 1: unconnected-(D1-K-Pad1) -> GND
- D53 pad 2: unconnected-(D1-A-Pad2) -> Net-(D53-A)
- D54 pad 1: unconnected-(D1-K-Pad1) -> GND
- D54 pad 2: unconnected-(D1-A-Pad2) -> Net-(D54-A)
- D55 pad 1: unconnected-(D1-K-Pad1) -> GND
- D55 pad 2: unconnected-(D1-A-Pad2) -> Net-(D55-A)
- D56 pad 1: unconnected-(D1-K-Pad1) -> GND
- D56 pad 2: unconnected-(D1-A-Pad2) -> Net-(D56-A)
- D57 pad 1: unconnected-(D1-K-Pad1) -> GND
- D57 pad 2: unconnected-(D1-A-Pad2) -> Net-(D57-A)
- D58 pad 1: unconnected-(D1-K-Pad1) -> GND
- D58 pad 2: unconnected-(D1-A-Pad2) -> Net-(D58-A)
- D59 pad 1: unconnected-(D1-K-Pad1) -> GND
- D59 pad 2: unconnected-(D1-A-Pad2) -> Net-(D59-A)
- D6 pad 1: unconnected-(D1-K-Pad1) -> GND
- D6 pad 2: unconnected-(D1-A-Pad2) -> Net-(D6-A)
- D60 pad 1: unconnected-(D1-K-Pad1) -> GND
- D60 pad 2: unconnected-(D1-A-Pad2) -> Net-(D60-A)
- D61 pad 1: unconnected-(D1-K-Pad1) -> GND
- D61 pad 2: unconnected-(D1-A-Pad2) -> Net-(D61-A)
- D62 pad 1: unconnected-(D1-K-Pad1) -> GND
- D62 pad 2: unconnected-(D1-A-Pad2) -> Net-(D62-A)
- D63 pad 1: unconnected-(D1-K-Pad1) -> GND
- D63 pad 2: unconnected-(D1-A-Pad2) -> Net-(D63-A)
- D64 pad 1: unconnected-(D1-K-Pad1) -> GND
- D64 pad 2: unconnected-(D1-A-Pad2) -> Net-(D64-A)
- D7 pad 1: unconnected-(D1-K-Pad1) -> GND
- D7 pad 2: unconnected-(D1-A-Pad2) -> Net-(D7-A)
- D8 pad 1: unconnected-(D1-K-Pad1) -> GND
- D8 pad 2: unconnected-(D1-A-Pad2) -> Net-(D8-A)
- D9 pad 1: unconnected-(D1-K-Pad1) -> GND
- D9 pad 2: unconnected-(D1-A-Pad2) -> Net-(D9-A)
- R1 pad 1: +5V -> /LED_1
- R1 pad 2: Net-(U2-ISET) -> Net-(D1-A)

Commit message: arrow pcb
Parts:
- added H1: M2.5, MountingHole:MountingHole_2.5mm_Pad_Via, F.Cu at (164.4, 105.5)
- added H2: M2.5, MountingHole:MountingHole_2.5mm_Pad_Via, F.Cu at (125.9, 105.5)
- added J2: INDICATOR, Connector_PinHeader_2.54mm:PinHeader_1x02_P2.54mm_Vertical, F.Cu at (126.4, 100.2)
- added REF**: OSHW-Logo_5.7x6mm_Copper, Symbol:OSHW-Logo_5.7x6mm_Copper, F.Cu at (145.1, 94.2)
- C10, C9, J1, R65, U2: moved to B.Cu
- R1, R10, R11, R2, R3, R4, R5, R6, R7, R8, R9: footprint Resistor_SMD:R_0805_2012Metric -> Resistor_SMD:R_0603_1608Metric; moved to F.Cu
- R12, R13, R14, R15, R16, R17, R18, R19, R20, R21, R22, R23, R24, R25, R26, R27, R28, R29, R30, R31, R32, R33, R34, R35, R36, R37, R38, R39, R40, R41, R42, R43, R44, R45, R46, R47, R48, R49, R50, R51, R52, R53, R54, R55, R56, R57, R58, R59, R60, R61, R62, R63, R64: footprint Resistor_SMD:R_0805_2012Metric -> Resistor_SMD:R_0603_1608Metric
- moved IC3 148.8 mm to (173.1, 106.0), turned to 90 degrees
- moved IC2 142.4 mm to (166.6, 91.5), turned to 90 degrees
- moved IC4 128.3 mm to (150.4, 133.5)
- moved IC1 126.5 mm to (150.4, 78.2), turned to 180 degrees
- moved J1 120.6 mm to (145.1, 127.5)
- moved C3 118.7 mm to (169.1, 103.7), turned to 90 degrees
- moved IC5 116.8 mm to (139.9, 133.5)
- moved C2 115.8 mm to (162.6, 89.2), turned to 90 degrees
- moved R45 111.4 mm to (114.6, 118.6), turned to 112.5 degrees
- moved R46 109.7 mm to (113.5, 115.6), turned to 106.875 degrees
- moved IC8 109.5 mm to (139.9, 78.2), turned to 180 degrees
- moved R47 108.1 mm to (112.7, 112.4), turned to 101.25 degrees
- moved R48 106.6 mm to (112.3, 109.2), turned to 95.625 degrees
- moved R49 105.0 mm to (112.1, 106.0), turned to 90 degrees
- moved R50 103.5 mm to (112.3, 102.8), turned to 84.375 degrees
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Connections:
- net DIG_0 renamed /DIG_1
- net DIG_1 renamed /DIG_2
- net DIG_2 renamed /DIG_3
- net MOSI renamed /MOSI
- net SEG_A renamed /SEG_A
- net SEG_B renamed /SEG_B
- net SEG_C renamed /SEG_C
- net SEG_D renamed /SEG_D
- net SEG_DP renamed /SEG_DP
- net SEG_E renamed /SEG_E
- net SEG_F renamed /SEG_F
- net SEG_G renamed /SEG_G
- net ~{CS} renamed /~{CS}
- C10 pad 1: +5V -> GND
- C10 pad 2: GND -> +5V
- C9 pad 1: +5V -> GND
- C9 pad 2: GND -> +5V
- IC1 pad 3: CLK -> /CLK
- IC2 pad 10: /LED_37 -> /LED_13
- IC2 pad 11: /LED_38 -> /LED_14
- IC2 pad 12: /LED_39 -> /LED_15
- IC2 pad 13: /LED_40 -> /LED_16
- IC2 pad 14: /SIOUT_5 -> /SIOUT_2
- IC2 pad 2: /SIOUT_4 -> /SIOUT_1
- IC2 pad 3: CLK -> /CLK
- IC2 pad 5: /LED_33 -> /LED_9
- IC2 pad 6: /LED_34 -> /LED_10
- IC2 pad 7: /LED_35 -> /LED_11
- IC2 pad 9: /LED_36 -> /LED_12
- IC3 pad 10: /LED_13 -> /LED_21
- IC3 pad 11: /LED_14 -> /LED_22
- IC3 pad 12: /LED_15 -> /LED_23
- IC3 pad 13: /LED_16 -> /LED_24
- IC3 pad 14: /SIOUT_2 -> /SIOUT_3
- IC3 pad 2: /SIOUT_1 -> /SIOUT_2
- IC3 pad 3: CLK -> /CLK
- IC3 pad 5: /LED_9 -> /LED_17
- IC3 pad 6: /LED_10 -> /LED_18
- IC3 pad 7: /LED_11 -> /LED_19
- IC3 pad 9: /LED_12 -> /LED_20
- IC4 pad 10: /LED_45 -> /LED_29
- IC4 pad 11: /LED_46 -> /LED_30
- IC4 pad 12: /LED_47 -> /LED_31
- IC4 pad 13: /LED_48 -> /LED_32
- IC4 pad 14: /SIOUT_6 -> /SIOUT_4
- IC4 pad 2: /SIOUT_5 -> /SIOUT_3
- IC4 pad 3: CLK -> /CLK
- IC4 pad 5: /LED_41 -> /LED_25
- IC4 pad 6: /LED_42 -> /LED_26
- IC4 pad 7: /LED_43 -> /LED_27
- IC4 pad 9: /LED_44 -> /LED_28
- IC5 pad 10: /LED_21 -> /LED_37
- IC5 pad 11: /LED_22 -> /LED_38
- IC5 pad 12: /LED_23 -> /LED_39
- IC5 pad 13: /LED_24 -> /LED_40
- IC5 pad 14: /SIOUT_3 -> /SIOUT_5
- IC5 pad 2: /SIOUT_2 -> /SIOUT_4
- IC5 pad 3: CLK -> /CLK
- IC5 pad 5: /LED_17 -> /LED_33
- IC5 pad 6: /LED_18 -> /LED_34
- IC5 pad 7: /LED_19 -> /LED_35
- IC5 pad 9: /LED_20 -> /LED_36
- IC6 pad 10: /LED_53 -> /LED_45
- IC6 pad 11: /LED_54 -> /LED_46
- IC6 pad 12: /LED_55 -> /LED_47
- IC6 pad 13: /LED_56 -> /LED_48
- IC6 pad 14: /SIOUT_7 -> /SIOUT_6
- IC6 pad 2: /SIOUT_6 -> /SIOUT_5
- IC6 pad 3: CLK -> /CLK
- IC6 pad 5: /LED_49 -> /LED_41
- IC6 pad 6: /LED_50 -> /LED_42
- IC6 pad 7: /LED_51 -> /LED_43
- IC6 pad 9: /LED_52 -> /LED_44
- IC7 pad 10: /LED_29 -> /LED_53
- IC7 pad 11: /LED_30 -> /LED_54
- IC7 pad 12: /LED_31 -> /LED_55
- IC7 pad 13: /LED_32 -> /LED_56
- IC7 pad 14: /SIOUT_4 -> /SIOUT_7
- IC7 pad 2: /SIOUT_3 -> /SIOUT_6
- IC7 pad 3: CLK -> /CLK
- IC7 pad 5: /LED_25 -> /LED_49
- IC7 pad 6: /LED_26 -> /LED_50
- IC7 pad 7: /LED_27 -> /LED_51
- IC7 pad 9: /LED_28 -> /LED_52
- IC8 pad 3: CLK -> /CLK
- J1 pad 7: CLK -> /CLK
- U2 pad 13: CLK -> /CLK_SPI
Routing:
- net +3V3: track 0.00 -> 186.0 mm, vias 0 -> 6
- net /LATCH: track 0.00 -> 142.0 mm, vias 0 -> 10
- net /CLK: track 0.00 -> 139.4 mm, vias 0 -> 10
- net /SIOUT_5: track 0.00 -> 45.9 mm, vias 0 -> 2
- net /SIOUT_3: track 0.00 -> 45.0 mm, vias 0 -> 2
- net /SIOUT_7: track 0.00 -> 36.2 mm, vias 0 -> 2
- net /LED_41: track 0.00 -> 29.6 mm, vias 0 -> 2
- net /SIOUT_1: track 0.00 -> 29.6 mm, vias 0 -> 2
- net /LED_42: track 0.00 -> 26.9 mm, vias 0 -> 2
- net /LED_24: track 0.00 -> 24.6 mm, vias 0 -> 2
- net /LED_49: track 0.00 -> 24.4 mm, vias 0 -> 2
- net /LED_57: track 0.00 -> 24.2 mm, vias 0 -> 2
- net /LED_25: track 0.00 -> 24.2 mm, vias 0 -> 2
- net /LED_43: track 0.00 -> 23.7 mm, vias 0 -> 2
- net /SIOUT_6: track 0.00 -> 23.5 mm, vias 0 -> 2
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- added copper zone on B.Cu, net GND
- added copper zone on F.Cu, net GND
Other:
- outline, holes or cut-outs redrawn

Commit message: arrow pcp updates
Parts:
- moved C10 10.8 mm to (133.1, 125.0)
- moved C9 10.8 mm to (133.2, 123.0)
- moved R65 10.8 mm to (135.9, 124.0)
- moved U2 10.8 mm to (134.9, 116.0)
- moved C8 1.25 mm to (134.9, 80.5), turned to 90 degrees
- moved J1 0.75 mm to (145.1, 128.2)
Connections:
- J1 pad 1: unconnected-(J1-Pad1) -> +5V
- J1 pad 10: unconnected-(J1-Pad10) -> /LATCH
- J1 pad 11: unconnected-(J1-Pad11) -> /CLK
- J1 pad 12: +5V -> /SI
- J1 pad 2: unconnected-(J1-Pad2) -> +5V
- J1 pad 3: unconnected-(J1-Pad3) -> /MOSI
- J1 pad 4: unconnected-(J1-Pad4) -> /CLK_SPI
- J1 pad 7: /CLK -> unconnected-(J1-Pad7)
- J1 pad 9: /MOSI -> unconnected-(J1-Pad9)
Routing:
- net /SI: track 0.00 -> 72.5 mm, vias 0 -> 1
- net /LATCH: track 142.0 -> 174.2 mm, vias 10 -> 11
- net /SEG_DP: track 0.00 -> 29.6 mm, vias 0 -> 1
- net /SIOUT_5: track 45.9 -> 17.3 mm
- net /SEG_D: track 0.00 -> 28.5 mm, vias 0 -> 1
- net /MOSI: track 0.00 -> 27.2 mm, vias 0 -> 2
- net /SEG_C: track 0.00 -> 26.6 mm, vias 0 -> 1
- net /CLK: track 139.4 -> 165.8 mm, vias 10 -> 12
- net /SEG_G: track 0.00 -> 23.4 mm, vias 0 -> 1
- net /SEG_B: track 0.00 -> 21.9 mm, vias 0 -> 1
- net /SEG_E: track 0.00 -> 21.4 mm, vias 0 -> 1
- net /~{CS}: track 0.00 -> 20.1 mm, vias 0 -> 2
- net /DIG_3: track 0.00 -> 19.2 mm, vias 0 -> 1
- net +3V3: track 186.0 -> 166.9 mm, vias 6 -> 9
- net /DIG_1: track 0.00 -> 15.3 mm, vias 0 -> 1
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
Commit message: arrowpcb update
Parts:
- moved C7 5.83 mm to (122.6, 96.5), turned to 0 degrees
- moved C2 3.02 mm to (163.9, 86.5), turned to 180 degrees
- moved C8 1.27 mm to (134.6, 79.2), turned to -90 degrees
- moved C1 0.95 mm to (145.4, 80.2)
Connections:
- J1 pad 3: /MOSI -> GND
- J1 pad 4: /CLK_SPI -> /MOSI
- J1 pad 5: /~{CS} -> /CLK_SPI
- J1 pad 6: unconnected-(J1-Pad6) -> /~{CS}
- J1 pad 7: unconnected-(J1-Pad7) -> VBATT
- J1 pad 8: unconnected-(J1-Pad8) -> +3V3
- J1 pad 9: unconnected-(J1-Pad9) -> GND
Routing:
- net VBATT: track 0.00 -> 49.2 mm, vias 0 -> 2
- net /SIOUT_5: track 17.3 -> 47.5 mm
- net /LATCH: track 174.2 -> 196.3 mm, vias 11 -> 10
- net /CLK: track 165.8 -> 187.3 mm, vias 12 -> 9
- net +3V3: track 166.9 -> 187.2 mm, vias 9 -> 13
- net GND: track 3.74 -> 19.2 mm, vias 29 -> 102
- net /SIOUT_7: track 36.2 -> 29.6 mm
- net /SEG_B: track 21.9 -> 23.7 mm
- net /LED_58: track 21.2 -> 22.2 mm
- net /LED_45: track 12.0 -> 13.0 mm, vias 3 -> 2

Commit message: main pcb and arrow updatws
Parts:
- C1, C10, C2, C3, C4, C5, C6, C7, C8: value 100nF -> 100n
- C9: value 10uF -> 10u
Connections:
- net /CLK renamed /CLK_SR
- net /LATCH renamed /LATCH_SR
- net /SI renamed /SI_SR
- J1 pad 4: /MOSI -> /~{CS}_SPI
- J1 pad 5: /CLK_SPI -> /MOSI_SPI
- J1 pad 6: /~{CS} -> /CLK_SPI
- U2 pad 1: /MOSI -> /MOSI_SPI
- U2 pad 12: /~{CS} -> /~{CS}_SPI
Routing:
- net /MOSI_SPI: track 0.00 -> 27.6 mm, vias 0 -> 2
- net /MOSI: track 27.4 -> 0.00 mm, vias 2 -> 0
- net /~{CS}: track 20.3 -> 0.00 mm, vias 2 -> 0
- net /~{CS}_SPI: track 0.00 -> 17.3 mm, vias 0 -> 2
- net VBATT: track 49.2 -> 49.8 mm

Commit message: asda
Connections:
- J1 pad 4: /~{CS}_SPI -> /MOSI_SPI
- J1 pad 5: /MOSI_SPI -> /CLK_SPI
- J1 pad 6: /CLK_SPI -> /~{CS}_SPI
Routing:
- net /~{CS}_SPI: track 17.3 -> 20.3 mm
- net GND: track 19.2 -> 17.8 mm
Changed lines of the file:
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@@
 			(size 0.3 0.8)
 			(layers "B.Cu" "B.Paste")
-			(net 172 "/~{CS}_SPI")
+			(net 170 "/MOSI_SPI")
 			(pinfunction "4")
 			(pintype "passive")
@@
 			(size 0.3 0.8)
 			(layers "B.Cu" "B.Paste")
-			(net 170 "/MOSI_SPI")
+			(net 169 "/CLK_SPI")
 			(pinfunction "5")
 			(pintype "passive")
@@
 			(size 0.3 0.8)
 			(layers "B.Cu" "B.Paste")
-			(net 169 "/CLK_SPI")
+			(net 172 "/~{CS}_SPI")
 			(pinfunction "6")
 			(pintype "passive")
@@
 	)
 	(segment
-		(start 141.262437 125.746503)
-		(end 142.111437 126.595503)
-		(width 0.25)
-		(layer "B.Cu")
-		(net 4)
-	)
-	(segment
-		(start 142.111437 126.595503)
-		(end 142.111437 126.746503)
-		(width 0.25)
-		(layer "B.Cu")
-		(net 4)
-	)
-	(segment
 		(start 143.361437 129.496503)
 		(end 143.361437 130.246503)
@@
 	)
 	(segment
-		(start 144.861437 127.496503)
-		(end 144.861437 129.496503)
-		(width 0.25)
-		(layer "B.Cu")
-		(net 169)
-	)
-	(segment
-		(start 141.846437 120.646503)
-		(end 141.861437 120.661503)
-		(width 0.25)
+		(start 141.846437 124.346437)
+		(end 141.846437 120.646503)
+		(width 0.2)
 		(layer "B.Cu")
 		(net 169)
 	)
 	(segment
-		(start 141.861437 120.661503)
-		(end 141.861437 124.496503)
-		(width 0.25)
+		(start 144.361437 129.496503)
+		(end 144.361437 126.861437)
+		(width 0.2)
 		(layer "B.Cu")
 		(net 169)
 	)
 	(segment
-		(start 141.861437 124.496503)
-		(end 144.861437 127.496503)
-		(width 0.25)
+		(start 144.361437 126.861437)
+		(end 141.846437 124.346437)
+		(width 0.2)
 		(layer "B.Cu")
 		(net 169)
@@
 	)
 	(segment
-		(start 144.361437 129.496503)
-		(end 144.361437 127.996503)
+		(start 138.111437 124.996503)
+		(end 141.746503 124.996503)
 		(width 0.25)
 		(layer "B.Cu")
@@
 	)
 	(segment
-		(start 130.861437 115.496503)
-		(end 127.876437 112.511503)
+		(start 141.746503 124.996503)
+		(end 143.861437 127.111437)
 		(width 0.25)
 		(layer "B.Cu")
@@
 	)
 	(segment
-		(start 144.361437 127.996503)
-		(end 141.361437 124.996503)
+		(start 130.861437 115.496503)
+		(end 127.876437 112.511503)
 		(width 0.25)
 		(layer "B.Cu")
@@
 	)
 	(segment
-		(start 138.111437 124.996503)
-		(end 141.361437 124.996503)
+		(start 143.861437 127.111437)
+		(end 143.861437 129.496503)
 		(width 0.25)
 		(layer "B.Cu")
@@
 		(width 0.25)
 		(layer "B.Cu")
+		(net 172)
+	)
+	(segment
+		(start 144.861437 126.496503)
+		(end 144.861437 129.496503)
+		(width 0.25)
+		(layer "B.Cu")
