File: GPS-Compass_Arrow/GPS-Compass_Arrow.kicad_pcb (KiCad board)
At the start: 2 copper layers, 73.9 x 73.9 mm, 155 parts, among them IC1 74VHC9595FT, IC2 74VHC9595FT, IC3 74VHC9595FT, IC4 74VHC9595FT, IC5 74VHC9595FT, IC6 74VHC9595FT, IC7 74VHC9595FT, IC8 74VHC9595FT, J1 FFC2B28-12-G, J2 INDICATOR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

Commit message: generated step files
Routing:
- net /MOSI_SPI: track 27.6 -> 30.3 mm
Changed lines of the file:
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@@
 			(keep_text_aligned yes)
 		)
-		(gr_text "30,6147"
+		(gr_text "30.6147"
 			(at 182.507683 68.597498 315)
 			(layer "Dwgs.User")
@@
 			(keep_text_aligned yes)
 		)
-		(gr_text "73,9104"
+		(gr_text "73.9104"
 			(at 145.125 55.1 0)
 			(layer "Dwgs.User")
@@
 			(keep_text_aligned yes)
 		)
-		(gr_text "73,9104"
+		(gr_text "73.9104"
 			(at 78.85 105.980181 90)
 			(layer "Dwgs.User")
@@
 			(keep_text_aligned yes)
 		)
-		(gr_text "70,0114"
+		(gr_text "70.0114"
 			(at 145.105719 45.13 0)
 			(layer "Dwgs.User")
@@
 			(keep_text_aligned yes)
 		)
-		(gr_text "30,6147"
+		(gr_text "30.6147"
 			(at 145.125 62.05 0)
 			(layer "Edge.Cuts")
@@
 	)
 	(via
-		(at 109.611437 91.996503)
+		(at 110.361437 91.246503)
 		(size 0.5)
 		(drill 0.3)
@@
 	)
 	(via
-		(at 109.361437 97.496503)
+		(at 109.611437 95.746503)
 		(size 0.5)
 		(drill 0.3)
@@
 	)
 	(via
-		(at 112.861437 87.246503)
+		(at 113.861437 86.746503)
 		(size 0.5)
 		(drill 0.3)
@@
 	)
 	(segment
-		(start 141.846437 124.346437)
+		(start 141.846437 123.981503)
 		(end 141.846437 120.646503)
-		(width 0.2)
+		(width 0.25)
 		(layer "B.Cu")
 		(net 169)
@@
 	(segment
 		(start 144.361437 129.496503)
-		(end 144.361437 126.861437)
-		(width 0.2)
+		(end 144.361437 126.496503)
+		(width 0.25)
 		(layer "B.Cu")
 		(net 169)
 	)
 	(segment
-		(start 144.361437 126.861437)
-		(end 141.846437 124.346437)
-		(width 0.2)
+		(start 144.361437 126.496503)
+		(end 141.846437 123.981503)
+		(width 0.25)
 		(layer "B.Cu")
 		(net 169)
 	)
 	(segment
-		(start 130.861437 118.996503)
-		(end 136.861437 124.996503)
+		(start 135.361437 116.996503)
+		(end 138.111437 119.746503)
 		(width 0.25)
 		(layer "F.Cu")
@@
 	)
 	(segment
-		(start 136.861437 124.996503)
+		(start 138.111437 119.746503)
 		(end 138.111437 124.996503)
 		(width 0.25)
@@
 	)
 	(segment
-		(start 130.861437 115.496503)
-		(end 130.861437 118.996503)
+		(start 129.611437 116.996503)
+		(end 135.361437 116.996503)
 		(width 0.25)
 		(layer "F.Cu")
@@
 	)
 	(via
-		(at 130.861437 115.496503)
+		(at 129.611437 116.996503)
 		(size 0.5)
 		(drill 0.3)
@@
 	)
 	(segment
-		(start 127.876437 112.511503)
-		(end 127.876437 111.346503)
+		(start 141.746503 124.996503)
+		(end 143.861437 127.111437)
 		(width 0.25)
 		(layer "B.Cu")
@@
 	)
 	(segment
-		(start 141.746503 124.996503)
-		(end 143.861437 127.111437)
+		(start 129.611437 114.246503)
+		(end 127.876437 112.511503)
 		(width 0.25)
 		(layer "B.Cu")
@@
 	)
 	(segment
-		(start 130.861437 115.496503)
-		(end 127.876437 112.511503)
+		(start 129.611437 116.996503)
+		(end 129.611437 114.246503)
+		(width 0.25)
+		(layer "B.Cu")
+		(net 170)
+	)
+	(segment
+		(start 127.876437 112.511503)
+		(end 127.876437 111.346503)
 		(width 0.25)
 		(layer "B.Cu")
@@
 	)
 	(segment
-		(start 142.611437 124.246503)
+		(start 142.611437 123.496503)
 		(end 142.611437 112.246503)
 		(width 0.25)
@@
 	)
 	(via
-		(at 142.611437 124.246503)
+		(at 142.611437 123.496503)
 		(size 0.5)
 		(drill 0.3)
@@
 	)
 	(segment
-		(start 142.611437 124.246503)
-		(end 144.861437 126.496503)
+		(start 144.861437 125.746503)
+		(end 144.861437 129.496503)
 		(width 0.25)
 		(layer "B.Cu")
@@
 	)
 	(segment
-		(start 144.861437 126.496503)
-		(end 144.861437 129.496503)
+		(start 142.611437 123.496503)
+		(end 144.861437 125.746503)
 		(width 0.25)
 		(layer "B.Cu")

Commit message: 3d updates
Parts:
- H1, H2: value M2.5 -> M3; footprint MountingHole:MountingHole_2.5mm_Pad_Via -> MountingHole:MountingHole_3.2mm_M3_Pad_Via
- moved H1 22.4 mm to (186.8, 106.0)
- moved H2 22.4 mm to (103.5, 106.0)
Routing:
- net VBATT: track 49.8 -> 50.3 mm
Other:
- board size 73.9 x 73.9 mm -> 90.8 x 73.9 mm
