File: _electrical/GPS-Compass/GPS-Compass.kicad_sch (KiCad schematic)
At the start: 116 parts, among them J1 Conn_01x02_Pin, J2 USB_TypeC, J3 01x10, J4 01x10, J5 Conn_01x02_Pin, J6 FFC2B28-12-G, Q1 SI2393DS, SW1 SHIP-MODE, SW2 RST, SW3 RESET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

Commit message: renders, code
Other:
- note added: "possibly too little capacitance and indcutunce"
- note removed: "USE REGS TO CHANGE LIMIT"
- moved on the sheet: L3
Changed lines of the file:
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@@
 		)
 	)
-	(text "pinout checked"
-		(exclude_from_sim no)
-		(at 162.56 151.13 0)
-		(effects
-			(font
-				(size 1.27 1.27)
-			)
-			(justify left bottom)
-		)
-	)
 	(text "EEPROM"
 		(exclude_from_sim no)
@@
 		)
 	)
-	(text "pinout checked"
-		(exclude_from_sim no)
-		(at 220.345 64.135 0)
-		(effects
-			(font
-				(size 1.27 1.27)
-			)
-			(justify left bottom)
-		)
-	)
 	(text "MCU and IMU"
 		(exclude_from_sim no)
@@
 		)
 	)
-	(text "USE REGS TO CHANGE LIMIT"
+	(text "possibly too little capacitance and indcutunce"
 		(exclude_from_sim no)
-		(at 144.78 142.875 0)
+		(at 263.525 109.22 0)
 		(effects
 			(font
-				(size 1 1)
+				(size 1.27 1.27)
 			)
+			(justify left bottom)
 		)
 	)
@@
 		)
 	)
-	(text "pinout checked"
-		(exclude_from_sim no)
-		(at 179.07 64.77 0)
-		(effects
-			(font
-				(size 1.27 1.27)
-			)
-			(justify left bottom)
-		)
-	)
 	(text "GNSS CONN."
 		(exclude_from_sim no)
@@
 		)
 	)
-	(text "pinout checked"
-		(exclude_from_sim no)
-		(at 237.8823 109.3718 0)
-		(effects
-			(font
-				(size 1.27 1.27)
-			)
-			(justify left bottom)
-		)
-	)
-	(text "pinout checked"
-		(exclude_from_sim no)
-		(at 288.29 149.86 0)
-		(effects
-			(font
-				(size 1.27 1.27)
-			)
-			(justify left bottom)
-		)
-	)
 	(text "Typically these can be used, but you need to make sure they are \nnot in the wrong state during boot.\n\ngpio.0 Boot Mode. Weak pullup during reset. \n(Boot Mode 0=Boot from Flash, 1=Download)\ngpio.3 JTAG Mode. Weak pull down during reset. \n(JTAG Config)\ngpio.45 SPI voltage. Weak pull down during reset. \n(SPI Voltage 0=3.3v 1=1.8v)\ngpio.46 Boot mode. Weak pull down during reset. \n(Enabling/Disabling ROM Messages Print During Booting)"
 		(exclude_from_sim no)
@@
 		)
 	)
-	(polyline
-		(pts
-			(xy 252.095 69.85) (xy 256.54 69.85)
-		)
-		(stroke
-			(width 0)
-			(type default)
-		)
-	)
 	(wire
 		(pts
@@
 	(wire
 		(pts
-			(xy 276.86 92.71) (xy 287.02 92.71)
+			(xy 278.13 92.71) (xy 287.02 92.71)
 		)
 		(stroke
@@
 		)
 	)
-	(polyline
-		(pts
-			(xy 191.77 77.47) (xy 196.215 77.47)
-		)
-		(stroke
-			(width 0)
-			(type default)
-		)
-	)
 	(wire
 		(pts
@@
 	(wire
 		(pts
-			(xy 261.62 92.71) (xy 269.24 92.71)
+			(xy 261.62 92.71) (xy 270.51 92.71)
 		)
 		(stroke
@@
 		)
 	)
-	(polyline
-		(pts
-			(xy 123.825 69.85) (xy 128.27 69.85)
-		)
-		(stroke
-			(width 0)
-			(type default)
-		)
-	)
 	(wire
 		(pts
@@
 		)
 	)
-	(polyline
-		(pts
-			(xy 198.755 69.85) (xy 203.2 69.85)
-		)
-		(stroke
-			(width 0)
-			(type default)
-		)
-	)
 	(wire
 		(pts
@@
 	(symbol
 		(lib_id "Device:L")
-		(at 273.05 92.71 90)
+		(at 274.32 92.71 90)
 		(unit 1)
 		(exclude_from_sim no)
@@
 		(dnp no)
 		(property "Reference" "L3"
-			(at 273.05 88.265 90)
+			(at 274.32 88.265 90)
 			(effects
 				(font
@@
 		)
 		(property "Value" "1.5u"
-			(at 273.05 90.17 90)
+			(at 274.32 90.17 90)
 			(effects
 				(font
@@
 		)
 		(property "Footprint" "Inductor_SMD:L_Vishay_IHLP-1212"
-			(at 273.05 92.71 0)
+			(at 274.32 92.71 0)
 			(effects
 				(font
@@
 		)
 		(property "Datasheet" "https://cz.mouser.com/ProductDetail/Vishay-Dale/IHLP1212BZEV1R5M5A?qs=BJlw7L4Cy7%2FLPKyjRWwgFw%3D%3D"
-			(at 273.05 92.71 0)
+			(at 274.32 92.71 0)
 			(effects
 				(font
@@
 		)
 		(property "Description" "Inductor"
-			(at 273.05 92.71 0)
+			(at 274.32 92.71 0)
 			(effects
 				(font
@@
 		)
 		(property "Sim.Device" ""
-			(at 273.05 92.71 0)
+			(at 274.32 92.71 0)
 			(effects
 				(font
@@
 		)
 		(property "Sim.Pins" ""
-			(at 273.05 92.71 0)
+			(at 274.32 92.71 0)
 			(effects
 				(font
@@
 		)
 		(property "Sim.Type" ""
-			(at 273.05 92.71 0)
+			(at 274.32 92.71 0)
 			(effects
 				(font
@@
 		)
 		(property "Comment" ""
-			(at 273.05 92.71 90)
+			(at 274.32 92.71 90)
 			(effects
 				(font
