File: _electrical/GPS-Compass/GPS-Compass.kicad_sch (KiCad schematic)
At the start: 116 parts, among them J1 Conn_01x02_Pin, J2 USB_TypeC, J3 01x10, J4 01x10, J5 Conn_01x02_Pin, J6 FFC2B28-12-G, Q1 SI2393DS, SW1 SHIP-MODE, SW2 RST, SW3 RESET, SW4 BOOT, U1 USBLC6-2SC6, U2 ESP32-S3-WROOM-1, U3 BQ25895RTW, U4 FUSB302B11MPX, U5 BNO055, U6 KTS1605EUB-1-TR, U7 TPS613222ADBV, U8 TPS565242DRLR, U9 24CW1280T-I/OT, Y1 32.768k

Commit message: added DMP folder
I will sort it out later, most definitely
Parts:
- C28: now not fitted
Changed lines of the file:
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@@
 	(rectangle
 		(start 380.365 184.15)
-		(end 429.26 212.725)
+		(end 428.625 212.725)
 		(stroke
 			(width 0)
@@
 		(on_board yes)
 		(in_pos_files yes)
-		(dnp no)
+		(dnp yes)
 		(property "Reference" "C28"
 			(at 410.845 239.395 0)
