File: _electrical/GPS-Compass_Arrow/GPS-Compass_Arrow.kicad_sch (KiCad schematic)
At the start: 153 parts, among them IC1 74VHC9595FT, IC2 74VHC9595FT, IC3 74VHC9595FT, IC4 74VHC9595FT, IC5 74VHC9595FT, IC6 74VHC9595FT, IC7 74VHC9595FT, IC8 74VHC9595FT, J1 FFC2B28-12-G, J2 INDICATOR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

Commit message: Code update, schematic plots, text update
Other:
- note removed: "1) Uvod 2) Obsah 3) Koncept 4-7) Popis realizace 8) Zaver - splneni veci"
Changed lines of the file:
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@@
 		)
 	)
-	(text "1) Uvod\n2) Obsah\n3) Koncept\n4-7) Popis realizace\n8) Zaver - splneni veci"
-		(exclude_from_sim no)
-		(at 30.48 240.665 0)
-		(effects
-			(font
-				(size 3 3)
-			)
-			(justify left)
-		)
-	)
 	(text "CONNECTORS"
 		(exclude_from_sim no)
@@
 	)
 	(image
-		(at 355.6 118.11)
+		(at -66.675 116.205)
 		(data "iVBORw0KGgoAAAANSUhEUgAAAf4AAAFGCAYAAACL9v09AAAABHNCSVQICAgIfAhkiAAAIABJREFU"
 			"eJzs3XlUVVXjxvFvIFevTIIIgoACouAEOKE4m2maU86m9qZl+ZqVpjY7VDZp08/K10Yrs0FzTDPN"
