File: _electrical/GPS-Compass_GNSS/GPS-Compass_GNSS.kicad_sch (KiCad schematic)
At the start: 36 parts, among them J3 01x10, J4 636101112001, Q1 MMBT3904, SW1 GNSS_RST, U1 BGA725L6E6327FTSA1, U2 TESEO-LIV3R

Commit message: Code update, schematic plots, text update
Parts:
- removed AE1: Antenna, symbol Device:Antenna
Connections:
- no-connect marks 3 -> 2
